File: schematics/Full Board Prototype/Parallel CS Prototype pick & place ident.brd (EAGLE design)
At the start: 123.3 x 113.5 mm, 107 parts, among them U1 ADG714BRUZ, X2 CTR_ARD, X4 DSUB _T, X5 DSUB_B

Commit message: Added ident layer to gerbers and finalised Pick and Place data
Parts:
- removed I_OUT, I_OUT1, I_OUT2: 332-02, con-garry:332-02
- removed JP1, JP10, JP11, JP12, JP13, JP14, JP15, JP16, JP17, JP18, JP19, JP2, JP20, JP21, JP22, JP23, JP24, JP25, JP26, JP27, JP28, JP29, JP3, JP30, JP31, JP32, JP4, JP5, JP6, JP7, JP8, JP9: (no value), SwitchBoard:1X01
- removed JP33: PWR, pinhead:1X02
- removed JP34: (no value), SwitchBoard:1X02
- removed X2: CTR_ARD, con-subd:F09HP
- removed X4: DSUB _T, con-subd:F37HP
- removed X5: DSUB_B, con-subd:M37HP
Connections:
- removed net OUT_1: JP1.1, X4.1, X5.1
- removed net OUT_10: JP10.1, X4.10, X5.10
- removed net OUT_11: JP11.1, X4.11, X5.11
- removed net OUT_12: JP12.1, X4.12, X5.12
- removed net OUT_13: JP13.1, X4.13, X5.13
- removed net OUT_14: JP14.1, X4.14, X5.14
- removed net OUT_15: JP15.1, X4.15, X5.15
- removed net OUT_16: JP16.1, X4.16, X5.16
- removed net OUT_17: JP17.1, X4.17, X5.17
- removed net OUT_18: JP18.1, X4.18, X5.18
- removed net OUT_19: JP19.1, X4.19, X5.19
- removed net OUT_2: JP2.1, X4.2, X5.2
- removed net OUT_20: JP20.1, X4.20, X5.20
- removed net OUT_21: JP21.1, X4.21, X5.21
- removed net OUT_22: JP22.1, X4.22, X5.22
- removed net OUT_23: JP23.1, X4.23, X5.23
- removed net OUT_24: JP24.1, X4.24, X5.24
- removed net OUT_25: JP25.1, X4.25, X5.25
- removed net OUT_26: JP26.1, X4.26, X5.26
- removed net OUT_27: JP27.1, X4.27, X5.27
- removed net OUT_28: JP28.1, X4.28, X5.28
- removed net OUT_29: JP29.1, X4.29, X5.29
- removed net OUT_3: JP3.1, X4.3, X5.3
- removed net OUT_30: JP30.1, X4.30, X5.30
- removed net OUT_31: JP31.1, X4.31, X5.31
- removed net OUT_32: JP32.1, X4.32, X5.32
- removed net OUT_33: X4.33, X5.33
- removed net OUT_34: X4.34, X5.34
- removed net OUT_35: X4.35, X5.35
- removed net OUT_36: X4.36, X5.36
- removed net OUT_37: X4.37, X5.37
- removed net OUT_4: JP4.1, X4.4, X5.4
- removed net OUT_5: JP5.1, X4.5, X5.5
- removed net OUT_6: JP6.1, X4.6, X5.6
- removed net OUT_7: JP7.1, X4.7, X5.7
- removed net OUT_8: JP8.1, X4.8, X5.8
- removed net OUT_9: JP9.1, X4.9, X5.9
- net ARD_5V: no longer X2.4
- net FSYNC_ARD: no longer X2.9
- net GND: no longer JP33.1, JP34.2, X2.6
- net GND_CS: no longer I_OUT.2
- net GND_CS1: no longer I_OUT1.2
- net GND_CS2: no longer I_OUT2.2
- net IOUT: no longer I_OUT.1
- net IOUT1: no longer I_OUT1.1
- net IOUT2: no longer I_OUT2.1
- net SCLK_IN: no longer X2.2
- net SDATA_IN: no longer X2.3
- net SW_SCLK: no longer X2.1
- net SW_~RESET: no longer X2.8
- net SW_~SYNC: no longer X2.7
- net VDD: no longer JP33.2, JP34.1
Routing:
- net OUT_10: track 94.6 -> 0.00 mm
Other:
- board text removed: "Bottom Layer"
- board text removed: "Inner2"
- board text removed: "Top layer"
