File: schematics/Full Board Prototype/Parallel CS Prototype multiple sources.brd (EAGLE design)
At the start: 144.8 x 113.5 mm, 75 parts, among them U1 ADG714BRUZ, X2 CTR_ARD, X4 DSUB _T, X5 DSUB_B

Commit message: Finalised design for 8 channel parallel CS, to be submitted to fabrication house.
Parts:
- added CLOCK1: LTC69000, LTC6900:SOT95P280X100-6N
- added C_BIAS1: 4.7u, resistor:C0805
- added C_BYP1, C_DDS1: 10n, resistor:C0402
- added C_CLK_BYP1, C_DDS_BYP5, C_DDS_BYP8, C_ISO1B1, C_ISO2B1: 0.1u, resistor:C0402
- added C_DDS2: 100n, resistor:C0402
- added C_DDS_BYP6, C_DDS_BYP7: 10u, resistor:C0402
- added C_IN1: 2.2u, resistor:C0805
- added C_ISO1A1, C_ISO2A1: 1u, resistor:C0402
- added C_OUT3: 47u, resistor:C0805
- added C_OUT4: 10u, resistor:C0805
- added DDS1: AD9833BRMZ, ad9833:SOP50P490X110-10N
- added DIGITAL_ISO2: ADUM1410ARWZ, SwitchBoard:SOIC127P1032X265-16N
- added H_H1, R_H1, R_H1A1, R_H2A1: 10k, resistor:R0603
- added I_OUT1: 332-02, con-garry:332-02
- added LED2: (no value), eagle-ltspice:LED_SML0603
- added OPAMP1: LMC6482IMM, LMC6482:SOP65P490X109-8N
- added R_ADJ3: 6.8k, resistor:R0201
- added R_ADJ4: 300k, resistor:R0201
- added R_H1B1, R_H2B1: 3.3k, resistor:R0603
- added R_LED1: 2700, resistor:R0402
- added R_SET1: 20k, resistor:R0603
- added S3: TL36POPVB4, switch:PVB4-EE
- added S4: TL46WOMULTICOMP_2MD, switch:TL4XPO
- added TP_GND1, TP_VSIN1: PTR1PAD1-13, testpad:P1-13
- added U$2: LTM8048, LTM8048:BGA-49
Connections:
- new net ARD_5V1: C_ISO1A1.1, C_ISO1B1.1, DIGITAL_ISO2.1
- new net CLK_OUT1: CLOCK1.1, DDS1.5
- new net COMP1: C_DDS1.2, DDS1.1
- new net FSYNC1: DDS1.8, DIGITAL_ISO2.14
- new net FSYNC_IN1: DIGITAL_ISO2.3
- new net GND1: C_BIAS1.2, C_IN1.2, C_ISO1A1.2, C_ISO1B1.2, DIGITAL_ISO2.2, DIGITAL_ISO2.7, DIGITAL_ISO2.8, R_ADJ3.1, S3.1, U$2.GND@1, U$2.GND@10, U$2.GND@11, U$2.GND@12, U$2.GND@13, U$2.GND@14, U$2.GND@15, U$2.GND@16, U$2.GND@2, U$2.GND@3, U$2.GND@4, U$2.GND@5, U$2.GND@6, U$2.GND@7, U$2.GND@8, U$2.GND@9
- new net GND_CS1: CLOCK1.2, CLOCK1.3, C_CLK_BYP1.2, C_DDS2.1, C_DDS_BYP5.2, C_DDS_BYP6.2, C_DDS_BYP7.2, C_DDS_BYP8.2, C_ISO2A1.2, C_ISO2B1.2, C_OUT3.1, C_OUT4.1, DDS1.4, DDS1.9, DIGITAL_ISO2.15, DIGITAL_ISO2.9, I_OUT1.2, LED2.C, OPAMP1.4, R_ADJ4.2, R_H1.1, R_SET1.1, TP_GND1.TP, U$2.VOUT-@1, U$2.VOUT-@2, U$2.VOUT-@3, U$2.VOUT-@4, U$2.VOUT-@5, U$2.VOUT-@6, U$2.VOUT-@7, U$2.VOUT-@8, U$2.VOUT-@9
- new net IOUT1: I_OUT1.1, OPAMP1.3, S4.2
- new net N$16: C_BIAS1.1, U$2.BIAS
- new net N$17: R_ADJ3.2, U$2.ADJ1
- new net N$18: R_ADJ4.1, U$2.ADJ2
- new net N$19: C_BYP1.1, U$2.BYP
- new net N$20: C_DDS2.2, DDS1.3
- new net N$21: CLOCK1.4, R_SET1.2
- new net N$22: R_H1B1.2, R_H2B1.1, S4.1
- new net N$23: S3.2@1, S3.2@2, U$2.RUN
- new net N$24: LED2.A, R_LED1.1
- new net N$25: R_H2A1.2, S4.6
- new net N$26: R_H1A1.2, R_H2A1.1, S4.3
- new net N$27: R_H2B1.2, S4.4
- new net NEGA1: H_H1.1, OPAMP1.2, R_H1.2
- new net OP_OUTA1: H_H1.2, OPAMP1.1, S4.5
- new net SCLK1: DDS1.7, DIGITAL_ISO2.12
- new net SCLK_IN1: DIGITAL_ISO2.5
- new net SDATA1: DDS1.6, DIGITAL_ISO2.13
- new net SDATA_IN1: DIGITAL_ISO2.4
- new net VDD1: C_IN1.1, S3.3, U$2.VIN@1, U$2.VIN@2, U$2.VIN@3, U$2.VIN@4
- new net VDD_CS_ANA1: C_BYP1.2, C_DDS_BYP7.1, C_DDS_BYP8.1, C_OUT4.2, OPAMP1.8, U$2.VOUT2@1, U$2.VOUT2@2, U$2.VOUT2@3, U$2.VOUT2@4
- new net VDD_CS_DIG1: CLOCK1.6, C_CLK_BYP1.1, C_DDS1.1, C_DDS_BYP5.1, C_DDS_BYP6.1, C_ISO2A1.1, C_ISO2B1.1, C_OUT3.2, DDS1.2, DIGITAL_ISO2.16, R_LED1.2, U$2.VOUT1@1, U$2.VOUT1@2, U$2.VOUT1@3, U$2.VOUT1@4, U$2.VOUT1@5, U$2.VOUT1@6
- new net V_SINE1: DDS1.10, R_H1A1.1, R_H1B1.1, TP_VSIN1.TP
Routing:
- net GND_CS1: track 0.00 -> 71.7 mm, vias 0 -> 10
- net GND1: track 0.00 -> 51.6 mm, vias 0 -> 6
- net VDD_CS_DIG1: track 0.00 -> 50.2 mm, vias 0 -> 6
- net V_SINE1: track 0.00 -> 25.1 mm
- net SCLK_IN1: track 0.00 -> 20.6 mm
- net OP_OUTA1: track 0.00 -> 20.4 mm
- net SDATA_IN1: track 0.00 -> 19.7 mm
- net N$23: track 0.00 -> 19.0 mm
- net VDD_CS_ANA1: track 0.00 -> 17.9 mm, vias 0 -> 2
- net IOUT1: track 0.00 -> 17.9 mm, vias 0 -> 1
- net ARD_5V1: track 0.00 -> 17.7 mm, vias 0 -> 1
- net VDD1: track 0.00 -> 13.7 mm, vias 0 -> 2
- net SDATA1: track 0.00 -> 12.3 mm, vias 0 -> 2
- net SCLK1: track 0.00 -> 11.7 mm
- net FSYNC1: track 0.00 -> 9.97 mm
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- added copper zone on layer 15, net GND_CS1
- added copper zone on layer 2, net VDD_CS_ANA1
- added copper zone on layer 2, net VDD_CS_DIG1
Other:
- board text added: "Amplitude"
