File: schematics/Full Board Prototype/Parallel CS Prototype multiple sources.sch (EAGLE design)
At the start: 75 parts, among them U1 ADG714BRUZ, X2 CTR_ARD, X4 DSUB _T, X5 DSUB_B

Commit message: Finalised design for 8 channel parallel CS, to be submitted to fabrication house.
Parts:
- added CLOCK1: LTC69000, LTC6900:LTC69000
- added C_BIAS1: 4.7u, resistor:C-EUC0805
- added C_BYP1, C_DDS2: 10n, resistor:C-EUC0402
- added C_CLK_BYP1, C_DDS_BYP6, C_DDS_BYP8, C_ISO1B1, C_ISO2B1: 0.1u, resistor:C-EUC0402
- added C_DDS1: 100n, resistor:C-EUC0402
- added C_DDS_BYP5, C_DDS_BYP7: 10u, resistor:C-EUC0402
- added C_IN1: 2.2u, resistor:C-EUC0805
- added C_ISO1A1, C_ISO2A1: 1u, resistor:C-EUC0402
- added C_OUT3: 47u, resistor:C-EUC0805
- added C_OUT4: 10u, resistor:C-EUC0805
- added DDS1: AD9833BRMZ, ad9833:AD9833BRMZ
- added DIGITAL_ISO2: ADUM1410ARWZ, SwitchBoard:ADUM1410ARWZ
- added H_H1, R_H1, R_H1A1, R_H2A1: 10k, resistor:R-US_R0603
- added I_OUT1: 332-02, con-garry:332-02
- added LED2: (no value), eagle-ltspice:LED_ESML0603
- added OPAMP1: LMC6482IMM, LMC6482:LMC6482IMM
- added R_ADJ3: 6.8k, resistor:R-US_R0201
- added R_ADJ4: 300k, resistor:R-US_R0201
- added R_H1B1, R_H2B1: 3.3k, resistor:R-US_R0603
- added R_LED1: 2700, resistor:R-US_R0402
- added R_SET1: 20k, resistor:R-US_R0603
- added S3: TL36POPVB4, switch:TL36POPVB4
- added S4: TL46WOMULTICOMP_2MD, switch:TL46WOMULTICOMP_2MD
- added TP_GND1, TP_VSIN1: PTR1PAD1-13, testpad:PTR1PAD1-13
- added U$2: LTM8048, LTM8048:LTM8048
Connections:
- new net CLK_OUT1: CLOCK1.OUT, DDS1.MCLK
- new net IOUT1: I_OUT1-1.S, OPAMP1.POSA, S4.P
- new net N$14: R_ADJ4.1, U$2.ADJ2
- new net N$16: C_BYP1.1, U$2.BYP
- new net N$17: S3.P, U$2.RUN
- new net N$18: LED2.A, R_LED1.1
- new net N$19: C_DDS1.2, DDS1.CAP/2.5V
- new net N$20: CLOCK1.SET, R_SET1.2
- new net N$21: R_H1B1.2, R_H2B1.1, S4.O
- new net N$22: R_H2A1.2, S4.S1
- new net N$23: R_H1A1.2, R_H2A1.1, S4.S
- new net N$24: R_H2B1.2, S4.O1
- new net N$4: C_BIAS1.1, U$2.BIAS
- new net N$5: R_ADJ3.2, U$2.ADJ1
- new net NEGA1: H_H1.1, OPAMP1.NEGA, R_H1.2
- new net V_SINE1: DDS1.VOUT, R_H1A1.1, R_H1B1.1, TP_VSIN1.TP
- net ARD_5V: now also C_ISO1A1.1, C_ISO1B1.1, DIGITAL_ISO2.VDD1
- net COMP: now also C_DDS2.2, DDS1.COMP
- net FSYNC: now also DDS1.FSYNC, DIGITAL_ISO2.VOA
- net FSYNC_IN: now also DIGITAL_ISO2.VIA
- net GND: now also C_BIAS1.2, C_IN1.2, C_ISO1A1.2, C_ISO1B1.2, DIGITAL_ISO2.DISABLE, DIGITAL_ISO2.GND1, DIGITAL_ISO2.GND1_2, R_ADJ3.1, S3.O, U$2.GND
- net GND_CS: now also CLOCK1.DIV, CLOCK1.GND, C_CLK_BYP1.2, C_DDS1.1, C_DDS_BYP5.2, C_DDS_BYP6.2, C_DDS_BYP7.2, C_DDS_BYP8.2, C_ISO2A1.2, C_ISO2B1.2, C_OUT3.1, C_OUT4.1, DDS1.AGND, DDS1.DGND, DIGITAL_ISO2.GND2, DIGITAL_ISO2.GND2_2, I_OUT1-2.S, LED2.C, OPAMP1.V-, R_ADJ4.2, R_H1.1, R_SET1.1, TP_GND1.TP, U$2.VOUT-
- net OP_OUTA: now also H_H1.2, OPAMP1.OUTA, S4.P1
- net SCLK: now also DDS1.SCLK, DIGITAL_ISO2.VOC
- net SCLK_IN: now also DIGITAL_ISO2.VIC
- net SDATA: now also DDS1.SDATA, DIGITAL_ISO2.VOB
- net SDATA_IN: now also DIGITAL_ISO2.VIB
- net VDD: now also C_IN1.1, S3.S, U$2.VIN
- net VDD_CS_ANA: now also C_BYP1.2, C_DDS_BYP7.1, C_DDS_BYP8.1, C_OUT4.2, OPAMP1.V+, U$2.VOUT2
- net VDD_CS_DIG: now also CLOCK1.V+, C_CLK_BYP1.1, C_DDS2.1, C_DDS_BYP5.1, C_DDS_BYP6.1, C_ISO2A1.1, C_ISO2B1.1, C_OUT3.2, DDS1.VDD, DIGITAL_ISO2.VDD2, R_LED1.2, U$2.VOUT1
