File: schematics/Full Board Prototype/Parallel CS Prototype not linked to schematic.brd (EAGLE design)
At the start: 123.3 x 113.5 mm, 107 parts, among them U1 ADG714BRUZ, X2 CTR_ARD, X4 DSUB _T, X5 DSUB_B

Commit message: Finalised design for 8 channel parallel CS, to be submitted to fabrication house.
Parts:
- removed RN1, RN2, RN3: CTS742C083, resistor-net:CTS742C083
- added CLOCK3, CLOCK4, CLOCK5, CLOCK6, CLOCK7: LTC69000, LTC6900:SOT95P280X100-6N
- added C_BIAS3, C_BIAS4, C_BIAS5, C_BIAS6, C_BIAS7: 4.7u, resistor:C0805
- added C_BYP3, C_BYP4, C_BYP5, C_BYP6, C_BYP7, C_DDS11, C_DDS13, C_DDS15, C_DDS7, C_DDS9: 10n, resistor:C0402
- added C_CLK_BYP, C_CLK_BYP1, C_CLK_BYP2, C_CLK_BYP3, C_CLK_BYP4, C_CLK_BYP5, C_CLK_BYP6, C_CLK_BYP7, C_DDS_BYP12, C_DDS_BYP13, C_DDS_BYP16, C_DDS_BYP17, C_DDS_BYP20, C_DDS_BYP21, C_DDS_BYP24, C_DDS_BYP25, C_DDS_BYP28, C_DDS_BYP29, C_DDS_BYP32, C_DDS_BYP8, C_DDS_BYP9, C_ISO1B3, C_ISO1B4, C_ISO1B5, C_ISO1B6, C_ISO1B7, C_ISO2B3, C_ISO2B4, C_ISO2B5, C_ISO2B6, C_ISO2B7: 0.1u, resistor:C0402
- added C_DDS10, C_DDS12, C_DDS14, C_DDS16, C_DDS8: 100n, resistor:C0402
- added C_DDS_BYP10, C_DDS_BYP11, C_DDS_BYP14, C_DDS_BYP15, C_DDS_BYP18, C_DDS_BYP19, C_DDS_BYP22, C_DDS_BYP23, C_DDS_BYP26, C_DDS_BYP27, C_DDS_BYP30, C_DDS_BYP31, C_DDS_BYP7: 10u, resistor:C0402
- added C_IN3, C_IN4, C_IN5, C_IN6, C_IN7: 2.2u, resistor:C0805
- added C_ISO1A3, C_ISO1A4, C_ISO1A5, C_ISO1A6, C_ISO1A7, C_ISO2A3, C_ISO2A4, C_ISO2A5, C_ISO2A6, C_ISO2A7: 1u, resistor:C0402
- added C_OUT10, C_OUT12, C_OUT14, C_OUT16, C_OUT8: 10u, resistor:C0805
- added C_OUT11, C_OUT13, C_OUT15, C_OUT7, C_OUT9: 47u, resistor:C0805
- added DDS3, DDS4, DDS5, DDS6, DDS7: AD9833BRMZ, ad9833:SOP50P490X110-10N
- added DIGITAL_ISO4, DIGITAL_ISO5, DIGITAL_ISO6, DIGITAL_ISO7, DIGITAL_ISO8: ADUM1410ARWZ, SwitchBoard:SOIC127P1032X265-16N
- added H_H1, H_H2, H_H3, H_H4, H_H5, H_H6, H_H7, H_H8, R_H1, R_H1A, R_H1A1, R_H1A2, R_H1A3, R_H1A4, R_H1A5, R_H1A6, R_H1A7, R_H2, R_H2A, R_H2A1, R_H2A2, R_H2A3, R_H2A4, R_H2A5, R_H2A6, R_H2A7, R_H3, R_H4, R_H5, R_H6, R_H7, R_H8: 10k, resistor:R0603
- added I_OUT3, I_OUT4, I_OUT5, I_OUT6, I_OUT7: 332-02, con-garry:332-02
- added LED1, LED2, LED3, LED4, LED5, LED6, LED7, LED8: (no value), eagle-ltspice:LED_SML0603
- added OPAMP3, OPAMP4, OPAMP5, OPAMP6, OPAMP7: LMC6482IMM, LMC6482:SOP65P490X109-8N
- added R_ADJ10, R_ADJ12, R_ADJ14, R_ADJ16, R_ADJ8: 300k, resistor:R0201
- added R_ADJ11, R_ADJ13, R_ADJ15, R_ADJ7, R_ADJ9: 6.8k, resistor:R0201
- added R_H1B, R_H1B1, R_H1B2, R_H1B3, R_H1B4, R_H1B5, R_H1B6, R_H1B7, R_H2B, R_H2B1, R_H2B2, R_H2B3, R_H2B4, R_H2B5, R_H2B6, R_H2B7: 3.3k, resistor:R0603
- added R_LED, R_LED1, R_LED2, R_LED3, R_LED4, R_LED5, R_LED6, R_LED7: 2700, resistor:R0402
- added R_SET3, R_SET4, R_SET5, R_SET6, R_SET7: 20k, resistor:R0603
- added S1, S11, S13, S15, S3, S5, S7, S9: TL36POPVB4, switch:PVB4-EE
- added S10, S12, S14, S16, S2, S4, S6, S8: TL46WOMULTICOMP_2MD, switch:TL4XPO
- added TP_GND, TP_GND1, TP_GND2, TP_GND3, TP_GND4, TP_GND5, TP_GND6, TP_GND7, TP_VSIN, TP_VSIN1, TP_VSIN2, TP_VSIN3, TP_VSIN4, TP_VSIN5, TP_VSIN6, TP_VSIN7: PTR1PAD1-13, testpad:P1-13
- added U$4, U$5, U$6, U$7, U$8: LTM8048, LTM8048:BGA-49
- CLOCK, CLOCK1, CLOCK2: value LTC6906IS6PBF -> LTC69000; device LTC6906:SOT95P280X100-6N -> LTC6900:SOT95P280X100-6N
- C_BYP, C_BYP1, C_BYP2: value 0.01u -> 10n; device resistor:C0201 -> resistor:C0402
- C_DDS_BYP3: value 0.1u -> 10u
- C_DDS_BYP4: value 10u -> 0.1u
- R_SET, R_SET1, R_SET2: value 200k -> 20k
- moved X5 146.1 mm to (91.3, -137.3)
- moved U1 125.4 mm to (-9.53, -55.5)
- moved JP20 113.5 mm to (67.8, -49.1)
- moved JP21 113.5 mm to (70.5, -49.1)
- moved JP22 113.5 mm to (73.3, -49.1)
- moved JP23 113.5 mm to (76.0, -49.1)
- moved JP24 113.5 mm to (78.9, -49.1)
- moved JP25 113.5 mm to (81.6, -49.1)
- moved JP26 113.5 mm to (84.3, -49.1)
- moved JP27 113.5 mm to (87.2, -49.1)
- moved JP28 113.5 mm to (89.9, -49.1)
- moved JP29 113.5 mm to (92.7, -49.1)
- moved JP30 113.5 mm to (95.4, -49.1)
- moved JP31 113.5 mm to (98.3, -49.1)
- moved JP32 113.5 mm to (101.0, -49.1)
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Connections:
- removed net N$16 (its old number): OPAMP1.2, RN2.3, RN2.4
- removed net N$17 (its old number): OPAMP1.1, RN2.6, RN2.7
- removed net SCLK_IN1: DIGITAL_ISO2.5
- removed net SCLK_IN2: DIGITAL_ISO3.5
- removed net SDATA_IN1: DIGITAL_ISO2.4
- removed net SDATA_IN2: DIGITAL_ISO3.4
- new net CLK_OUT3: CLOCK3.1, DDS3.5
- new net CLK_OUT4: CLOCK4.1, DDS4.5
- new net CLK_OUT5: CLOCK5.1, DDS5.5
- new net CLK_OUT6: CLOCK6.1, DDS6.5
- new net CLK_OUT7: CLOCK7.1, DDS7.5
- new net COMP3: C_DDS7.2, DDS3.1
- new net COMP4: C_DDS9.2, DDS4.1
- new net COMP5: C_DDS11.2, DDS5.1
- new net COMP6: C_DDS13.2, DDS6.1
- new net COMP7: C_DDS15.2, DDS7.1
- new net FSYNC3: DDS3.8, DIGITAL_ISO4.14
- new net FSYNC4: DDS4.8, DIGITAL_ISO5.14
- new net FSYNC5: DDS5.8, DIGITAL_ISO6.14
- new net FSYNC6: DDS6.8, DIGITAL_ISO7.14
- new net FSYNC7: DDS7.8, DIGITAL_ISO8.14
- new net FSYNC_IN3: DIGITAL_ISO4.3
- new net FSYNC_IN4: DIGITAL_ISO5.3
- new net FSYNC_IN5: DIGITAL_ISO6.3
- new net FSYNC_IN6: DIGITAL_ISO7.3
- new net FSYNC_IN7: DIGITAL_ISO8.3
- new net GND_CS3: CLOCK3.2, CLOCK3.3, C_CLK_BYP3.2, C_DDS8.1, C_DDS_BYP13.2, C_DDS_BYP14.2, C_DDS_BYP15.2, C_DDS_BYP16.2, C_ISO2A3.2, C_ISO2B3.2, C_OUT7.1, C_OUT8.1, DDS3.4, DDS3.9, DIGITAL_ISO4.15, DIGITAL_ISO4.9, I_OUT3.2, LED4.C, OPAMP3.4, R_ADJ8.2, R_H4.1, R_SET3.1, TP_GND3.TP, U$4.VOUT-@1, U$4.VOUT-@2, U$4.VOUT-@3, U$4.VOUT-@4, U$4.VOUT-@5, U$4.VOUT-@6, U$4.VOUT-@7, U$4.VOUT-@8, U$4.VOUT-@9
- new net GND_CS4: CLOCK4.2, CLOCK4.3, C_CLK_BYP4.2, C_DDS10.1, C_DDS_BYP17.2, C_DDS_BYP18.2, C_DDS_BYP19.2, C_DDS_BYP20.2, C_ISO2A4.2, C_ISO2B4.2, C_OUT10.1, C_OUT9.1, DDS4.4, DDS4.9, DIGITAL_ISO5.15, DIGITAL_ISO5.9, I_OUT4.2, LED5.C, OPAMP4.4, R_ADJ10.2, R_H5.1, R_SET4.1, TP_GND4.TP, U$5.VOUT-@1, U$5.VOUT-@2, U$5.VOUT-@3, U$5.VOUT-@4, U$5.VOUT-@5, U$5.VOUT-@6, U$5.VOUT-@7, U$5.VOUT-@8, U$5.VOUT-@9
- new net GND_CS5: CLOCK5.2, CLOCK5.3, C_CLK_BYP5.2, C_DDS12.1, C_DDS_BYP21.2, C_DDS_BYP22.2, C_DDS_BYP23.2, C_DDS_BYP24.2, C_ISO2A5.2, C_ISO2B5.2, C_OUT11.1, C_OUT12.1, DDS5.4, DDS5.9, DIGITAL_ISO6.15, DIGITAL_ISO6.9, I_OUT5.2, LED6.C, OPAMP5.4, R_ADJ12.2, R_H6.1, R_SET5.1, TP_GND5.TP, U$6.VOUT-@1, U$6.VOUT-@2, U$6.VOUT-@3, U$6.VOUT-@4, U$6.VOUT-@5, U$6.VOUT-@6, U$6.VOUT-@7, U$6.VOUT-@8, U$6.VOUT-@9
- new net GND_CS6: CLOCK6.2, CLOCK6.3, C_CLK_BYP6.2, C_DDS14.1, C_DDS_BYP25.2, C_DDS_BYP26.2, C_DDS_BYP27.2, C_DDS_BYP28.2, C_ISO2A6.2, C_ISO2B6.2, C_OUT13.1, C_OUT14.1, DDS6.4, DDS6.9, DIGITAL_ISO7.15, DIGITAL_ISO7.9, I_OUT6.2, LED7.C, OPAMP6.4, R_ADJ14.2, R_H7.1, R_SET6.1, TP_GND6.TP, U$7.VOUT-@1, U$7.VOUT-@2, U$7.VOUT-@3, U$7.VOUT-@4, U$7.VOUT-@5, U$7.VOUT-@6, U$7.VOUT-@7, U$7.VOUT-@8, U$7.VOUT-@9
- new net GND_CS7: CLOCK7.2, CLOCK7.3, C_CLK_BYP7.2, C_DDS16.1, C_DDS_BYP29.2, C_DDS_BYP30.2, C_DDS_BYP31.2, C_DDS_BYP32.2, C_ISO2A7.2, C_ISO2B7.2, C_OUT15.1, C_OUT16.1, DDS7.4, DDS7.9, DIGITAL_ISO8.15, DIGITAL_ISO8.9, I_OUT7.2, LED8.C, OPAMP7.4, R_ADJ16.2, R_H8.1, R_SET7.1, TP_GND7.TP, U$8.VOUT-@1, U$8.VOUT-@2, U$8.VOUT-@3, U$8.VOUT-@4, U$8.VOUT-@5, U$8.VOUT-@6, U$8.VOUT-@7, U$8.VOUT-@8, U$8.VOUT-@9
- new net IOUT3: I_OUT3.1, OPAMP3.3, S8.2
- new net IOUT4: I_OUT4.1, OPAMP4.3, S10.2
- new net IOUT5: I_OUT5.1, OPAMP5.3, S12.2
- new net IOUT6: I_OUT6.1, OPAMP6.3, S14.2
- new net IOUT7: I_OUT7.1, OPAMP7.3, S16.2
- new net N$100: R_H1B7.2, R_H2B7.1, S16.1
- new net N$101: S15.2@1, S15.2@2, U$8.RUN
- new net N$102: LED8.A, R_LED7.1
- new net N$103: R_H2A7.2, S16.6
- new net N$104: R_H1A7.2, R_H2A7.1, S16.3
- new net N$105: R_H2B7.2, S16.4
- new net N$12: R_H1B.2, R_H2B.1, S2.1
- new net N$15: R_H1A.2, R_H2A.1, S2.3
- new net N$22: R_H1B1.2, R_H2B1.1, S4.1
- new net N$23: S3.2@1, S3.2@2, U$2.RUN
- new net N$24: LED2.A, R_LED1.1
- new net N$25: R_H2A1.2, S4.6
- new net N$35: R_H1B2.2, R_H2B2.1, S6.1
- new net N$36: S5.2@1, S5.2@2, U$3.RUN
- new net N$37: LED3.A, R_LED2.1
- new net N$38: R_H2A2.2, S6.6
- new net N$39: R_H1A2.2, R_H2A2.1, S6.3
- new net N$40: R_H2B2.2, S6.4
- new net N$42: C_BIAS3.1, U$4.BIAS
- new net N$43: R_ADJ7.2, U$4.ADJ1
- new net N$44: R_ADJ8.1, U$4.ADJ2
- new net N$45: C_BYP3.1, U$4.BYP
- new net N$46: C_DDS8.2, DDS3.3
- new net N$47: CLOCK3.4, R_SET3.2
- new net N$48: R_H1B3.2, R_H2B3.1, S8.1
- new net N$49: S7.2@1, S7.2@2, U$4.RUN
- new net N$50: LED4.A, R_LED3.1
- new net N$51: R_H2A3.2, S8.6
- new net N$52: R_H1A3.2, R_H2A3.1, S8.3
- new net N$53: R_H2B3.2, S8.4
- new net N$55: C_BIAS4.1, U$5.BIAS
- new net N$56: R_ADJ9.2, U$5.ADJ1
- new net N$57: R_ADJ10.1, U$5.ADJ2
- new net N$58: C_BYP4.1, U$5.BYP
- new net N$59: C_DDS10.2, DDS4.3
- new net N$6: LED1.A, R_LED.1
- new net N$60: CLOCK4.4, R_SET4.2
- new net N$61: R_H1B4.2, R_H2B4.1, S10.1
- new net N$62: S9.2@1, S9.2@2, U$5.RUN
- new net N$63: LED5.A, R_LED4.1
- new net N$64: R_H2A4.2, S10.6
- new net N$65: R_H1A4.2, R_H2A4.1, S10.3
- new net N$66: R_H2B4.2, S10.4
- new net N$68: C_BIAS5.1, U$6.BIAS
- new net N$69: R_ADJ11.2, U$6.ADJ1
- new net N$70: R_ADJ12.1, U$6.ADJ2
- new net N$71: C_BYP5.1, U$6.BYP
- new net N$72: C_DDS12.2, DDS5.3
- new net N$73: CLOCK5.4, R_SET5.2
- new net N$74: R_H1B5.2, R_H2B5.1, S12.1
- new net N$75: S11.2@1, S11.2@2, U$6.RUN
- new net N$76: LED6.A, R_LED5.1
- new net N$77: R_H2A5.2, S12.6
- new net N$78: R_H1A5.2, R_H2A5.1, S12.3
- new net N$79: R_H2B5.2, S12.4
- new net N$81: C_BIAS6.1, U$7.BIAS
- new net N$82: R_ADJ13.2, U$7.ADJ1
- new net N$83: R_ADJ14.1, U$7.ADJ2
- new net N$84: C_BYP6.1, U$7.BYP
- new net N$85: C_DDS14.2, DDS6.3
- new net N$86: CLOCK6.4, R_SET6.2
- new net N$87: R_H1B6.2, R_H2B6.1, S14.1
- new net N$88: S13.2@1, S13.2@2, U$7.RUN
- new net N$89: LED7.A, R_LED6.1
- new net N$9: R_H2B.2, S2.4
- new net N$90: R_H2A6.2, S14.6
- new net N$91: R_H1A6.2, R_H2A6.1, S14.3
- new net N$92: R_H2B6.2, S14.4
- new net N$94: C_BIAS7.1, U$8.BIAS
- new net N$95: R_ADJ15.2, U$8.ADJ1
- new net N$96: R_ADJ16.1, U$8.ADJ2
- new net N$97: C_BYP7.1, U$8.BYP
- new net N$98: C_DDS16.2, DDS7.3
- new net N$99: CLOCK7.4, R_SET7.2
- new net NEGA: H_H4.1, OPAMP.2, R_H3.2
- new net NEGA1: H_H1.1, OPAMP1.2, R_H1.2
- new net NEGA2: H_H2.1, OPAMP2.2, R_H2.2
- new net NEGA3: H_H3.1, OPAMP3.2, R_H4.2
- new net NEGA4: H_H5.1, OPAMP4.2, R_H5.2
- new net NEGA5: H_H6.1, OPAMP5.2, R_H6.2
- new net NEGA6: H_H7.1, OPAMP6.2, R_H7.2
- new net NEGA7: H_H8.1, OPAMP7.2, R_H8.2
- new net OP_OUTA: H_H4.2, OPAMP.1, S2.5
- new net OP_OUTA1: H_H1.2, OPAMP1.1, S4.5
- new net OP_OUTA2: H_H2.2, OPAMP2.1, S6.5
- new net OP_OUTA3: H_H3.2, OPAMP3.1, S8.5
- new net OP_OUTA4: H_H5.2, OPAMP4.1, S10.5
- new net OP_OUTA5: H_H6.2, OPAMP5.1, S12.5
- new net OP_OUTA6: H_H7.2, OPAMP6.1, S14.5
- new net OP_OUTA7: H_H8.2, OPAMP7.1, S16.5
- new net SCLK3: DDS3.7, DIGITAL_ISO4.12
- new net SCLK4: DDS4.7, DIGITAL_ISO5.12
- new net SCLK5: DDS5.7, DIGITAL_ISO6.12
- new net SCLK6: DDS6.7, DIGITAL_ISO7.12
- new net SCLK7: DDS7.7, DIGITAL_ISO8.12
- new net SDATA3: DDS3.6, DIGITAL_ISO4.13
- new net SDATA4: DDS4.6, DIGITAL_ISO5.13
- new net SDATA5: DDS5.6, DIGITAL_ISO6.13
- new net SDATA6: DDS6.6, DIGITAL_ISO7.13
- new net SDATA7: DDS7.6, DIGITAL_ISO8.13
- new net SW_DIN: U1.3, X2.5
- new net VDD_CS_ANA3: C_BYP3.2, C_DDS_BYP15.1, C_DDS_BYP16.1, C_OUT8.2, OPAMP3.8, U$4.VOUT2@1, U$4.VOUT2@2, U$4.VOUT2@3, U$4.VOUT2@4
- new net VDD_CS_ANA4: C_BYP4.2, C_DDS_BYP19.1, C_DDS_BYP20.1, C_OUT10.2, OPAMP4.8, U$5.VOUT2@1, U$5.VOUT2@2, U$5.VOUT2@3, U$5.VOUT2@4
- new net VDD_CS_ANA5: C_BYP5.2, C_DDS_BYP23.1, C_DDS_BYP24.1, C_OUT12.2, OPAMP5.8, U$6.VOUT2@1, U$6.VOUT2@2, U$6.VOUT2@3, U$6.VOUT2@4
- new net VDD_CS_ANA6: C_BYP6.2, C_DDS_BYP27.1, C_DDS_BYP28.1, C_OUT14.2, OPAMP6.8, U$7.VOUT2@1, U$7.VOUT2@2, U$7.VOUT2@3, U$7.VOUT2@4
- new net VDD_CS_ANA7: C_BYP7.2, C_DDS_BYP31.1, C_DDS_BYP32.1, C_OUT16.2, OPAMP7.8, U$8.VOUT2@1, U$8.VOUT2@2, U$8.VOUT2@3, U$8.VOUT2@4
- new net VDD_CS_DIG3: CLOCK3.6, C_CLK_BYP3.1, C_DDS7.1, C_DDS_BYP13.1, C_DDS_BYP14.1, C_ISO2A3.1, C_ISO2B3.1, C_OUT7.2, DDS3.2, DIGITAL_ISO4.16, R_LED3.2, U$4.VOUT1@1, U$4.VOUT1@2, U$4.VOUT1@3, U$4.VOUT1@4, U$4.VOUT1@5, U$4.VOUT1@6
- new net VDD_CS_DIG4: CLOCK4.6, C_CLK_BYP4.1, C_DDS9.1, C_DDS_BYP17.1, C_DDS_BYP18.1, C_ISO2A4.1, C_ISO2B4.1, C_OUT9.2, DDS4.2, DIGITAL_ISO5.16, R_LED4.2, U$5.VOUT1@1, U$5.VOUT1@2, U$5.VOUT1@3, U$5.VOUT1@4, U$5.VOUT1@5, U$5.VOUT1@6
- new net VDD_CS_DIG5: CLOCK5.6, C_CLK_BYP5.1, C_DDS11.1, C_DDS_BYP21.1, C_DDS_BYP22.1, C_ISO2A5.1, C_ISO2B5.1, C_OUT11.2, DDS5.2, DIGITAL_ISO6.16, R_LED5.2, U$6.VOUT1@1, U$6.VOUT1@2, U$6.VOUT1@3, U$6.VOUT1@4, U$6.VOUT1@5, U$6.VOUT1@6
- new net VDD_CS_DIG6: CLOCK6.6, C_CLK_BYP6.1, C_DDS13.1, C_DDS_BYP25.1, C_DDS_BYP26.1, C_ISO2A6.1, C_ISO2B6.1, C_OUT13.2, DDS6.2, DIGITAL_ISO7.16, R_LED6.2, U$7.VOUT1@1, U$7.VOUT1@2, U$7.VOUT1@3, U$7.VOUT1@4, U$7.VOUT1@5, U$7.VOUT1@6
- new net VDD_CS_DIG7: CLOCK7.6, C_CLK_BYP7.1, C_DDS15.1, C_DDS_BYP29.1, C_DDS_BYP30.1, C_ISO2A7.1, C_ISO2B7.1, C_OUT15.2, DDS7.2, DIGITAL_ISO8.16, R_LED7.2, U$8.VOUT1@1, U$8.VOUT1@2, U$8.VOUT1@3, U$8.VOUT1@4, U$8.VOUT1@5, U$8.VOUT1@6
- new net V_SINE3: DDS3.10, R_H1A3.1, R_H1B3.1, TP_VSIN3.TP
- new net V_SINE4: DDS4.10, R_H1A4.1, R_H1B4.1, TP_VSIN4.TP
- new net V_SINE5: DDS5.10, R_H1A5.1, R_H1B5.1, TP_VSIN5.TP
- new net V_SINE6: DDS6.10, R_H1A6.1, R_H1B6.1, TP_VSIN6.TP
- new net V_SINE7: DDS7.10, R_H1A7.1, R_H1B7.1, TP_VSIN7.TP
- net ARD_5V: now also C_ISO1A3.1, C_ISO1A4.1, C_ISO1A5.1, C_ISO1A6.1, C_ISO1A7.1, C_ISO1B3.1, C_ISO1B4.1, C_ISO1B5.1, C_ISO1B6.1, C_ISO1B7.1, DIGITAL_ISO4.1, DIGITAL_ISO5.1, DIGITAL_ISO6.1, DIGITAL_ISO7.1, DIGITAL_ISO8.1
- net GND: now also C_BIAS3.2, C_BIAS4.2, C_BIAS5.2, C_BIAS6.2, C_BIAS7.2, C_IN3.2, C_IN4.2, C_IN5.2, C_IN6.2, C_IN7.2, C_ISO1A3.2, C_ISO1A4.2, C_ISO1A5.2, C_ISO1A6.2, C_ISO1A7.2, C_ISO1B3.2, C_ISO1B4.2, C_ISO1B5.2, C_ISO1B6.2, C_ISO1B7.2, DIGITAL_ISO4.2, DIGITAL_ISO4.7, DIGITAL_ISO4.8, DIGITAL_ISO5.2, DIGITAL_ISO5.7, DIGITAL_ISO5.8, DIGITAL_ISO6.2, DIGITAL_ISO6.7, DIGITAL_ISO6.8, DIGITAL_ISO7.2, DIGITAL_ISO7.7, DIGITAL_ISO7.8, DIGITAL_ISO8.2, DIGITAL_ISO8.7, DIGITAL_ISO8.8, R_ADJ11.1, R_ADJ13.1, R_ADJ15.1, R_ADJ7.1, R_ADJ9.1, S1.1, S11.1, S13.1, S15.1, S3.1, S5.1, S7.1, S9.1, U$4.GND@1, U$4.GND@10, U$4.GND@11, U$4.GND@12, U$4.GND@13, U$4.GND@14, U$4.GND@15, U$4.GND@16, U$4.GND@2, U$4.GND@3, U$4.GND@4, U$4.GND@5, U$4.GND@6, U$4.GND@7, U$4.GND@8, U$4.GND@9, U$5.GND@1, U$5.GND@10, U$5.GND@11, U$5.GND@12, U$5.GND@13, U$5.GND@14, U$5.GND@15, U$5.GND@16, U$5.GND@2, U$5.GND@3, U$5.GND@4, U$5.GND@5, U$5.GND@6, U$5.GND@7, U$5.GND@8, U$5.GND@9, U$6.GND@1, U$6.GND@10, U$6.GND@11, U$6.GND@12, U$6.GND@13, U$6.GND@14, U$6.GND@15, U$6.GND@16, U$6.GND@2, U$6.GND@3, U$6.GND@4, U$6.GND@5, U$6.GND@6, U$6.GND@7, U$6.GND@8, U$6.GND@9, U$7.GND@1, U$7.GND@10, U$7.GND@11, U$7.GND@12, U$7.GND@13, U$7.GND@14, U$7.GND@15, U$7.GND@16, U$7.GND@2, U$7.GND@3, U$7.GND@4, U$7.GND@5, U$7.GND@6, U$7.GND@7, U$7.GND@8, U$7.GND@9, U$8.GND@1, U$8.GND@10, U$8.GND@11, U$8.GND@12, U$8.GND@13, U$8.GND@14, U$8.GND@15, U$8.GND@16, U$8.GND@2, U$8.GND@3, U$8.GND@4, U$8.GND@5, U$8.GND@6, U$8.GND@7, U$8.GND@8, U$8.GND@9; no longer U1.4
- net GND_CS: now also C_CLK_BYP.2, C_DDS_BYP3.2, C_DDS_BYP4.2, LED1.C, R_H3.1, TP_GND.TP; no longer RN1.5
- net GND_CS1: now also C_CLK_BYP1.2, C_DDS_BYP5.2, C_DDS_BYP6.2, C_DDS_BYP7.2, C_DDS_BYP8.2, LED2.C, R_H1.1, TP_GND1.TP; no longer C_DDS_BYP3.2, C_DDS_BYP4.2, RN2.5
- net GND_CS2: now also C_CLK_BYP2.2, C_DDS_BYP10.2, C_DDS_BYP11.2, C_DDS_BYP12.2, C_DDS_BYP9.2, LED3.C, R_H2.1, TP_GND2.TP; no longer C_DDS_BYP5.2, C_DDS_BYP6.2, RN3.5
- net IOUT: now also S2.2; no longer RN1.1, RN1.2
- net IOUT1: now also S4.2; no longer RN2.1, RN2.2
- net IOUT2: now also S6.2; no longer RN3.1, RN3.2
- net N$26: now also R_H1A1.2, R_H2A1.1, S4.3; no longer OPAMP2.2, RN3.3, RN3.4
- net N$27: now also R_H2B1.2, S4.4; no longer OPAMP2.1, RN3.6, RN3.7
- net N$3: now also S1.2@1, S1.2@2, U$1.RUN; no longer OPAMP.2, RN1.3, RN1.4
- net N$7: now also R_H2A.2, S2.6; no longer OPAMP.1, RN1.6, RN1.7
- net SCLK_IN: now also DIGITAL_ISO2.5, DIGITAL_ISO3.5, DIGITAL_ISO4.5, DIGITAL_ISO5.5, DIGITAL_ISO6.5, DIGITAL_ISO7.5, DIGITAL_ISO8.5
- net SDATA_IN: now also DIGITAL_ISO2.4, DIGITAL_ISO3.4, DIGITAL_ISO4.4, DIGITAL_ISO5.4, DIGITAL_ISO6.4, DIGITAL_ISO7.4, DIGITAL_ISO8.4
- net VDD: now also C_IN3.1, C_IN4.1, C_IN5.1, C_IN6.1, C_IN7.1, S1.3, S11.3, S13.3, S15.3, S3.3, S5.3, S7.3, S9.3, U$4.VIN@1, U$4.VIN@2, U$4.VIN@3, U$4.VIN@4, U$5.VIN@1, U$5.VIN@2, U$5.VIN@3, U$5.VIN@4, U$6.VIN@1, U$6.VIN@2, U$6.VIN@3, U$6.VIN@4, U$7.VIN@1, U$7.VIN@2, U$7.VIN@3, U$7.VIN@4, U$8.VIN@1, U$8.VIN@2, U$8.VIN@3, U$8.VIN@4; no longer U$1.RUN, U$2.RUN, U$3.RUN
- net VDD_CS_ANA: now also C_DDS_BYP3.1, C_DDS_BYP4.1
- net VDD_CS_ANA1: now also C_DDS_BYP7.1, C_DDS_BYP8.1
- net VDD_CS_ANA2: now also C_DDS_BYP11.1, C_DDS_BYP12.1
- net VDD_CS_DIG: now also C_CLK_BYP.1, R_LED.2
- net VDD_CS_DIG1: now also C_CLK_BYP1.1, C_DDS_BYP5.1, C_DDS_BYP6.1, R_LED1.2; no longer C_DDS_BYP3.1, C_DDS_BYP4.1
- net VDD_CS_DIG2: now also C_CLK_BYP2.1, C_DDS_BYP10.1, C_DDS_BYP9.1, R_LED2.2; no longer C_DDS_BYP5.1, C_DDS_BYP6.1
- net V_SINE: now also R_H1A.1, R_H1B.1, TP_VSIN.TP; no longer RN1.8
- net V_SINE1: now also R_H1A1.1, R_H1B1.1, TP_VSIN1.TP; no longer RN2.8
- net V_SINE2: now also R_H1A2.1, R_H1B2.1, TP_VSIN2.TP; no longer RN3.8
Routing:
- net ARD_5V: track 153.8 -> 400.8 mm, vias 3 -> 8
- net SCLK_IN: track 119.9 -> 328.8 mm, vias 3 -> 8
- net SDATA_IN: track 117.7 -> 323.6 mm, vias 3 -> 8
- net GND: track 229.3 -> 421.3 mm, vias 19 -> 49
- net FSYNC_IN7: track 0.00 -> 106.6 mm, vias 0 -> 2
- net FSYNC_IN6: track 0.00 -> 96.2 mm, vias 0 -> 4
- net SW_DIN: track 0.00 -> 95.1 mm
- net OUT_31: track 99.7 -> 180.5 mm
- net OUT_29: track 99.7 -> 180.3 mm
- net OUT_32: track 99.7 -> 180.3 mm
- net OUT_30: track 99.7 -> 180.2 mm
- net OUT_26: track 99.7 -> 180.1 mm
- net OUT_28: track 99.7 -> 180.1 mm
- net OUT_25: track 99.7 -> 180.1 mm
- net OUT_27: track 99.7 -> 180.1 mm
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- added copper zone on layer 15, net GND_CS3
- added copper zone on layer 15, net GND_CS4
- added copper zone on layer 15, net GND_CS5
- added copper zone on layer 15, net GND_CS6
- added copper zone on layer 15, net GND_CS7
- added copper zone on layer 2, net VDD_CS_ANA3
- added copper zone on layer 2, net VDD_CS_ANA4
- added copper zone on layer 2, net VDD_CS_ANA5
- added copper zone on layer 2, net VDD_CS_ANA6
- added copper zone on layer 2, net VDD_CS_ANA7
- added copper zone on layer 2, net VDD_CS_DIG3
- added copper zone on layer 2, net VDD_CS_DIG4
- added copper zone on layer 2, net VDD_CS_DIG5
- added copper zone on layer 2, net VDD_CS_DIG6
- added copper zone on layer 2, net VDD_CS_DIG7
- removed copper zone on layer 15, net S$1
- removed copper zone on layer 2, net X
Other:
- board size 123.3 x 113.5 mm -> 145.8 x 195.3 mm
- board text added: "1"
- board text added: "10"
- board text added: "11"
- board text added: "12"
- board text added: "13"
- board text added: "14"
- board text added: "15"
- board text added: "16"
- board text added: "17"
- board text added: "18"
- board text added: "19"
- board text added: "2"
- board text added: "20"
- board text added: "200uA"
- board text added: "21"
- board text added: "22"
- board text added: "23"
- board text added: "24"
- board text added: "25"
- board text added: "26"
- board text added: "27"
- board text added: "28"
- board text added: "29"
- board text added: "3"
- board text added: "30"
- board text added: "31"
- board text added: "32"
- board text added: "4"
- board text added: "5"
- board text added: "6"
- board text added: "60uA"
- board text added: "7"
- board text added: "8"
- board text added: "9"
- board text added: "ARD_5V"
- board text added: "Amplitude"
- board text added: "FS SD SC"
- board text added: "FSYNC_ARD"
- board text added: "GND"
- board text added: "GND PWR"
- board text added: "GND Vsin"
- board text added: "I+ GND"
- board text added: "Inner 1 Layer"
- board text added: "Inner 2 Layer"
- board text added: "On/Off"
- board text added: "PWR GND"
- board text added: "SCLK_IN"
- board text added: "SDATA_IN"
- board text added: "SW_CLK"
- board text added: "SW_DIN"
- board text added: "SW_SCLK"
- board text added: "SW_~RESET"
- board text added: "SW_~SYNC"
- board text added: "Top Layer"
- board text added: "UCL Parallel CS V1 - T. Dowrick November 2015"
- board text added: "V_AN"
- board text added: "V_DIG"
- board text removed: "Bottom Solder Resist"
- board text removed: "Inner1"
- board text removed: "Inner2"
- board text removed: "Top Solder Resist"
- board text removed: "Top layer"
