File: schematics/Full Board Prototype/Parallel CS Prototype V2 pick & place ident.brd (EAGLE design)
At the start: 145.8 x 195.3 mm, 334 parts, among them U1 ADG714BRUZ, X2 CTR_ARD, X4 DSUB _T, X5 DSUB_B

Commit message: Final Pick & Place Data, Ident Layers, for Assembly
Parts:
- removed I_OUT, I_OUT1, I_OUT2, I_OUT3, I_OUT4, I_OUT5, I_OUT6, I_OUT7: 332-02, con-garry:332-02
- removed JP1, JP10, JP11, JP12, JP13, JP14, JP15, JP16, JP17, JP18, JP19, JP2, JP20, JP21, JP22, JP23, JP24, JP25, JP26, JP27, JP28, JP29, JP3, JP30, JP31, JP32, JP4, JP5, JP6, JP7, JP8, JP9: (no value), SwitchBoard:1X01
- removed JP33: PWR, pinhead:1X02
- removed JP34: (no value), SwitchBoard:1X02
- removed S10, S12, S14, S16, S2, S4, S6, S8: TL46WOMULTICOMP_2MD, switch:TL4XPO
- removed TP_GND, TP_GND1, TP_GND2, TP_GND3, TP_GND4, TP_GND5, TP_GND6, TP_GND7, TP_VSIN, TP_VSIN1, TP_VSIN2, TP_VSIN3, TP_VSIN4, TP_VSIN5, TP_VSIN6, TP_VSIN7: PTR1PAD1-13, testpad:P1-13
- removed X2: CTR_ARD, con-subd:F09HP
- removed X4: DSUB _T, con-subd:F37HP
- removed X5: DSUB_B, con-subd:M37HP
Connections:
- removed net OUT_1: JP1.1, X4.1, X5.1
- removed net OUT_10: JP10.1, X4.10, X5.10
- removed net OUT_11: JP11.1, X4.11, X5.11
- removed net OUT_12: JP12.1, X4.12, X5.12
- removed net OUT_13: JP13.1, X4.13, X5.13
- removed net OUT_14: JP14.1, X4.14, X5.14
- removed net OUT_15: JP15.1, X4.15, X5.15
- removed net OUT_16: JP16.1, X4.16, X5.16
- removed net OUT_17: JP17.1, X4.17, X5.17
- removed net OUT_18: JP18.1, X4.18, X5.18
- removed net OUT_19: JP19.1, X4.19, X5.19
- removed net OUT_2: JP2.1, X4.2, X5.2
- removed net OUT_20: JP20.1, X4.20, X5.20
- removed net OUT_21: JP21.1, X4.21, X5.21
- removed net OUT_22: JP22.1, X4.22, X5.22
- removed net OUT_23: JP23.1, X4.23, X5.23
- removed net OUT_24: JP24.1, X4.24, X5.24
- removed net OUT_25: JP25.1, X4.25, X5.25
- removed net OUT_26: JP26.1, X4.26, X5.26
- removed net OUT_27: JP27.1, X4.27, X5.27
- removed net OUT_28: JP28.1, X4.28, X5.28
- removed net OUT_29: JP29.1, X4.29, X5.29
- removed net OUT_3: JP3.1, X4.3, X5.3
- removed net OUT_30: JP30.1, X4.30, X5.30
- removed net OUT_31: JP31.1, X4.31, X5.31
- removed net OUT_32: JP32.1, X4.32, X5.32
- removed net OUT_33: X4.33, X5.33
- removed net OUT_34: X4.34, X5.34
- removed net OUT_35: X4.35, X5.35
- removed net OUT_36: X4.36, X5.36
- removed net OUT_37: X4.37, X5.37
- removed net OUT_4: JP4.1, X4.4, X5.4
- removed net OUT_5: JP5.1, X4.5, X5.5
- removed net OUT_6: JP6.1, X4.6, X5.6
- removed net OUT_7: JP7.1, X4.7, X5.7
- removed net OUT_8: JP8.1, X4.8, X5.8
- removed net OUT_9: JP9.1, X4.9, X5.9
- net ARD_5V: no longer X2.4
- net FSYNC_ARD: no longer X2.9
- net GND: no longer JP33.1, JP34.2, X2.6
- net GND_CS: no longer I_OUT.2, TP_GND.TP
- net GND_CS1: no longer I_OUT1.2, TP_GND1.TP
- net GND_CS2: no longer I_OUT2.2, TP_GND2.TP
- net GND_CS3: no longer I_OUT3.2, TP_GND3.TP
- net GND_CS4: no longer I_OUT4.2, TP_GND4.TP
- net GND_CS5: no longer I_OUT5.2, TP_GND5.TP
- net GND_CS6: no longer I_OUT6.2, TP_GND6.TP
- net GND_CS7: no longer I_OUT7.2, TP_GND7.TP
- net IOUT: no longer I_OUT.1, S2.2
- net IOUT1: no longer I_OUT1.1, S4.2
- net IOUT2: no longer I_OUT2.1, S6.2
- net IOUT3: no longer I_OUT3.1, S8.2
- net IOUT4: no longer I_OUT4.1, S10.2
- net IOUT5: no longer I_OUT5.1, S12.2
- net IOUT6: no longer I_OUT6.1, S14.2
- net IOUT7: no longer I_OUT7.1, S16.2
- net N$100: no longer S16.1
- net N$103: no longer S16.6
- net N$104: no longer S16.3
- net N$105: no longer S16.4
- net N$12: no longer S2.1
- net N$15: no longer S2.3
- net N$22: no longer S4.1
- net N$25: no longer S4.6
- net N$26: no longer S4.3
- net N$27: no longer S4.4
- net N$35: no longer S6.1
- net N$38: no longer S6.6
- net N$39: no longer S6.3
- net N$40: no longer S6.4
- net N$48: no longer S8.1
- net N$51: no longer S8.6
- net N$52: no longer S8.3
- net N$53: no longer S8.4
- net N$61: no longer S10.1
- net N$64: no longer S10.6
- net N$65: no longer S10.3
- net N$66: no longer S10.4
- net N$7: no longer S2.6
- net N$74: no longer S12.1
- net N$77: no longer S12.6
- net N$78: no longer S12.3
- net N$79: no longer S12.4
- net N$87: no longer S14.1
- net N$9: no longer S2.4
- net N$90: no longer S14.6
- net N$91: no longer S14.3
- net N$92: no longer S14.4
- net OP_OUTA: no longer S2.5
- net OP_OUTA1: no longer S4.5
- net OP_OUTA2: no longer S6.5
- net OP_OUTA3: no longer S8.5
- net OP_OUTA4: no longer S10.5
- net OP_OUTA5: no longer S12.5
- net OP_OUTA6: no longer S14.5
- net OP_OUTA7: no longer S16.5
- net SCLK_IN: no longer X2.2
- net SDATA_IN: no longer X2.3
- net SW_DIN: no longer X2.5
- net SW_SCLK: no longer X2.1
- net SW_~RESET: no longer X2.8
- net SW_~SYNC: no longer X2.7
- net VDD: no longer JP33.2, JP34.1
- net V_SINE: no longer TP_VSIN.TP
- net V_SINE1: no longer TP_VSIN1.TP
- net V_SINE2: no longer TP_VSIN2.TP
- net V_SINE3: no longer TP_VSIN3.TP
- net V_SINE4: no longer TP_VSIN4.TP
- net V_SINE5: no longer TP_VSIN5.TP
- net V_SINE6: no longer TP_VSIN6.TP
- net V_SINE7: no longer TP_VSIN7.TP
Routing:
- net OUT_31: track 180.5 -> 0.00 mm
- net OUT_29: track 180.3 -> 0.00 mm
- net OUT_32: track 180.3 -> 0.00 mm
- net OUT_30: track 180.2 -> 0.00 mm
- net OUT_26: track 180.1 -> 0.00 mm
- net OUT_28: track 180.1 -> 0.00 mm
- net OUT_25: track 180.1 -> 0.00 mm
- net OUT_27: track 180.1 -> 0.00 mm
- net OUT_21: track 180.0 -> 0.00 mm
- net OUT_23: track 179.7 -> 0.00 mm
- net OUT_24: track 179.7 -> 0.00 mm
- net OUT_22: track 179.7 -> 0.00 mm
- net OUT_20: track 179.4 -> 0.00 mm
- net OUT_35: track 178.4 -> 0.00 mm
- net OUT_37: track 178.4 -> 0.00 mm
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Other:
- board text added: "S1"
- board text added: "S11"
- board text added: "S13"
- board text added: "S15"
- board text added: "S3"
- board text added: "S5"
- board text added: "S7"
- board text added: "S9"
- board text removed: "1"
- board text removed: "10"
- board text removed: "11"
- board text removed: "12"
- board text removed: "13"
- board text removed: "14"
- board text removed: "15"
- board text removed: "16"
- board text removed: "17"
- board text removed: "18"
- board text removed: "19"
- board text removed: "2"
- board text removed: "20"
- board text removed: "200uA"
- board text removed: "21"
- board text removed: "22"
- board text removed: "23"
- board text removed: "24"
- board text removed: "25"
- board text removed: "26"
- board text removed: "27"
- board text removed: "28"
- board text removed: "29"
- board text removed: "3"
- board text removed: "30"
- board text removed: "31"
- board text removed: "32"
- board text removed: "4"
- board text removed: "5"
- board text removed: "6"
- board text removed: "60uA"
- board text removed: "7"
- board text removed: "8"
- board text removed: "9"
- board text removed: "ARD_5V"
- board text removed: "Amplitude"
- board text removed: "FS SD SC"
- board text removed: "FSYNC_ARD"
- board text removed: "GND"
- board text removed: "GND PWR"
- board text removed: "GND Vsin"
- board text removed: "I+ GND"
- board text removed: "On/Off"
- board text removed: "PWR GND"
- board text removed: "SCLK_IN"
- board text removed: "SDATA_IN"
- board text removed: "SW_CLK"
- board text removed: "SW_DIN"
- board text removed: "SW_SCLK"
- board text removed: "SW_~RESET"
- board text removed: "SW_~SYNC"
- board text removed: "UCL Parallel CS V1 - T. Dowrick November 2015"
- board text removed: "V_AN"
- board text removed: "V_DIG"
