File: schematics/Rev.Dec.2016/Parallel CS V5 repeated.brd (EAGLE design)
At the start: 99.9 x 150.1 mm, 290 parts, among them U1 ADG714BRUZ

Commit message: V5.1 Board - fixing error with footprint of op-amp
Parts:
- moved LED_VSS 6.00 mm to (72.0, 70.5)
- moved R_VSS_LED 5.50 mm to (72.0, 64.5)
Routing:
- net VSS: track 133.1 -> 127.8 mm
- net S$2: track 0.00 -> 5.00 mm
- net S$1: track 0.00 -> 5.00 mm
- net GND: track 346.6 -> 341.6 mm
- net N$22: track 5.54 -> 6.10 mm
Changed lines of the file:
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@@
 <attribute name="VALUE" x="74" y="87" size="1.27" layer="27" rot="R180"/>
 </element>
-<element name="LED_VSS" library="led" package="SML0805" value="" x="72" y="64.5" smashed="yes" rot="R180">
-<attribute name="NAME" x="73.5" y="63.5" size="1.27" layer="25" rot="R180"/>
-<attribute name="VALUE" x="73.5" y="66.5" size="1.27" layer="27" rot="R180"/>
+<element name="LED_VSS" library="led" package="SML0805" value="" x="72" y="70.5" smashed="yes" rot="R180">
+<attribute name="NAME" x="73.5" y="69.5" size="1.27" layer="25" rot="R180"/>
+<attribute name="VALUE" x="73.5" y="72.5" size="1.27" layer="27" rot="R180"/>
 </element>
 <element name="R_VDD_LED" library="resistor" package="M0805" value="1k" x="72" y="79" smashed="yes">
@@
 <attribute name="VALUE" x="70.73" y="76.46" size="1.27" layer="27"/>
 </element>
-<element name="R_VSS_LED" library="resistor" package="M0805" value="1k" x="72" y="70" smashed="yes">
-<attribute name="NAME" x="70.73" y="71.27" size="1.27" layer="25"/>
-<attribute name="VALUE" x="70.73" y="67.46" size="1.27" layer="27"/>
+<element name="R_VSS_LED" library="resistor" package="M0805" value="1k" x="72" y="64.5" smashed="yes">
+<attribute name="NAME" x="70.73" y="65.77" size="1.27" layer="25"/>
+<attribute name="VALUE" x="70.73" y="61.96" size="1.27" layer="27"/>
 </element>
 <element name="U$1" library="Arduino-clone" package="NANO" value="NANO" x="28" y="76.5" smashed="yes" rot="R90"/>
@@
 <wire x1="86.5" y1="144.26" x2="86.76" y2="144" width="0.254" layer="1"/>
 <wire x1="86.76" y1="144" x2="88.5" y2="144" width="0.254" layer="1"/>
-<wire x1="73.05" y1="64.5" x2="73.0528" y2="64.5028" width="0.254" layer="1"/>
-<wire x1="73.0528" y1="64.5028" x2="78.0108" y2="64.5028" width="0.254" layer="1"/>
 <wire x1="73.55" y1="85" x2="73.5528" y2="84.9972" width="0.254" layer="1"/>
 <wire x1="73.5528" y1="84.9972" x2="78.0108" y2="84.9972" width="0.254" layer="1"/>
@@
 <wire x1="86.5" y1="15.26" x2="86.76" y2="15" width="0.254" layer="1"/>
 <wire x1="86.76" y1="15" x2="88.5" y2="15" width="0.254" layer="1"/>
+<wire x1="78.0108" y1="64.5028" x2="73.05" y2="70.5" width="0" layer="19" extent="1-1"/>
 </signal>
 <signal name="FSYNC_CS8">
@@
 <via x="84.5" y="139" extent="1-16" drill="0.6" shape="square"/>
 <wire x1="84.5" y1="139" x2="84.5" y2="139.5" width="0.254" layer="16"/>
-<wire x1="72.95" y1="70" x2="73.4472" y2="70.4972" width="0.254" layer="1"/>
-<wire x1="73.4472" y1="70.4972" x2="78.0108" y2="70.4972" width="0.254" layer="1"/>
 <contactref element="OP_S2D1" pad="4"/>
 <contactref element="OP_GAIN1" pad="4"/>
@@
 <via x="84.5" y="30" extent="1-16" drill="0.6" shape="square"/>
 <wire x1="84.5" y1="30" x2="84.5" y2="30.5" width="0.254" layer="16"/>
+<wire x1="78.0108" y1="70.4972" x2="72.95" y2="64.5" width="0" layer="19" extent="1-1"/>
 </signal>
 <signal name="DDS_SCLK_5V">
@@
 <contactref element="R_VSS_LED" pad="1"/>
 <contactref element="LED_VSS" pad="A"/>
-<wire x1="71.05" y1="70" x2="70.95" y2="69.9" width="0.254" layer="1"/>
-<wire x1="70.95" y1="69.9" x2="70.95" y2="64.5" width="0.254" layer="1"/>
+<wire x1="71.05" y1="64.5" x2="70.95" y2="64.5" width="0.4064" layer="1"/>
+<wire x1="70.95" y1="64.5" x2="70.95" y2="70.5" width="0.4064" layer="1"/>
 </signal>
 <signal name="N$23">
@@
 <wire x1="77.1752" y1="16.9652" x2="79.7902" y2="16.9652" width="0.254" layer="1"/>
 </signal>
+<signal name="S$1">
+<wire x1="73" y1="64.5" x2="78" y2="64.5" width="0.4064" layer="1"/>
+</signal>
+<signal name="S$2">
+<wire x1="73" y1="70.5" x2="78" y2="70.5" width="0.4064" layer="1"/>
+</signal>
 </signals>
