File: schematics/Rev.Dec.2016/Parallel CS V5.brd (EAGLE design)
At the start: 99.9 x 150.1 mm, 72 parts, among them U1 ADG714BRUZ, X2 CTR_ARD

Commit message: Changed power connecters, split output stage op amps into 2 separate ICs for medical safety regs
Parts:
- removed X2: CTR_ARD, con-subd:F09HP
- added OP_HOWL1: RC4560SOP65, RC4560:SOP65P490X109-8N
- added U$1: NANO, Arduino-clone:NANO
- OP_GAIN, OP_HOWL, OP_S2D: value RC4560 -> RC4560SOP65; device RC4560:DIL08 -> RC4560:SOP65P490X109-8N
- R_HOWB3: value 1k -> 100k
- R_HOWB4: value 100k -> 1k
- renumbered R_HOW1 to R_HOWB2, R_HOW10 to R_HOWA3, R_HOW2 to R_HOWA1, R_HOW3 to R_HOWB1, R_HOW4 to R_HOWA2, R_HOW5 to R_HOWB4, R_HOW6 to R_HOWB5, R_HOW7 to R_HOWA4, R_HOW8 to R_HOWA5, R_HOW9 to R_HOWB3
Connections:
- removed net DDS_SDATA_5V: R3.2, X2.2
- removed net N$16: OP_HOWL.1, R_HOWB4.2, R_HOWB5.2
- new net N$23: R3.2, U$1.D11
- new net N$24: OP_HOWL1.1, R_HOWB4.2, R_HOWB5.2
- new net V-: OP_HOWL.4
- net DDS_SCLK_5V: now also U$1.D13; no longer X2.3
- net FSYNC_IN_5V: now also U$1.D5; no longer X2.9
- net GND: now also U$1.GND; no longer X2.6
- net N$11: now also OP_HOWL1.3; no longer OP_HOWL.3
- net N$12: now also OP_HOWL1.2; no longer OP_HOWL.2
- net SW_DIN_5V: now also U$1.D4; no longer X2.5
- net SW_SCLK_5V: now also U$1.D9; no longer X2.1
- net SW_~RESET_5V: now also U$1.D3; no longer X2.8
- net SW_~SYNC_5V: now also U$1.D2; no longer X2.7
- net VDD: now also OP_HOWL1.8
- net VSS: now also OP_HOWL1.4; no longer OP_HOWL.4
Routing:
- net N$8: track 38.9 -> 12.2 mm, vias 1 -> 0
- net GND: track 82.4 -> 63.1 mm, vias 17 -> 13
- net VDD: track 43.3 -> 59.5 mm
- net N$12: track 12.4 -> 0.07 mm
- net N$7: track 25.6 -> 35.5 mm
- net N$3: track 38.2 -> 47.1 mm
- net N$16: track 6.94 -> 0.00 mm
- net FSYNC_IN_5V: track 7.19 -> 0.84 mm
- net DDS_SCLK_5V: track 6.23 -> 0.00 mm
- net N$10: track 19.2 -> 25.0 mm
- net N$5: track 24.2 -> 28.4 mm
- net N$9: track 7.10 -> 11.1 mm
- net VSIN: track 26.0 -> 30.0 mm
- net N$11: track 25.1 -> 28.6 mm
- net N$20: track 27.9 -> 31.4 mm
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
Commit message: Changed FSYNC pull up resistor to pull down
Parts:
- R12, R13, R14, R2, R4, R6, R8: device resistor:R0603 -> resistor:R0805
Connections:
- net GND: now also R_PULLUP.1
- net VDD: no longer R_PULLUP.1
Routing:
- net VDD: track 59.5 -> 56.5 mm, vias 5 -> 4

Commit message: Changes complete - PCB layout ready for tiling
Parts:
- removed OP_HOWL, OP_HOWL1: RC4560SOP65, RC4560:SOP65P490X109-8N
- removed R14: 20k, resistor:R0805
- added C_OPD1, C_OPD2: 0.1u, resistor:C0805
- added OP_HOWLA, OP_HOWLB: RC4560SOP65, RC4560:SOP65P490X109-8N
- added R_GAIN2: 1, rcl:R0805
- R_HOWA5, R_HOWB4: value 1k -> 10k
- R_PULLDOWN: value 10k -> 20k
- R_SET: device resistor:R0603 -> resistor:R0805
- moved R_VDD_LED 158.5 mm to (72.0, 72.0)
- moved LED_VDD 157.0 mm to (72.5, 78.0), turned to 180 degrees
- moved R_VSS_LED 154.2 mm to (72.0, 63.0)
- moved LED_VSS 143.0 mm to (72.0, 57.5), turned to 180 degrees
- moved S1 141.4 mm to (80.5, 75.0), turned to 90 degrees
- moved S2 138.3 mm to (80.5, 60.5), turned to 90 degrees
- moved U$1 136.9 mm to (28.0, 69.5), turned to 90 degrees
- moved TP_SDATA 55.8 mm to (4.11, 78.4)
- moved TP_SCLK 24.5 mm to (7.61, 50.5)
- moved R1 22.2 mm to (3.68, 55.1)
- moved R12 22.0 mm to (34.5, 78.5)
- moved R9 22.0 mm to (29.5, 78.5)
- moved TP_GND 21.8 mm to (89.8, 84.1)
- moved R2 20.8 mm to (9.23, 55.1), turned to 180 degrees
- moved R_HOWA3 20.0 mm to (72.7, 135.7), turned to 0 degrees
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- renumbered R_PULLUP to R_PULLDOWN
Connections:
- removed net V-: OP_HOWL.4
- new net N$16: JP+.1, S1.4
- net FSYNC_IN: no longer R14.2
- net GND: now also C_OPD1.2, C_OPD2.2; no longer R14.1
- net N$11: now also OP_HOWLB.3; no longer OP_HOWL1.3
- net N$12: now also OP_HOWLB.2; no longer OP_HOWL1.2
- net N$17: now also OP_HOWLA.7; no longer OP_HOWL.7
- net N$20: now also OP_HOWLA.6; no longer OP_HOWL.6
- net N$24: now also OP_HOWLB.1; no longer OP_HOWL1.1
- net N$3: now also R_GAIN2.1
- net N$5: now also R_GAIN2.2
- net N$7: now also OP_HOWLA.5; no longer OP_HOWL.5
- net VDD: now also C_OPD1.1, OP_HOWLA.8, OP_HOWLB.8; no longer OP_HOWL.8, OP_HOWL1.8
- net VSS: now also C_OPD2.1, OP_HOWLA.4, OP_HOWLB.4; no longer OP_HOWL1.4
Routing:
- net CLK_OUT: track 61.2 -> 2.71 mm, vias 1 -> 0
- net GND: track 63.0 -> 94.0 mm, vias 13 -> 20
- net SW_~SYNC: track 48.0 -> 22.8 mm
- net N$8: track 12.2 -> 34.1 mm, vias 0 -> 1
- net N$7: track 35.5 -> 16.3 mm, vias 1 -> 2
- net N$14: track 10.5 -> 28.4 mm
- net N$20: track 31.4 -> 14.0 mm
- net N$24: track 0.00 -> 17.3 mm
- net N$17: track 3.12 -> 18.1 mm
- net SW_~RESET_5V: track 18.4 -> 3.97 mm
- net N$3: track 47.1 -> 33.5 mm
- net N$12: track 0.07 -> 13.6 mm
- net SW_~SYNC_5V: track 18.0 -> 4.67 mm
- net VSS: track 13.7 -> 26.6 mm, vias 1 -> 5
- net N$11: track 28.6 -> 15.9 mm, vias 1 -> 2
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Other:
- board text added: "DDS Decoup"
- board text added: "DDS OUT"
- board text added: "Vdiff A"
- board text added: "Vdiff B"

Commit message: V5.1 Board - fixing error with footprint of op-amp
Parts:
- R11: value 10k -> 1.5k
- moved TP_GND 31.4 mm to (58.8, 79.1)
- moved TP_VDD 17.7 mm to (53.4, 79.1)
- moved TP_VSS 15.9 mm to (64.0, 79.1)
Connections:
- removed net FSYNC: DDS.8, R_PULLDOWN.2, TP_FSYNC.TP
- net FSYNC_CS1: now also DDS.8, R_PULLDOWN.2, TP_FSYNC.TP
Routing:
- net N$18: track 0.00 -> 11.7 mm
- net N$16: track 0.00 -> 11.0 mm
- net N$19: track 0.00 -> 10.0 mm
- net N$15: track 0.00 -> 9.66 mm
- net FSYNC_CS1: track 0.00 -> 8.73 mm
- net FSYNC: track 8.73 -> 0.00 mm
- net VDD: track 55.1 -> 57.2 mm
Other:
- board text added: "DDS SDATA"
- board text added: "FSYNC"
- board text added: "GND"
- board text added: "Master Clock"
- board text added: "VDD"
- board text added: "VSS"
Changed lines of the file:
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@@
 <text x="60" y="139.5" size="0.8128" layer="27">Vdiff A</text>
 <text x="60" y="134" size="0.8128" layer="27">Vdiff B</text>
+<text x="52" y="80.5" size="0.8128" layer="112">VDD</text>
+<text x="63" y="80.5" size="0.8128" layer="112">VSS</text>
+<text x="57.5" y="77" size="0.8128" layer="112">GND</text>
+<text x="53" y="63" size="0.8128" layer="112">Master
+Clock</text>
+<text x="5.5" y="78.5" size="0.8128" layer="112">DDS
+SDATA</text>
+<text x="20" y="142" size="0.8128" layer="112">FSYNC</text>
 </plain>
 <attributes>
@@
 <attribute name="VALUE" x="18.97" y="141.43" size="0.0254" layer="27"/>
 </element>
-<element name="TP_GND" library="testpad" package="P1-13" value="PTR1PAD1-13" x="89.79" y="84.09" smashed="yes">
-<attribute name="TP_SIGNAL_NAME" value="" x="88.52" y="81.55" size="1" layer="37"/>
-<attribute name="NAME" x="88.774" y="85.36" size="1.27" layer="25" ratio="10"/>
-<attribute name="VALUE" x="89.79" y="84.09" size="0.0254" layer="27"/>
+<element name="TP_GND" library="testpad" package="P1-13" value="PTR1PAD1-13" x="58.79" y="79.09" smashed="yes">
+<attribute name="TP_SIGNAL_NAME" value="" x="57.52" y="76.55" size="1" layer="37"/>
+<attribute name="NAME" x="57.774" y="80.36" size="1.27" layer="25" ratio="10"/>
+<attribute name="VALUE" x="58.79" y="79.09" size="0.0254" layer="27"/>
 </element>
 <element name="TP_MCLK" library="testpad" package="P1-13" value="PTR1PAD1-13" x="54.43" y="66.51" smashed="yes">
@@
 <attribute name="VALUE" x="4.11" y="78.43" size="0.0254" layer="27"/>
 </element>
-<element name="TP_VDD" library="testpad" package="P1-13" value="PTR1PAD1-13" x="70.4" y="84.09" smashed="yes">
-<attribute name="TP_SIGNAL_NAME" value="" x="69.13" y="81.55" size="1" layer="37"/>
-<attribute name="NAME" x="69.384" y="85.36" size="1.27" layer="25" ratio="10"/>
-<attribute name="VALUE" x="70.4" y="84.09" size="0.0254" layer="27"/>
+<element name="TP_VDD" library="testpad" package="P1-13" value="PTR1PAD1-13" x="53.4" y="79.09" smashed="yes">
+<attribute name="TP_SIGNAL_NAME" value="" x="52.13" y="76.55" size="1" layer="37"/>
+<attribute name="NAME" x="52.384" y="80.36" size="1.27" layer="25" ratio="10"/>
+<attribute name="VALUE" x="48.9" y="77.09" size="0.0254" layer="27"/>
 </element>
 <element name="TP_VSIN" library="testpad" package="P1-13" value="PTR1PAD1-13" x="12.18" y="145.59" smashed="yes">
@@
 <attribute name="VALUE" x="61.59" y="136.51" size="0.0254" layer="27"/>
 </element>
-<element name="TP_VSS" library="testpad" package="P1-13" value="PTR1PAD1-13" x="78.01" y="86.59" smashed="yes">
-<attribute name="TP_SIGNAL_NAME" value="" x="76.74" y="84.05" size="1" layer="37"/>
-<attribute name="NAME" x="76.994" y="87.86" size="1.27" layer="25" ratio="10"/>
-<attribute name="VALUE" x="78.01" y="86.59" size="0.0254" layer="27"/>
+<element name="TP_VSS" library="testpad" package="P1-13" value="PTR1PAD1-13" x="64.01" y="79.09" smashed="yes">
+<attribute name="TP_SIGNAL_NAME" value="" x="62.74" y="76.55" size="1" layer="37"/>
+<attribute name="NAME" x="62.994" y="80.36" size="1.27" layer="25" ratio="10"/>
+<attribute name="VALUE" x="64.01" y="79.09" size="0.0254" layer="27"/>
 </element>
 <element name="U1" library="SwitchBoard" package="SOP65P640X120-24N" value="ADG714BRUZ" x="46" y="68.89" smashed="yes">
@@
 <attribute name="VALUE" x="22.46" y="71.135" size="1.27" layer="27" rot="R270"/>
 </element>
-<element name="R11" library="resistor" package="R0805" value="10k" x="23" y="78" smashed="yes">
+<element name="R11" library="resistor" package="R0805" value="1.5k" x="23" y="78" smashed="yes">
 <attribute name="NAME" x="22.365" y="79.27" size="1.27" layer="25"/>
 <attribute name="VALUE" x="21.365" y="79.46" size="1.27" layer="27"/>
@@
 <element name="S1" library="switch-misc" package="PVA1F" value="PVA1F" x="80.5" y="75" smashed="yes" rot="R90">
 <attribute name="NAME" x="81.135" y="81.985" size="1.27" layer="25" ratio="10" rot="R90"/>
-<attribute name="VALUE" x="83.04" y="81.985" size="1.27" layer="27" ratio="10" rot="R90"/>
 </element>
 <element name="S2" library="switch-misc" package="PVA1F" value="PVA1F" x="80.5" y="60.5" smashed="yes" rot="R90">
 <attribute name="NAME" x="81.135" y="67.485" size="1.27" layer="25" ratio="10" rot="R90"/>
-<attribute name="VALUE" x="83.04" y="67.485" size="1.27" layer="27" ratio="10" rot="R90"/>
 </element>
 <element name="LED_VDD" library="led" package="SML0805" value="" x="72.5" y="78" smashed="yes" rot="R180">
@@
 <wire x1="88.5" y1="146" x2="89" y2="146" width="0.254" layer="2"/>
 <wire x1="84.2098" y1="145.9652" x2="84.2446" y2="146" width="0.254" layer="1"/>
-<wire x1="84.2446" y1="146" x2="88.5" y2="146" width="0.254" layer="1"/>
 <wire x1="72.95" y1="72" x2="72.9528" y2="72.0028" width="0.254" layer="1"/>
 <wire x1="72.9528" y1="72.0028" x2="78.0108" y2="72.0028" width="0.254" layer="1"/>
-<wire x1="88.5" y1="146" x2="86.5" y2="146.16" width="0" layer="19" extent="1-2"/>
+<wire x1="86.5" y1="146.16" x2="86.66" y2="146" width="0.3048" layer="1"/>
+<wire x1="86.66" y1="146" x2="88.5" y2="146" width="0.3048" layer="1"/>
+<wire x1="88.5" y1="146" x2="88.4652" y2="145.9652" width="0.3048" layer="1"/>
+<wire x1="88.4652" y1="145.9652" x2="84.2098" y2="145.9652" width="0.3048" layer="1"/>
 </signal>
 <signal name="SW_DIN">
@@
 <signal name="FSYNC_CS1">
 <contactref element="U1" pad="6"/>
+<contactref element="DDS" pad="8"/>
+<contactref element="TP_FSYNC" pad="TP"/>
+<contactref element="R_PULLDOWN" pad="2"/>
+<wire x1="19.09" y1="137.13" x2="18.22" y2="138" width="0.254" layer="1"/>
+<wire x1="18.22" y1="138" x2="17" y2="138" width="0.254" layer="1"/>
+<wire x1="17" y1="138" x2="16.25" y2="138.75" width="0.254" layer="1"/>
+<wire x1="16.25" y1="138.75" x2="15.3852" y2="138.75" width="0.254" layer="1"/>
+<wire x1="18.97" y1="141.43" x2="19.09" y2="141.31" width="0.254" layer="1"/>
+<wire x1="19.09" y1="141.31" x2="19.09" y2="137.13" width="0.254" layer="1"/>
+<wire x1="43.1806" y1="69.2202" x2="19.09" y2="137.13" width="0" layer="19" extent="1-1"/>
 </signal>
 <signal name="FSYNC_CS3">
@@
 <wire x1="1.33" y1="55.15" x2="1.33" y2="59.34" width="0.4064" layer="1"/>
 </signal>
-<signal name="FSYNC">
-<contactref element="DDS" pad="8"/>
-<contactref element="TP_FSYNC" pad="TP"/>
-<contactref element="R_PULLDOWN" pad="2"/>
-<wire x1="19.09" y1="137.13" x2="18.22" y2="138" width="0.254" layer="1"/>
-<wire x1="18.22" y1="138" x2="17" y2="138" width="0.254" layer="1"/>
-<wire x1="17" y1="138" x2="16.25" y2="138.75" width="0.254" layer="1"/>
-<wire x1="16.25" y1="138.75" x2="15.3852" y2="138.75" width="0.254" layer="1"/>
-<wire x1="18.97" y1="141.43" x2="19.09" y2="141.31" width="0.254" layer="1"/>
-<wire x1="19.09" y1="141.31" x2="19.09" y2="137.13" width="0.254" layer="1"/>
-</signal>
 <signal name="N$1">
 <contactref element="DDS" pad="3"/>
@@
 <contactref element="JP+" pad="2"/>
 <contactref element="S1" pad="2"/>
-<wire x1="82.9892" y1="72.0028" x2="92.48" y2="72.4" width="0" layer="19" extent="1-1"/>
+<wire x1="82.9892" y1="72.0028" x2="83.3864" y2="72.4" width="0.6096" layer="1"/>
+<wire x1="83.3864" y1="72.4" x2="92.48" y2="72.4" width="0.6096" layer="1"/>
 </signal>
 <signal name="N$18">
 <contactref element="JP-" pad="2"/>
 <contactref element="S2" pad="2"/>
-<wire x1="82.9892" y1="57.5028" x2="92.48" y2="62.75" width="0" layer="19" extent="1-1"/>
+<wire x1="82.9892" y1="57.5028" x2="88.2364" y2="62.75" width="0.6096" layer="1"/>
+<wire x1="88.2364" y1="62.75" x2="92.48" y2="62.75" width="0.6096" layer="1"/>
 </signal>
 <signal name="N$19">
 <contactref element="JP-" pad="1"/>
 <contactref element="S2" pad="4"/>
-<wire x1="82.9892" y1="63.4972" x2="92.48" y2="64.75" width="0" layer="19" extent="1-1"/>
+<wire x1="82.9892" y1="63.4972" x2="84.242" y2="64.75" width="0.6096" layer="1"/>
+<wire x1="84.242" y1="64.75" x2="92.48" y2="64.75" width="0.6096" layer="1"/>
 </signal>
 <signal name="N$21">
@@
 <contactref element="JP+" pad="1"/>
 <contactref element="S1" pad="4"/>
-<wire x1="82.9892" y1="77.9972" x2="92.48" y2="74.4" width="0" layer="19" extent="1-1"/>
+<wire x1="82.9892" y1="77.9972" x2="86.5864" y2="74.4" width="0.6096" layer="1"/>
+<wire x1="86.5864" y1="74.4" x2="92.48" y2="74.4" width="0.6096" layer="1"/>
 </signal>
 </signals>
