File: schematics/Rev.Dec.2016/Parallel CS V5.sch (EAGLE design)
At the start: 72 parts, among them U1 ADG714BRUZ, X2 CTR_ARD

Commit message: Changed power connecters, split output stage op amps into 2 separate ICs for medical safety regs
Parts:
- removed R_HOW1, R_HOW10, R_HOW2, R_HOW3, R_HOW5, R_HOW6, R_HOW7: 100k, rcl:R-US_R0805
- removed R_HOW8, R_HOW9: 1k, rcl:R-US_R0805
- removed X2: CTR_ARD, con-subd:F09HP
- added OP_HOWL1: RC4560SOP65, RC4560:RC4560SOP65
- added R_HOWA1, R_HOWA3, R_HOWA4, R_HOWB1, R_HOWB2, R_HOWB3, R_HOWB5: 100k, rcl:R-US_R0805
- added R_HOWA5, R_HOWB4: 1k, rcl:R-US_R0805
- added U$1: NANO, Arduino-clone:NANO
- OP_GAIN, OP_HOWL, OP_S2D: value RC4560 -> RC4560SOP65; device RC4560:RC4560 -> RC4560:RC4560SOP65
- renumbered R_HOW4 to R_HOWA2
Connections:
- removed net DDS_SDATA_5V: R3.2, X2.2
- removed net N$16: OP_HOWL.OUTA, R_HOW5.2, R_HOW6.2
- new net N$23: R3.2, U$1.D11
- new net N$24: OP_HOWL1.OUTA, R_HOWB4.2, R_HOWB5.2
- net DDS_SCLK_5V: now also U$1.D13; no longer X2.3
- net FSYNC_IN_5V: now also U$1.D5; no longer X2.9
- net GND: now also U$1.GND; no longer X2.6
- net N$11: now also OP_HOWL1.POSA, R_HOWB2.1, R_HOWB3.1; no longer OP_HOWL.POSA, R_HOW1.1, R_HOW9.1
- net N$12: now also OP_HOWL1.NEGA, R_HOWB1.1, R_HOWB5.1; no longer OP_HOWL.NEGA, R_HOW3.1, R_HOW6.1
- net N$13: now also R_HOWB3.2, R_HOWB4.1; no longer R_HOW5.1, R_HOW9.2
- net N$14: now also R_HOWA3.2, R_HOWA5.2; no longer R_HOW10.2, R_HOW8.2
- net N$17: now also R_HOWA4.1, R_HOWA5.1; no longer R_HOW7.1, R_HOW8.1
- net N$20: now also R_HOWA4.2; no longer R_HOW7.2
- net N$4: now also R_HOWA1.2, R_HOWB1.2; no longer R_HOW2.2, R_HOW3.2
- net N$7: now also R_HOWA1.1, R_HOWA3.1; no longer R_HOW10.1, R_HOW2.1
- net N$8: now also R_HOWB2.2; no longer R_HOW1.2
- net SW_DIN_5V: now also U$1.D4; no longer X2.5
- net SW_SCLK_5V: now also U$1.D9; no longer X2.1
- net SW_~RESET_5V: now also U$1.D3; no longer X2.8
- net SW_~SYNC_5V: now also U$1.D2; no longer X2.7
- net VDD: now also OP_HOWL1.V+
- net VSS: now also OP_HOWL1.V-; no longer OP_HOWL.V-
Other:
- note added: "5V from Arduino needs to be convertred to ~3.3V to set the right levels for the DDS & Switch ICs, which are powered by 3.7V batteries. Hence resistor dividers."
- note added: "Arduino Socket"
- note added: "Battery Connector & Power LEDs"
- note added: "Howland Current Pump Using two separate ICs for medical safety to cover case where a single device fails."
- note added: "Switch to route FSYNC to each CS"
- note added: "Test Points"
- note removed: "Battery Connector"
- note removed: "DSUB FROM ARDUINO"
- note removed: "Howland Current Pump Can select between two outputs with different magnitudes"
- note removed: "Switch to route FSYNC, powered by Arduino"
- moved on the sheet: CLOCK, C_CLK_BYP, JP+, JP-, JP_OUT, LED_VDD, LED_VSS, OP_HOWL, R1, R10, R11, R12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

Commit message: Changed FSYNC pull up resistor to pull down
Parts:
- R12, R13, R14, R2, R4, R6, R8: device resistor:R-US_R0603 -> resistor:R-US_R0805
Connections:
- net GND: now also R_PULLUP.1
- net VDD: no longer R_PULLUP.1
Changed lines of the file:
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@@
 <part name="TP_FSYNC" library="testpad" deviceset="PTR1" device="PAD1-13" value="PTR1PAD1-13"/>
 <part name="R1" library="resistor" deviceset="R-US_" device="R0805" value="10k"/>
-<part name="R2" library="resistor" deviceset="R-US_" device="R0603" value="20k"/>
+<part name="R2" library="resistor" deviceset="R-US_" device="R0805" value="20k"/>
 <part name="R3" library="resistor" deviceset="R-US_" device="R0805" value="10k"/>
-<part name="R4" library="resistor" deviceset="R-US_" device="R0603" value="20k"/>
+<part name="R4" library="resistor" deviceset="R-US_" device="R0805" value="20k"/>
 <part name="GND3" library="supply1" deviceset="GND" device=""/>
 <part name="R_DECOUP" library="rcl" deviceset="R-US_" device="R0805" value="10k"/>
@@
 <part name="R_HOWA3" library="rcl" deviceset="R-US_" device="R0805" value="100k"/>
 <part name="R5" library="resistor" deviceset="R-US_" device="R0805" value="10k"/>
-<part name="R6" library="resistor" deviceset="R-US_" device="R0603" value="20k"/>
+<part name="R6" library="resistor" deviceset="R-US_" device="R0805" value="20k"/>
 <part name="GND4" library="supply1" deviceset="GND" device=""/>
 <part name="R7" library="resistor" deviceset="R-US_" device="R0805" value="10k"/>
-<part name="R8" library="resistor" deviceset="R-US_" device="R0603" value="20k"/>
+<part name="R8" library="resistor" deviceset="R-US_" device="R0805" value="20k"/>
 <part name="R9" library="resistor" deviceset="R-US_" device="R0805" value="10k"/>
 <part name="R10" library="resistor" deviceset="R-US_" device="R0805" value="10k"/>
 <part name="R11" library="resistor" deviceset="R-US_" device="R0805" value="10k"/>
-<part name="R12" library="resistor" deviceset="R-US_" device="R0603" value="20k"/>
-<part name="R13" library="resistor" deviceset="R-US_" device="R0603" value="20k"/>
-<part name="R14" library="resistor" deviceset="R-US_" device="R0603" value="20k"/>
+<part name="R12" library="resistor" deviceset="R-US_" device="R0805" value="20k"/>
+<part name="R13" library="resistor" deviceset="R-US_" device="R0805" value="20k"/>
+<part name="R14" library="resistor" deviceset="R-US_" device="R0805" value="20k"/>
 <part name="S1" library="switch-misc" deviceset="PVA1" device="F"/>
 <part name="S2" library="switch-misc" deviceset="PVA1" device="F"/>
@@
 <part name="GND12" library="supply1" deviceset="GND" device=""/>
 <part name="OP_HOWL1" library="RC4560" deviceset="RC4560" device="SOP65" value="RC4560SOP65"/>
+<part name="GND13" library="supply1" deviceset="GND" device=""/>
 </parts>
 <sheets>
@@
 <instance part="R_HOWA3" gate="G$1" x="114.3" y="-30.48"/>
 <instance part="OP_HOWL1" gate="RC4560" x="96.52" y="68.58"/>
+<instance part="GND13" gate="1" x="-55.88" y="55.88"/>
 </instances>
 <busses>
@@
 <wire x1="-2.54" y1="-22.86" x2="17.78" y2="-22.86" width="0.1524" layer="91"/>
 <junction x="-2.54" y="-22.86"/>
-</segment>
-<segment>
-<pinref part="R_PULLUP" gate="G$1" pin="1"/>
-<wire x1="-55.88" y1="58.42" x2="-60.96" y2="58.42" width="0.1524" layer="91"/>
-<label x="-60.96" y="58.42" size="1.778" layer="95" rot="R180" xref="yes"/>
 </segment>
 <segment>
@@
 <label x="38.1" y="66.04" size="1.778" layer="95" rot="R180" xref="yes"/>
 </segment>
-</net>
+<segment>
+<pinref part="R_PULLUP" gate="G$1" pin="1"/>
+<pinref part="GND13" gate="1" pin="GND"/>
+</segment>
+</net>

Commit message: Changes complete - PCB layout ready for tiling
Parts:
- removed OP_HOWL, OP_HOWL1: RC4560SOP65, RC4560:RC4560SOP65
- removed R14: 20k, resistor:R-US_R0805
- removed R_PULLUP: 10k, rcl:R-US_R0805
- added C_OPD1, C_OPD2: 0.1u, resistor:C-EUC0805
- added OP_HOWLA, OP_HOWLB: RC4560SOP65, RC4560:RC4560SOP65
- added R_GAIN2: 1, rcl:R-US_R0805
- added R_PULLDOWN: 20k, rcl:R-US_R0805
- R_HOWA5, R_HOWB4: value 1k -> 10k
- R_SET: device resistor:R-US_R0603 -> resistor:R-US_R0805
Connections:
- new net N$16: JP+.1, S12.P
- net FSYNC: now also R_PULLDOWN.2; no longer R_PULLUP.2
- net FSYNC_IN: no longer R14.2
- net GND: now also C_OPD1.2, C_OPD2.2, R_PULLDOWN.1; no longer R14.1, R_PULLUP.1
- net N$11: now also OP_HOWLB.POSA; no longer OP_HOWL1.POSA
- net N$12: now also OP_HOWLB.NEGA; no longer OP_HOWL1.NEGA
- net N$17: now also OP_HOWLA.OUTB; no longer OP_HOWL.OUTB
- net N$20: now also OP_HOWLA.NEGB; no longer OP_HOWL.NEGB
- net N$24: now also OP_HOWLB.OUTA; no longer OP_HOWL1.OUTA
- net N$3: now also R_GAIN2.1
- net N$5: now also R_GAIN2.2
- net N$7: now also OP_HOWLA.POSB; no longer OP_HOWL.POSB
- net VDD: now also C_OPD1.1, OP_HOWLA.V+, OP_HOWLB.V+; no longer OP_HOWL.V+, OP_HOWL1.V+
- net VSS: now also C_OPD2.1, OP_HOWLA.V-, OP_HOWLB.V-; no longer OP_HOWL1.V-
Other:
- note added: "Gain Stage Can either put in fixed resistor (R_gain2) or potentiometer for setting gain"
- note added: "Left floating - is routed to the FSYNC pins of DDS chips which have a resistor to GND to form a potential divider, giving the correct voltage level for DDS IC"
- note added: "Single ended to differential"
- moved on the sheet: C_DDS1, C_DDS2, C_DDS3, C_DDS4, C_DECOUP, C_OPA1, C_OPA2, C_OPB1, C_OPB2, C_OPC1, C_OPC2, DDS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

Commit message: V5.1 Board - fixing error with footprint of op-amp
Parts:
- R11: value 10k -> 1.5k
Connections:
- removed net FSYNC: DDS.FSYNC, R_PULLDOWN.2, TP_FSYNC.TP
- net FSYNC_CS1: now also DDS.FSYNC, R_PULLDOWN.2, TP_FSYNC.TP
Changed lines of the file:
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@@
 <part name="R9" library="resistor" deviceset="R-US_" device="R0805" value="10k"/>
 <part name="R10" library="resistor" deviceset="R-US_" device="R0805" value="10k"/>
-<part name="R11" library="resistor" deviceset="R-US_" device="R0805" value="10k"/>
+<part name="R11" library="resistor" deviceset="R-US_" device="R0805" value="1.5k"/>
 <part name="R12" library="resistor" deviceset="R-US_" device="R0805" value="20k"/>
 <part name="R13" library="resistor" deviceset="R-US_" device="R0805" value="20k"/>
@@
 </segment>
 </net>
-<net name="FSYNC" class="0">
+<net name="FSYNC_CS1" class="0">
 <segment>
 <pinref part="DDS" gate="A" pin="FSYNC"/>
