File: schematics/Connector.Filter.Board/Connector.Board.brd (EAGLE design)
At the start: 160 x 100 mm, 12 parts, among them U1 RC4560S08-RC4560

Commit message: Added parts for 2 channels
Parts:
- removed R3: 220k, resistor:M0805
- removed R4: 1k, resistor:M0805
- removed U1: RC4560S08-RC4560, RC4560:SO8
- added C3, C4: (no value), resistor:C0805
- added JP1, JP2: (no value), pinhead:1X02/90
- added TP10, TP11, TP12, TP13, TP14, TP15, TP16, TP17, TP18, TP19, TP20, TP21, TP22, TP23, TP24, TP25, TP26, TP27, TP28, TP29, TP3, TP30, TP31, TP32, TP4, TP5, TP6, TP7, TP8, TP9: TOUCHPROOF, connector_board_lib:TOUCHPROOF_PIN
- C2: value 200uF -> (none)
- R2: value 220k -> (none); device resistor:M0805 -> resistor:R0805
- TP1, TP2: value PTR1PAD1-13 -> TOUCHPROOF; device testpad:P1-13 -> connector_board_lib:TOUCHPROOF_PIN
- moved U$2 204.6 mm to (139.7, 85.1), flipped to the bottom, turned to 180 degrees
- moved U$1 200.4 mm to (139.7, 91.4)
- moved R2 182.5 mm to (135.9, 95.2)
- moved C2 180.0 mm to (138.4, 97.8), turned to 180 degrees
- moved C1 179.3 mm to (143.5, 91.4), turned to 270 degrees
- moved R1 176.8 mm to (146.1, 91.4), turned to 270 degrees
- moved TP1 98.8 mm to (38.1, 88.9)
- moved X1 88.2 mm to (17.8, 66.0), turned to 90 degrees
- moved TP2 83.0 mm to (50.8, 88.9)
Connections:
- removed net N$2: R2.1, R3.2, U1.3
- removed net N$6: R4.2, U1.1
- new net BUF2: C2.1, U$1.7, U$2.4
- new net FILT2_BUF: U$1.9
- new net FILT2_OUT: C2.2, R2.2, U$1.10
- net FILT1_BUF: no longer TP2.TP
- net GND: now also C3.2, C4.2, JP1.2, JP2.2, R2.1; no longer R4.1, U1.2
- net PIN10: now also TP10.TP
- net PIN11: now also TP11.TP
- net PIN12: now also TP12.TP
- net PIN13: now also TP13.TP
- net PIN14: now also TP14.TP
- net PIN15: now also TP15.TP
- net PIN16: now also TP16.TP
- net PIN17: now also TP17.TP
- net PIN18: now also TP18.TP
- net PIN19: now also TP19.TP
- net PIN2: now also TP2.TP, U$1.6, U$2.5
- net PIN20: now also TP20.TP
- net PIN21: now also TP21.TP
- net PIN22: now also TP22.TP
- net PIN23: now also TP23.TP
- net PIN24: now also TP24.TP
- net PIN25: now also TP25.TP
- net PIN26: now also TP26.TP
- net PIN27: now also TP27.TP
- net PIN28: now also TP28.TP
- net PIN29: now also TP29.TP
- net PIN3: now also TP3.TP
- net PIN30: now also TP30.TP
- net PIN31: now also TP31.TP
- net PIN32: now also TP32.TP
- net PIN4: now also TP4.TP
- net PIN5: now also TP5.TP
- net PIN6: now also TP6.TP
- net PIN7: now also TP7.TP
- net PIN8: now also TP8.TP
- net PIN9: now also TP9.TP
- net VDD: now also C4.1, JP2.1; no longer C2.1, R2.2, U1.8
- net VSS: now also C3.1, JP1.1; no longer C2.2, R3.1, U1.4

Commit message: example layout for 4 channels
Parts:
- added C10, C11, C12, C5, C6, C7, C8, C9: (no value), resistor:C0805
- added R3, R4: (no value), resistor:R0805
- added U$3: AD8244, AD8244:MSOP10
- added X2: (no value), con-subd:M37HP
- moved C2 16.8 mm to (138.3, 81.0), flipped to the bottom, turned to 90 degrees
- moved R2 15.0 mm to (140.7, 81.0), flipped to the bottom, turned to 90 degrees
- moved U$2 12.2 mm to (134.5, 74.0)
- moved R1 11.7 mm to (140.7, 81.0), turned to 90 degrees
- moved X1 11.6 mm to (12.6, 55.6)
- moved C4 11.6 mm to (27.8, 16.3)
- moved JP2 11.6 mm to (27.8, 8.64)
- moved TP12 11.6 mm to (71.0, 65.8)
- moved TP13 11.6 mm to (83.7, 65.8)
- moved TP20 11.6 mm to (71.0, 53.1)
- moved TP21 11.6 mm to (83.7, 53.1)
- moved TP4 11.6 mm to (71.0, 78.5)
- moved TP5 11.6 mm to (83.7, 78.5)
- moved TP1 11.6 mm to (32.9, 78.5)
- moved TP11 11.6 mm to (58.3, 65.8)
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Connections:
- new net BUF3: C11.1, U$2.9, U$3.9
- new net BUF4: C12.1, U$2.7, U$3.7
- new net FILT10_BUF: X2.10
- new net FILT11_BUF: X2.11
- new net FILT12_BUF: X2.12
- new net FILT13_BUF: X2.13
- new net FILT14_BUF: X2.14
- new net FILT15_BUF: X2.15
- new net FILT16_BUF: X2.16
- new net FILT17_BUF: X2.17
- new net FILT18_BUF: X2.18
- new net FILT19_BUF: X2.19
- new net FILT20_BUF: X2.20
- new net FILT21_BUF: X2.21
- new net FILT22_BUF: X2.22
- new net FILT23_BUF: X2.23
- new net FILT24_BUF: X2.24
- new net FILT25_BUF: X2.25
- new net FILT26_BUF: X2.26
- new net FILT27_BUF: X2.27
- new net FILT28_BUF: X2.28
- new net FILT29_BUF: X2.29
- new net FILT30_BUF: X2.30
- new net FILT31_BUF: X2.31
- new net FILT32_BUF: X2.32
- new net FILT3_BUF: U$3.2, X2.3
- new net FILT3_OUT: C11.2, R3.2, U$3.1
- new net FILT4_BUF: U$3.4, X2.4
- new net FILT4_OUT: C12.2, R4.2, U$3.5
- new net FILT5_BUF: X2.5
- new net FILT6_BUF: X2.6
- new net FILT7_BUF: X2.7
- new net FILT8_BUF: X2.8
- new net FILT9_BUF: X2.9
- net BUF2: now also U$1.4; no longer U$1.7
- net FILT1_BUF: now also U$1.7, X2.1; no longer U$1.4
- net FILT1_OUT: now also U$1.6; no longer U$1.5
- net FILT2_BUF: now also X2.2
- net GND: now also C10.2, C5.2, C6.2, C7.2, C8.2, C9.2, R3.1, R4.1
- net PIN2: now also U$1.5; no longer U$1.6
- net PIN3: now also U$2.10, U$3.10
- net PIN4: now also U$2.6, U$3.6
- net VDD: now also C10.1, C7.1, C8.1, U$1.8, U$2.8, U$3.8; no longer U$1.3
- net VSS: now also C5.1, C6.1, C9.1, U$1.3, U$2.3, U$3.3; no longer U$1.8, U$2.8
Routing:
- net VDD: track 0.00 -> 41.2 mm, vias 0 -> 5
- net VSS: track 0.00 -> 37.6 mm, vias 0 -> 5
- net PIN2: track 0.00 -> 15.4 mm, vias 0 -> 1
- net FILT2_BUF: track 0.00 -> 12.8 mm
- net PIN4: track 0.00 -> 12.4 mm, vias 0 -> 1
- net FILT3_BUF: track 0.00 -> 10.9 mm
- net BUF1: track 0.00 -> 10.2 mm, vias 0 -> 1
- net PIN1: track 0.00 -> 9.76 mm, vias 0 -> 1
- net FILT4_BUF: track 0.00 -> 9.44 mm
- net PIN3: track 0.00 -> 9.07 mm, vias 0 -> 1
- net FILT1_BUF: track 0.00 -> 9.04 mm
- net FILT2_OUT: track 0.00 -> 8.45 mm, vias 0 -> 1
- net BUF2: track 0.00 -> 7.94 mm, vias 0 -> 2
- net BUF3: track 0.00 -> 7.86 mm, vias 0 -> 2
- net FILT3_OUT: track 0.00 -> 7.69 mm, vias 0 -> 1
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- added copper zone on layer 15, net GND

Commit message: now passing ERC
Routing:
- net FILT3_BUF: track 10.9 -> 12.3 mm
- net VSS: track 37.6 -> 38.4 mm
Changed lines of the file:
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@@
 <contactref element="U$3" pad="3"/>
 <contactref element="C9" pad="1"/>
-<wire x1="134.493" y1="65.387" x2="134.493" y2="64.643" width="0.2" layer="1"/>
-<via x="134.493" y="64.643" extent="1-16" drill="0.4"/>
-<wire x1="134.493" y1="64.643" x2="134.493" y2="64.516" width="0.2" layer="2"/>
-<wire x1="134.493" y1="64.516" x2="132.969" y2="64.516" width="0.2" layer="2"/>
+<wire x1="134.493" y1="65.387" x2="134.493" y2="64.135" width="0.2" layer="1"/>
+<via x="134.493" y="64.135" extent="1-16" drill="0.4"/>
 <wire x1="132.969" y1="64.516" x2="132.461" y2="65.024" width="0.2" layer="2"/>
 <wire x1="132.461" y1="65.024" x2="132.461" y2="65.659" width="0.2" layer="2"/>
@@
 <wire x1="138.303" y1="74.93" x2="138.303" y2="67.056" width="0.2" layer="2"/>
 <wire x1="138.303" y1="67.056" x2="135.89" y2="64.643" width="0.2" layer="2"/>
-<wire x1="135.89" y1="64.643" x2="134.493" y2="64.643" width="0.2" layer="2"/>
 <wire x1="133.604" y1="76.708" x2="133.223" y2="76.708" width="0.2" layer="2"/>
+<wire x1="132.969" y1="64.516" x2="133.35" y2="64.135" width="0.2" layer="2"/>
+<wire x1="133.35" y1="64.135" x2="134.493" y2="64.135" width="0.2" layer="2"/>
 <wire x1="46.543" y1="14.986" x2="130.871" y2="66.04" width="0" layer="19" extent="1-1"/>
 <wire x1="46.863" y1="12.446" x2="46.543" y2="14.986" width="0" layer="19" extent="1-1"/>
+<wire x1="135.89" y1="64.643" x2="135.382" y2="64.135" width="0.2" layer="2"/>
+<wire x1="135.382" y1="64.135" x2="134.493" y2="64.135" width="0.2" layer="2"/>
 </signal>
 <signal name="FILT1_BUF">
@@
 <contactref element="X2" pad="3"/>
 <contactref element="U$3" pad="2"/>
-<wire x1="133.993" y1="65.387" x2="133.993" y2="64.635" width="0.2" layer="1"/>
-<wire x1="133.993" y1="64.635" x2="135.001" y2="63.627" width="0.2" layer="1"/>
-<wire x1="135.001" y1="63.627" x2="143.383" y2="63.627" width="0.2" layer="1"/>
 <wire x1="143.383" y1="63.627" x2="143.637" y2="63.373" width="0.2" layer="1"/>
+<wire x1="133.993" y1="65.387" x2="133.993" y2="64.778" width="0.2" layer="1"/>
+<wire x1="133.993" y1="64.778" x2="133.604" y2="64.389" width="0.2" layer="1"/>
+<wire x1="133.604" y1="64.389" x2="133.604" y2="63.627" width="0.2" layer="1"/>
+<wire x1="133.604" y1="63.627" x2="133.858" y2="63.373" width="0.2" layer="1"/>
+<wire x1="133.858" y1="63.373" x2="135.509" y2="63.373" width="0.2" layer="1"/>
 <wire x1="147.32" y1="36.2966" x2="143.637" y2="63.373" width="0" layer="19" extent="1-1"/>
+<wire x1="135.509" y1="63.373" x2="135.763" y2="63.627" width="0.2" layer="1"/>
+<wire x1="135.763" y1="63.627" x2="143.383" y2="63.627" width="0.2" layer="1"/>
 </signal>
 <signal name="FILT4_BUF">
@@
 <contactref element="U$3" pad="4"/>
 <wire x1="134.993" y1="65.387" x2="134.993" y2="64.905" width="0.2" layer="1"/>
-<wire x1="134.993" y1="64.905" x2="135.636" y2="64.262" width="0.2" layer="1"/>
 <wire x1="135.636" y1="64.262" x2="143.51" y2="64.262" width="0.2" layer="1"/>
 <wire x1="143.51" y1="64.262" x2="143.637" y2="64.135" width="0.2" layer="1"/>
+<wire x1="134.993" y1="64.905" x2="134.993" y2="64.778" width="0.2" layer="1"/>
+<wire x1="134.993" y1="64.778" x2="135.001" y2="64.77" width="0.2" layer="1"/>
+<wire x1="135.001" y1="64.77" x2="135.509" y2="64.262" width="0.2" layer="1"/>
+<wire x1="135.509" y1="64.262" x2="135.636" y2="64.262" width="0.2" layer="1"/>
 <wire x1="147.32" y1="39.0652" x2="143.637" y2="64.135" width="0" layer="19" extent="1-1"/>
 </signal>

Commit message: Duplicated layout through renaming parts
Parts:
- added C13, C14, C15, C16, C17, C18, C19, C20, C21, C22: (no value), resistor:C0805
- added R5, R6, R7, R8: (no value), resistor:R0805
- added U$4, U$5, U$6: AD8244, AD8244:MSOP10
Connections:
- new net BUF5: C19.1, U$4.2, U$5.2
- new net BUF6: C20.1, U$4.4, U$5.4
- new net BUF7: C21.1, U$5.9, U$6.9
- new net BUF8: C22.1, U$5.7, U$6.7
- new net FILT5_OUT: C19.2, R5.2, U$4.6
- new net FILT6_OUT: C20.2, R6.2, U$4.10
- new net FILT7_OUT: C21.2, R7.2, U$6.1
- new net FILT8_OUT: C22.2, R8.2, U$6.5
- net FILT5_BUF: now also U$4.7
- net FILT6_BUF: now also U$4.9
- net FILT7_BUF: now also U$6.2
- net FILT8_BUF: now also U$6.4
- net GND: now also C13.2, C14.2, C15.2, C16.2, C17.2, C18.2, R5.1, R6.1, R7.1, R8.1
- net PIN5: now also U$4.1, U$5.1
- net PIN6: now also U$4.5, U$5.5
- net PIN7: now also U$5.10, U$6.10
- net PIN8: now also U$5.6, U$6.6
- net VDD: now also C15.1, C16.1, C18.1, U$4.8, U$5.8, U$6.8
- net VSS: now also C13.1, C14.1, C17.1, U$4.3, U$5.3, U$6.3
Routing:
- net VDD: track 41.2 -> 82.4 mm, vias 5 -> 10
- net VSS: track 38.4 -> 76.8 mm, vias 5 -> 10
- net PIN6: track 0.00 -> 15.4 mm, vias 0 -> 1
- net FILT6_BUF: track 0.00 -> 12.8 mm
- net PIN8: track 0.00 -> 12.4 mm, vias 0 -> 1
- net FILT7_BUF: track 0.00 -> 12.3 mm
- net BUF5: track 0.00 -> 10.2 mm, vias 0 -> 1
- net PIN5: track 0.00 -> 9.76 mm, vias 0 -> 1
- net FILT8_BUF: track 0.00 -> 9.52 mm
- net PIN7: track 0.00 -> 9.07 mm, vias 0 -> 1
- net FILT5_BUF: track 0.00 -> 9.04 mm
- net FILT6_OUT: track 0.00 -> 8.45 mm, vias 0 -> 1
- net BUF6: track 0.00 -> 7.94 mm, vias 0 -> 2
- net BUF7: track 0.00 -> 7.86 mm, vias 0 -> 2
- net FILT7_OUT: track 0.00 -> 7.69 mm, vias 0 -> 1
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
Commit message: 12 chn board finished
Parts:
- added C23, C24, C25, C26, C27, C28, C29, C30, C31, C32, C33, C34, C35, C36: (no value), resistor:C0805
- added D1, D3: 1N4148W-7-F, diode:SOD123
- added R10, R11, R12, R9: (no value), resistor:R0805
- added U$7, U$8, U$9: AD8244, AD8244:MSOP10
- moved JP2 87.8 mm to (114.8, 20.2)
- moved C4 87.7 mm to (114.8, 27.1)
- moved C3 77.3 mm to (121.9, 27.2)
- moved JP1 77.2 mm to (121.9, 20.2)
- moved C13 5.96 mm to (129.2, 62.9)
- moved C14 5.96 mm to (129.2, 57.7)
- moved C15 5.96 mm to (129.2, 55.5)
- moved C17 5.96 mm to (129.3, 48.4)
- moved C21 5.96 mm to (136.9, 49.9)
- moved C22 5.96 mm to (136.9, 49.9)
- moved R7 5.96 mm to (139.4, 49.9)
- moved R8 5.96 mm to (139.4, 49.9)
- moved C16 5.96 mm to (129.2, 65.5)
- moved C18 5.96 mm to (129.3, 50.8)
- moved C19 5.96 mm to (137.7, 63.4)
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Connections:
- removed net VDD: C10.1, C15.1, C16.1, C18.1, C4.1, C7.1, C8.1, JP2.1, U$1.8, U$2.8, U$3.8, U$4.8, U$5.8, U$6.8
- removed net VSS: C13.1, C14.1, C17.1, C3.1, C5.1, C6.1, C9.1, JP1.1, U$1.3, U$2.3, U$3.3, U$4.3, U$5.3, U$6.3
- new net BUF10: C28.1, U$7.4, U$8.4
- new net BUF11: C29.1, U$8.9, U$9.9
- new net BUF12: C30.1, U$8.7, U$9.7
- new net BUF9: C27.1, U$7.2, U$8.2
- new net FILT10_OUT: C28.2, R10.2, U$7.10
- new net FILT11_OUT: C29.2, R11.2, U$9.1
- new net FILT12_OUT: C30.2, R12.2, U$9.5
- new net FILT9_OUT: C27.2, R9.2, U$7.6
- new net V+: C13.1, C14.1, C17.1, C23.1, C24.1, C3.1, C31.1, C32.1, C35.1, C5.1, C6.1, C9.1, D1.C, JP1.1, U$1.3, U$2.3, U$3.3, U$4.3, U$5.3, U$6.3, U$7.3, U$8.3, U$9.3
- new net V-: C10.1, C15.1, C16.1, C18.1, C25.1, C26.1, C33.1, C34.1, C36.1, C4.1, C7.1, C8.1, D3.A, JP2.1, U$1.8, U$2.8, U$3.8, U$4.8, U$5.8, U$6.8, U$7.8, U$8.8, U$9.8
- net FILT10_BUF: now also U$7.9
- net FILT11_BUF: now also U$9.2
- net FILT12_BUF: now also U$9.4
- net FILT9_BUF: now also U$7.7
- net GND: now also C23.2, C24.2, C25.2, C26.2, C31.2, C32.2, C33.2, C34.2, C35.2, C36.2, D1.A, D3.C, R10.1, R11.1, R12.1, R9.1
- net PIN10: now also U$7.5, U$8.5
- net PIN11: now also U$8.10, U$9.10
- net PIN12: now also U$8.6, U$9.6
- net PIN9: now also U$7.1, U$8.1
Routing:
- net GND: track 0.00 -> 310.2 mm, vias 0 -> 14
- net PIN5: track 9.76 -> 188.4 mm
- net V-: track 0.00 -> 178.3 mm, vias 0 -> 15
- net PIN7: track 9.07 -> 185.4 mm
- net PIN8: track 12.4 -> 186.9 mm
- net PIN10: track 0.00 -> 170.9 mm, vias 0 -> 2
- net PIN6: track 15.4 -> 186.0 mm
- net PIN12: track 0.00 -> 170.3 mm, vias 0 -> 2
- net PIN9: track 0.00 -> 169.9 mm, vias 0 -> 2
- net PIN3: track 9.07 -> 177.5 mm
- net PIN4: track 12.4 -> 180.4 mm
- net V+: track 0.00 -> 165.1 mm, vias 0 -> 15
- net PIN11: track 0.00 -> 164.1 mm, vias 0 -> 2
- net PIN2: track 15.4 -> 179.1 mm
- net PIN1: track 9.76 -> 167.9 mm
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- added copper zone on layer 1, net GND
- added copper zone on layer 16, net GND
Other:
- board size 160 x 100 mm -> 159.4 x 72.1 mm
