File: schematics/Connector.Filter.Board/Connector.Board.brd (EAGLE design)
At the start: 159.4 x 72.1 mm, 95 parts, among them U1 AD8244, U2 AD8244, U3 AD8244, U4 AD8244, U5 AD8244, U6 AD8244, U7 AD8244, U8 AD8244, U9 AD8244, X1 EEGCON, X2 EITCON

Commit message: Renaming Sch and Brd but not matching yet
Parts:
- added C100A, C101A, C102A, C103A, C104A, C105A, C109A, C110A, C111A, C112A, C113A, C114A, C119A, C120A, C121A, C122A, C123A, C124A, C39, C40, C41, C42, C43, C44, C45, C49, C50, C51, C52, C53, C54, C59, C60, C61, C62, C63, C64, C69A, C70A, C71A, C72A, C73A, C74A, C75A, C79A, C80A, C81A, C82A, C83A, C84A, C89A, C90A, C91A, C92A, C93A, C94A, C99A: 0.1uF, resistor:C0805
- added C106A, C107A, C108A, C115A, C116A, C117A, C118A, C125, C126A, C37, C38, C46, C47, C48, C55, C56, C57, C58, C65, C66, C67A, C68A, C76A, C77A, C78A, C85A, C86A, C87A, C88A, C95A, C96A, C97A, C98A: (no value), resistor:C0805
- added R13, R14, R15, R16, R17, R18, R19, R20, R21, R22, R23, R24, R25A, R26A, R27A, R28A, R29A, R30A, R31, R32, R33A, R34A, R35A, R36A, R37A, R38A, R39A, R40A, R41A, R42A, R43A, R44A, R45A, R46A, R47, R48A: (no value), resistor:R0805
- added U10, U11, U12, U13, U14, U15, U16, U17, U18, U19A, U20A, U21A, U22A, U23A, U24, U25A, U26A, U27A, U28A, U29A, U30A, U31A, U32A, U33A, U34A, U35A, U36A: AD8244, AD8244:MSOP10
- moved X1 49.7 mm to (198.2, 55.2)
Connections:
- new net BUF13: C37.1, C97A.1, U10.2, U11.2, U28A.2, U29A.2
- new net BUF14: C38.1, C98A.1, U10.4, U11.4, U28A.4, U29A.4
- new net BUF15: C105A.1, C45.1, U11.9, U12.9, U29A.9, U30A.9
- new net BUF16: C106A.1, C46.1, U11.7, U12.7, U29A.7, U30A.7
- new net BUF17: C107A.1, C47.1, U13.2, U14.2, U31A.2, U32A.2
- new net BUF18: C108A.1, C48.1, U13.4, U14.4, U31A.4, U32A.4
- new net BUF19: C115A.1, C55.1, U14.9, U15.9, U32A.9, U33A.9
- new net BUF20: C116A.1, C56.1, U14.7, U15.7, U32A.7, U33A.7
- new net BUF21: C117A.1, C57.1, U16.2, U17.2, U34A.2, U35A.2
- new net BUF22: C118A.1, C58.1, U16.4, U17.4, U34A.4, U35A.4
- new net BUF23: C125.1, C65.1, U17.9, U18.9, U35A.9, U36A.9
- new net BUF24: C126A.1, C66.1, U17.7, U18.7, U35A.7, U36A.7
- new net BUF25: C67A.1, U19A.2, U20A.2
- new net BUF26: C68A.1, U19A.4, U20A.4
- new net BUF27: C75A.1, U20A.9, U21A.9
- new net BUF28: C76A.1, U20A.7, U21A.7
- new net BUF29: C77A.1, U22A.2, U23A.2
- new net BUF30: C78A.1, U22A.4, U23A.4
- new net BUF31: C85A.1, U23A.9, U24.9
- new net BUF32: C86A.1, U23A.7, U24.7
- new net BUF33: C87A.1, U25A.2, U26A.2
- new net BUF34: C88A.1, U25A.4, U26A.4
- new net BUF35: C95A.1, U26A.9, U27A.9
- new net BUF36: C96A.1, U26A.7, U27A.7
- new net FILT10_BUF1: U16.9
- new net FILT10_BUF2: U25A.9
- new net FILT10_OUT1: C58.2, R22.2, U16.10
- new net FILT10_OUT2: C88A.2, R34A.2, U25A.10
- new net FILT11_BUF1: U18.2
- new net FILT11_BUF2: U27A.2
- new net FILT11_OUT1: C65.2, R23.2, U18.1
- new net FILT11_OUT2: C95A.2, R35A.2, U27A.1
- new net FILT12_BUF1: U18.4
- new net FILT12_BUF2: U27A.4
- new net FILT12_OUT1: C66.2, R24.2, U18.5
- new net FILT12_OUT2: C96A.2, R36A.2, U27A.5
- new net FILT14_OUT: C98A.2, R38A.2, U28A.10
- new net FILT15_OUT: C105A.2, R39A.2, U30A.1
- new net FILT16_OUT: C106A.2, R40A.2, U30A.5
- new net FILT17_OUT: C107A.2, R41A.2, U31A.6
- new net FILT18_OUT: C108A.2, R42A.2, U31A.10
- new net FILT19_OUT: C115A.2, R43A.2, U33A.1
- new net FILT1_BUF1: U10.7
- new net FILT1_OUT1: C37.2, R13.2, U10.6
- new net FILT20_OUT: C116A.2, R44A.2, U33A.5
- new net FILT21_OUT: C117A.2, R45A.2, U34A.6
- new net FILT22_OUT: C118A.2, R46A.2, U34A.10
- new net FILT23_OUT: C125.2, R47.2, U36A.1
- new net FILT24_OUT: C126A.2, R48A.2, U36A.5
- new net FILT25_OUT: C67A.2, R25A.2, U19A.6
- new net FILT26_OUT: C68A.2, R26A.2, U19A.10
- new net FILT27_OUT: C75A.2, R27A.2, U21A.1
- new net FILT28_OUT: C76A.2, R28A.2, U21A.5
- new net FILT2_BUF1: U10.9
- new net FILT2_OUT1: C38.2, R14.2, U10.10
- new net FILT31_OUT: C85A.2, R31.2, U24.1
- new net FILT32_OUT: C86A.2, R32.2, U24.5
- new net FILT3_BUF1: U12.2
- new net FILT3_OUT1: C45.2, R15.2, U12.1
- new net FILT4_BUF1: U12.4
- new net FILT4_OUT1: C46.2, R16.2, U12.5
- new net FILT5_BUF1: U13.7
- new net FILT5_BUF2: U22A.7
- new net FILT5_OUT1: C47.2, R17.2, U13.6
- new net FILT5_OUT2: C77A.2, R29A.2, U22A.6
- new net FILT6_BUF1: U13.9
- new net FILT6_BUF2: U22A.9
- new net FILT6_OUT1: C48.2, R18.2, U13.10
- new net FILT6_OUT2: C78A.2, R30A.2, U22A.10
- new net FILT7_BUF1: U15.2
- new net FILT7_OUT1: C55.2, R19.2, U15.1
- new net FILT8_BUF1: U15.4
- new net FILT8_OUT1: C56.2, R20.2, U15.5
- new net FILT9_BUF1: U16.7
- new net FILT9_BUF2: U25A.7
- new net FILT9_OUT1: C57.2, R21.2, U16.6
- new net FILT9_OUT2: C87A.2, R33A.2, U25A.6
- new net PIN33: U10.1, U11.1
- new net PIN34: U10.5, U11.5
- new net PIN35: U11.10, U12.10
- new net PIN36: U11.6, U12.6
- new net PIN37: U13.1, U14.1
- new net PIN38: U13.5, U14.5
- new net PIN39: U14.10, U15.10
- new net PIN40: U14.6, U15.6
- new net PIN41: U16.1, U17.1
- new net PIN42: U16.5, U17.5
- new net PIN43: U17.10, U18.10
- new net PIN44: U17.6, U18.6
- new net PIN53: U25A.1, U26A.1
- new net PIN54: U25A.5, U26A.5
- new net PIN55: U26A.10, U27A.10
- new net PIN56: U26A.6, U27A.6
- net FILT13_BUF: now also U28A.7
- net FILT14_BUF: now also U28A.9
- net FILT15_BUF: now also U30A.2
- net FILT16_BUF: now also U30A.4
- net FILT17_BUF: now also U31A.7
- net FILT18_BUF: now also U31A.9
- net FILT19_BUF: now also U33A.2
- net FILT20_BUF: now also U33A.4
- net FILT21_BUF: now also U34A.7
- net FILT22_BUF: now also U34A.9
- net FILT23_BUF: now also U36A.2
- net FILT24_BUF: now also U36A.4
- net FILT25_BUF: now also U19A.7
- net FILT26_BUF: now also U19A.9
- net FILT27_BUF: now also U21A.2
- net FILT28_BUF: now also U21A.4
- net FILT31_BUF: now also U24.2
- net FILT32_BUF: now also U24.4
- net FILT3_OUT: now also C97A.2, R37A.2, U28A.6
- net GND: now also C100A.2, C101A.2, C102A.2, C103A.2, C104A.2, C109A.2, C110A.2, C111A.2, C112A.2, C113A.2, C114A.2, C119A.2, C120A.2, C121A.2, C122A.2, C123A.2, C124A.2, C39.2, C40.2, C41.2, C42.2, C43.2, C44.2, C49.2, C50.2, C51.2, C52.2, C53.2, C54.2, C59.2, C60.2, C61.2, C62.2, C63.2, C64.2, C69A.2, C70A.2, C71A.2, C72A.2, C73A.2, C74A.2, C79A.2, C80A.2, C81A.2, C82A.2, C83A.2, C84A.2, C89A.2, C90A.2, C91A.2, C92A.2, C93A.2, C94A.2, C99A.2, R13.1, R14.1, R15.1, R16.1, R17.1, R18.1, R19.1, R20.1, R21.1, R22.1, R23.1, R24.1, R25A.1, R26A.1, R27A.1, R28A.1, R29A.1, R30A.1, R31.1, R32.1, R33A.1, R34A.1, R35A.1, R36A.1, R37A.1, R38A.1, R39A.1, R40A.1, R41A.1, R42A.1, R43A.1, R44A.1, R45A.1, R46A.1, R47.1, R48A.1
- net PIN13: now also U28A.1, U29A.1
- net PIN14: now also U28A.5, U29A.5
- net PIN15: now also U29A.10, U30A.10
- net PIN16: now also U29A.6, U30A.6
- net PIN17: now also U31A.1, U32A.1
- net PIN18: now also U31A.5, U32A.5
- net PIN19: now also U32A.10, U33A.10
- net PIN20: now also U32A.6, U33A.6
- net PIN21: now also U34A.1, U35A.1
- net PIN22: now also U34A.5, U35A.5
- net PIN23: now also U35A.10, U36A.10
- net PIN24: now also U35A.6, U36A.6
- net PIN25: now also U19A.1, U20A.1
- net PIN26: now also U19A.5, U20A.5
- net PIN27: now also U20A.10, U21A.10
- net PIN28: now also U20A.6, U21A.6
- net PIN29: now also U22A.1, U23A.1
- net PIN30: now also U22A.5, U23A.5
- net PIN31: now also U23A.10, U24.10
- net PIN32: now also U23A.6, U24.6
- net V+: now also C100A.1, C103A.1, C109A.1, C110A.1, C113A.1, C119A.1, C120A.1, C123A.1, C39.1, C40.1, C43.1, C49.1, C50.1, C53.1, C59.1, C60.1, C63.1, C69A.1, C70A.1, C73A.1, C79A.1, C80A.1, C83A.1, C89A.1, C90A.1, C93A.1, C99A.1, U10.3, U11.3, U12.3, U13.3, U14.3, U15.3, U16.3, U17.3, U18.3, U19A.3, U20A.3, U21A.3, U22A.3, U23A.3, U24.3, U25A.3, U26A.3, U27A.3, U28A.3, U29A.3, U30A.3, U31A.3, U32A.3, U33A.3, U34A.3, U35A.3, U36A.3
- net V-: now also C101A.1, C102A.1, C104A.1, C111A.1, C112A.1, C114A.1, C121A.1, C122A.1, C124A.1, C41.1, C42.1, C44.1, C51.1, C52.1, C54.1, C61.1, C62.1, C64.1, C71A.1, C72A.1, C74A.1, C81A.1, C82A.1, C84A.1, C91A.1, C92A.1, C94A.1, U10.8, U11.8, U12.8, U13.8, U14.8, U15.8, U16.8, U17.8, U18.8, U19A.8, U20A.8, U21A.8, U22A.8, U23A.8, U24.8, U25A.8, U26A.8, U27A.8, U28A.8, U29A.8, U30A.8, U31A.8, U32A.8, U33A.8, U34A.8, U35A.8, U36A.8
Routing:
- net GND: track 310.2 -> 875.9 mm, vias 14 -> 44
- net V+: track 165.1 -> 621.4 mm, vias 15 -> 60
- net V-: track 178.3 -> 470.2 mm, vias 15 -> 60
- net FILT1_BUF: track 90.6 -> 7.96 mm, vias 1 -> 0
- net FILT2_BUF: track 88.9 -> 11.0 mm
- net FILT12_BUF: track 49.6 -> 6.55 mm, vias 1 -> 0
- net FILT11_BUF: track 51.2 -> 10.3 mm, vias 1 -> 0
- net FILT3_BUF: track 50.1 -> 11.9 mm, vias 1 -> 0
- net FILT4_BUF: track 45.3 -> 8.96 mm
- net PIN30: track 97.5 -> 127.9 mm, vias 0 -> 1
- net PIN18: track 58.5 -> 88.9 mm, vias 1 -> 2
- net PIN38: track 0.00 -> 30.4 mm, vias 0 -> 1
- net FILT5_BUF: track 35.8 -> 7.96 mm, vias 1 -> 0
- net FILT6_BUF: track 36.3 -> 11.0 mm, vias 1 -> 0
- net BUF13: track 0.00 -> 20.3 mm, vias 0 -> 2
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- removed copper zone on layer 1, net GND
- removed copper zone on layer 16, net GND
Other:
- board size 159.4 x 72.1 mm -> 188 x 72 mm

Commit message: brd and sch match
Parts:
- removed C100A, C101A, C102A, C103A, C104A, C105A, C109A, C110A, C111A, C112A, C113A, C114A, C119A, C120A, C121A, C122A, C123A, C124A, C75A, C89A, C90A, C91A, C92A, C93A, C94A, C99A: 0.1uF, resistor:C0805
- removed C106A, C107A, C108A, C115A, C116A, C117A, C118A, C125, C126A, C67A, C68A, C76A, C77A, C78A, C85A, C86A, C87A, C88A, C95A, C96A, C97A, C98A: (no value), resistor:C0805
- removed R25A, R26A, R27A, R28A, R29A, R30A, R33A, R34A, R35A, R36A, R37A, R38A, R39A, R40A, R41A, R42A, R43A, R44A, R45A, R46A, R47, R48A: (no value), resistor:R0805
- removed U25A, U26A, U27A, U28A, U29A, U30A, U31A, U32A, U33A, U34A, U35A, U36A: AD8244, AD8244:MSOP10
- added C67, C68, C76, C83, C84, C85, C86: (no value), resistor:C0805
- added C75: 0.1uF, resistor:C0805
- added R25, R26, R27, R28, R29, R30: (no value), resistor:R0805
- C47, C48, C65, C66: value (none) -> 0.1uF
- C53, C54, C59, C60: value 0.1uF -> (none)
- moved C48 41.5 mm to (145.4, 57.7), turned to 0 degrees
- moved C47 41.2 mm to (145.4, 62.9), turned to 180 degrees
- moved C65 40.3 mm to (145.5, 25.9), flipped to the top, turned to 180 degrees
- moved C66 40.3 mm to (145.5, 28.3), turned to 180 degrees
- moved C64 35.9 mm to (145.4, 43.1)
- moved C52 35.7 mm to (145.5, 50.8)
- moved C50 33.6 mm to (145.4, 65.5), flipped to the top, turned to 180 degrees
- moved C62 33.6 mm to (145.4, 35.2), flipped to the bottom, turned to 0 degrees
- moved C63 33.5 mm to (145.4, 33.0), flipped to the bottom, turned to 0 degrees
- moved C49 33.5 mm to (145.4, 55.5), flipped to the bottom, turned to 0 degrees
- moved C61 33.5 mm to (145.4, 40.4), flipped to the top, turned to 180 degrees
- moved C51 33.3 mm to (145.5, 48.4), flipped to the top, turned to 180 degrees
- moved C37 32.6 mm to (153.8, 86.0)
- moved C38 32.6 mm to (153.8, 86.0)
- moved C43 32.6 mm to (145.4, 71.0)
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- renumbered C69A to C69, C70A to C70, C71A to C71, C72A to C72, C73A to C73, C74A to C74, C79A to C77, C80A to C78, C81A to C79, C82A to C80, C83A to C81, C84A to C82, U19A to U19, U20A to U20, U21A to U21, U22A to U22, U23A to U23
Connections:
- net FILT1_OUT1 renamed FILT13_OUT
- removed net BUF33: C87A.1, U25A.2, U26A.2
- removed net BUF34: C88A.1, U25A.4, U26A.4
- removed net BUF35: C95A.1, U26A.9, U27A.9
- removed net BUF36: C96A.1, U26A.7, U27A.7
- removed net FILT10_BUF1: U16.9
- removed net FILT10_BUF2: U25A.9
- removed net FILT10_OUT1: C58.2, R22.2, U16.10
- removed net FILT10_OUT2: C88A.2, R34A.2, U25A.10
- removed net FILT11_BUF1: U18.2
- removed net FILT11_BUF2: U27A.2
- removed net FILT11_OUT1: C65.2, R23.2, U18.1
- removed net FILT11_OUT2: C95A.2, R35A.2, U27A.1
- removed net FILT12_BUF1: U18.4
- removed net FILT12_BUF2: U27A.4
- removed net FILT12_OUT1: C66.2, R24.2, U18.5
- removed net FILT12_OUT2: C96A.2, R36A.2, U27A.5
- removed net FILT1_BUF1: U10.7
- removed net FILT2_BUF1: U10.9
- removed net FILT2_OUT1: C38.2, R14.2, U10.10
- removed net FILT3_BUF1: U12.2
- removed net FILT3_OUT1: C45.2, R15.2, U12.1
- removed net FILT4_BUF1: U12.4
- removed net FILT4_OUT1: C46.2, R16.2, U12.5
- removed net FILT5_BUF1: U13.7
- removed net FILT5_BUF2: U22.7
- removed net FILT5_OUT1: C47.2, R17.2, U13.6
- removed net FILT5_OUT2: C77A.2, R29A.2, U22.6
- removed net FILT6_BUF1: U13.9
- removed net FILT6_BUF2: U22.9
- removed net FILT6_OUT1: C48.2, R18.2, U13.10
- removed net FILT6_OUT2: C78A.2, R30A.2, U22.10
- removed net FILT7_BUF1: U15.2
- removed net FILT7_OUT1: C55.2, R19.2, U15.1
- removed net FILT8_BUF1: U15.4
- removed net FILT8_OUT1: C56.2, R20.2, U15.5
- removed net FILT9_BUF1: U16.7
- removed net FILT9_BUF2: U25A.7
- removed net FILT9_OUT1: C57.2, R21.2, U16.6
- removed net FILT9_OUT2: C87A.2, R33A.2, U25A.6
- removed net PIN33: U10.1, U11.1
- removed net PIN34: U10.5, U11.5
- removed net PIN35: U11.10, U12.10
- removed net PIN36: U11.6, U12.6
- removed net PIN37: U13.1, U14.1
- removed net PIN38: U13.5, U14.5
- removed net PIN39: U14.10, U15.10
- removed net PIN40: U14.6, U15.6
- removed net PIN41: U16.1, U17.1
- removed net PIN42: U16.5, U17.5
- removed net PIN43: U17.10, U18.10
- removed net PIN44: U17.6, U18.6
- removed net PIN53: U25A.1, U26A.1
- removed net PIN54: U25A.5, U26A.5
- removed net PIN55: U26A.10, U27A.10
- removed net PIN56: U26A.6, U27A.6
- new net FILT29_OUT: C83.2, R29.2, U22.6
- new net FILT30_OUT: C84.2, R30.2, U22.10
- net BUF13: no longer C97A.1, U28A.2, U29A.2
- net BUF14: no longer C98A.1, U28A.4, U29A.4
- net BUF15: no longer C105A.1, U29A.9, U30A.9
- net BUF16: no longer C106A.1, U29A.7, U30A.7
- net BUF17: now also C53.1; no longer C107A.1, C47.1, U31A.2, U32A.2
- net BUF18: now also C54.1; no longer C108A.1, C48.1, U31A.4, U32A.4
- net BUF19: no longer C115A.1, U32A.9, U33A.9
- net BUF20: no longer C116A.1, U32A.7, U33A.7
- net BUF21: no longer C117A.1, U34A.2, U35A.2
- net BUF22: no longer C118A.1, U34A.4, U35A.4
- net BUF23: now also C59.1; no longer C125.1, C65.1, U35A.9, U36A.9
- net BUF24: now also C60.1; no longer C126A.1, C66.1, U35A.7, U36A.7
- net BUF25: now also C67.1; no longer C67A.1
- net BUF26: now also C68.1; no longer C68A.1
- net BUF27: now also C75.1; no longer C75A.1
- net BUF28: now also C76.1; no longer C76A.1
- net BUF29: now also C83.1; no longer C77A.1
- net BUF30: now also C84.1; no longer C78A.1
- net BUF31: now also C85.1; no longer C85A.1
- net BUF32: now also C86.1; no longer C86A.1
- net FILT13_BUF: now also U10.7; no longer U28A.7
- net FILT14_BUF: now also U10.9; no longer U28A.9
- net FILT14_OUT: now also C38.2, R14.2, U10.10; no longer C98A.2, R38A.2, U28A.10
- net FILT15_BUF: now also U12.2; no longer U30A.2
- net FILT15_OUT: now also C45.2, R15.2, U12.1; no longer C105A.2, R39A.2, U30A.1
- net FILT16_BUF: now also U12.4; no longer U30A.4
- net FILT16_OUT: now also C46.2, R16.2, U12.5; no longer C106A.2, R40A.2, U30A.5
- net FILT17_BUF: now also U13.7; no longer U31A.7
- net FILT17_OUT: now also C53.2, R17.2, U13.6; no longer C107A.2, R41A.2, U31A.6
- net FILT18_BUF: now also U13.9; no longer U31A.9
- net FILT18_OUT: now also C54.2, R18.2, U13.10; no longer C108A.2, R42A.2, U31A.10
- net FILT19_BUF: now also U15.2; no longer U33A.2
- net FILT19_OUT: now also C55.2, R19.2, U15.1; no longer C115A.2, R43A.2, U33A.1
- net FILT20_BUF: now also U15.4; no longer U33A.4
- net FILT20_OUT: now also C56.2, R20.2, U15.5; no longer C116A.2, R44A.2, U33A.5
- net FILT21_BUF: now also U16.7; no longer U34A.7
- net FILT21_OUT: now also C57.2, R21.2, U16.6; no longer C117A.2, R45A.2, U34A.6
- net FILT22_BUF: now also U16.9; no longer U34A.9
- net FILT22_OUT: now also C58.2, R22.2, U16.10; no longer C118A.2, R46A.2, U34A.10
- net FILT23_BUF: now also U18.2; no longer U36A.2
- net FILT23_OUT: now also C59.2, R23.2, U18.1; no longer C125.2, R47.2, U36A.1
- net FILT24_BUF: now also U18.4; no longer U36A.4
- net FILT24_OUT: now also C60.2, R24.2, U18.5; no longer C126A.2, R48A.2, U36A.5
- net FILT25_OUT: now also C67.2, R25.2; no longer C67A.2, R25A.2
- net FILT26_OUT: now also C68.2, R26.2; no longer C68A.2, R26A.2
- net FILT27_OUT: now also C75.2, R27.2; no longer C75A.2, R27A.2
- net FILT28_OUT: now also C76.2, R28.2; no longer C76A.2, R28A.2
- net FILT29_BUF: now also U22.7
- net FILT30_BUF: now also U22.9
- net FILT31_OUT: now also C85.2; no longer C85A.2
- net FILT32_OUT: now also C86.2; no longer C86A.2
- net FILT3_OUT: no longer C97A.2, R37A.2, U28A.6
- net GND: now also C47.2, C48.2, C65.2, C66.2, R25.1, R26.1, R27.1, R28.1, R29.1, R30.1; no longer C100A.2, C101A.2, C102A.2, C103A.2, C104A.2, C109A.2, C110A.2, C111A.2, C112A.2, C113A.2, C114A.2, C119A.2, C120A.2, C121A.2, C122A.2, C123A.2, C124A.2, C53.2, C54.2, C59.2, C60.2, C89A.2, C90A.2, C91A.2, C92A.2, C93A.2, C94A.2, C99A.2, R25A.1, R26A.1, R27A.1, R28A.1, R29A.1, R30A.1, R33A.1, R34A.1, R35A.1, R36A.1, R37A.1, R38A.1, R39A.1, R40A.1, R41A.1, R42A.1, R43A.1, R44A.1, R45A.1, R46A.1, R47.1, R48A.1
- net PIN13: now also U10.1, U11.1; no longer U28A.1, U29A.1
- net PIN14: now also U10.5, U11.5; no longer U28A.5, U29A.5
- net PIN15: now also U11.10, U12.10; no longer U29A.10, U30A.10
- net PIN16: now also U11.6, U12.6; no longer U29A.6, U30A.6
- net PIN17: now also U13.1, U14.1; no longer U31A.1, U32A.1
- net PIN18: now also U13.5, U14.5; no longer U31A.5, U32A.5
- net PIN19: now also U14.10, U15.10; no longer U32A.10, U33A.10
- net PIN20: now also U14.6, U15.6; no longer U32A.6, U33A.6
- net PIN21: now also U16.1, U17.1; no longer U34A.1, U35A.1
- net PIN22: now also U16.5, U17.5; no longer U34A.5, U35A.5
- net PIN23: now also U17.10, U18.10; no longer U35A.10, U36A.10
- net PIN24: now also U17.6, U18.6; no longer U35A.6, U36A.6
- net V+: now also C47.1, C48.1, C51.1, C61.1, C62.1, C65.1; no longer C100A.1, C103A.1, C109A.1, C110A.1, C113A.1, C119A.1, C120A.1, C123A.1, C49.1, C50.1, C53.1, C59.1, C60.1, C63.1, C89A.1, C90A.1, C93A.1, C99A.1, U25A.3, U26A.3, U27A.3, U28A.3, U29A.3, U30A.3, U31A.3, U32A.3, U33A.3, U34A.3, U35A.3, U36A.3
- net V-: now also C49.1, C50.1, C63.1, C66.1; no longer C101A.1, C102A.1, C104A.1, C111A.1, C112A.1, C114A.1, C121A.1, C122A.1, C124A.1, C51.1, C54.1, C61.1, C62.1, C91A.1, C92A.1, C94A.1, U25A.8, U26A.8, U27A.8, U28A.8, U29A.8, U30A.8, U31A.8, U32A.8, U33A.8, U34A.8, U35A.8, U36A.8
Routing:
- net GND: track 875.9 -> 615.5 mm, vias 44 -> 30
- net V+: track 621.4 -> 398.2 mm, vias 60 -> 40
- net V-: track 470.2 -> 340.2 mm, vias 60 -> 40
- net PIN38: track 30.4 -> 0.00 mm, vias 1 -> 0
- net PIN56: track 18.2 -> 0.00 mm, vias 1 -> 0
- net PIN44: track 18.2 -> 0.00 mm, vias 1 -> 0
- net PIN54: track 17.4 -> 0.00 mm, vias 1 -> 0
- net PIN42: track 17.4 -> 0.00 mm, vias 1 -> 0
- net PIN40: track 16.9 -> 0.00 mm, vias 1 -> 0
- net PIN36: track 16.5 -> 0.00 mm, vias 1 -> 0
- net PIN35: track 15.8 -> 0.00 mm, vias 1 -> 0
- net FILT2_BUF1: track 15.6 -> 0.00 mm
- net PIN34: track 15.4 -> 0.00 mm, vias 1 -> 0
- net PIN55: track 12.0 -> 0.00 mm, vias 1 -> 0
- net PIN43: track 12.0 -> 0.00 mm, vias 1 -> 0
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
Commit message: switched bypass caps to 0402
Parts:
- C1, C10, C11, C12, C13, C14, C15, C16, C17, C18, C2, C3, C39, C4, C40, C41, C42, C43, C44, C47, C48, C49, C5, C50, C51, C52, C6, C61, C62, C63, C64, C65, C66, C69, C7, C70, C71, C72, C73, C74, C77, C78, C79, C8, C80, C81, C82, C9: device resistor:C0805 -> resistor:C0402
- moved C31 37.8 mm to (84.1, 31.4)
- moved C32 37.8 mm to (77.0, 29.1)
- moved C33 37.8 mm to (84.1, 27.1)
- moved C34 37.8 mm to (77.0, 26.9)
- moved C35 37.8 mm to (84.1, 29.2)
- moved C36 37.8 mm to (77.0, 31.2)
- moved D1 37.8 mm to (84.1, 26.7)
- moved D2 37.8 mm to (77.0, 26.8)
- moved JP1 37.8 mm to (84.1, 20.1)
- moved JP2 37.8 mm to (77.0, 20.1)
- moved C64 3.45 mm to (145.8, 39.6)
- moved C2 3.43 mm to (129.3, 39.6)
- moved C10 2.57 mm to (129.5, 32.6)
- moved C62 2.57 mm to (145.8, 32.6)
- moved C14 2.30 mm to (129.5, 26.0)
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Routing:
- net V+: track 398.2 -> 467.5 mm
- net V-: track 340.2 -> 395.8 mm
- net GND: track 615.5 -> 658.6 mm
- net PIN18: track 88.9 -> 62.8 mm
- net FILT10_BUF: track 9.61 -> 29.5 mm
- net FILT9_BUF: track 7.82 -> 27.0 mm
- net FILT17_BUF: track 7.96 -> 25.4 mm
- net PIN30: track 127.9 -> 113.0 mm
- net PIN11: track 164.1 -> 171.8 mm
- net FILT28_BUF: track 1.47 -> 8.32 mm
- net PIN10: track 170.9 -> 177.7 mm
- net FILT27_BUF: track 4.29 -> 11.0 mm
- net PIN17: track 54.5 -> 48.8 mm
- net PIN12: track 170.3 -> 176.0 mm
- net PIN25: track 33.7 -> 39.1 mm
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
Commit message: Added Input resistor to ground. Started routing Dsub out
Parts:
- added R33, R34, R35, R36, R37, R38, R39, R40, R41, R42, R43, R44, R45, R46, R47, R48, R49, R50, R51, R52, R53, R54, R55, R56, R57, R58, R59, R60, R61, R62, R63, R64: (no value), resistor:R0805
- C31, C32, C33, C34, C35, C36, C37, C38, C46, C67, C68: value (none) -> 0.1uF; device resistor:C0805 -> resistor:C0402
- C45: device resistor:C0805 -> resistor:C0402
- C49, C50, C52, C73, C74, C77, C78, C79, C80, C81, C82: value 0.1uF -> (none); device resistor:C0402 -> resistor:C0805
- C51: device resistor:C0402 -> resistor:C0805
- R1, R10, R11, R12, R13, R14, R15, R16, R17, R18, R19, R2, R20, R21, R22, R23, R24, R25, R26, R27, R28, R29, R3, R30, R31, R32, R4, R5, R6, R7, R8, R9: device resistor:R0805 -> resistor:R0402
- moved C84 99.9 mm to (77.0, 26.9), flipped to the top, turned to 180 degrees
- moved C86 94.2 mm to (77.0, 31.2), turned to 180 degrees
- moved C83 93.2 mm to (84.1, 27.1), turned to 180 degrees
- moved C85 87.7 mm to (84.1, 29.2), flipped to the top, turned to 180 degrees
- moved C82 87.6 mm to (77.0, 29.1)
- moved C35 84.9 mm to (145.5, 87.8)
- moved C36 83.9 mm to (145.7, 79.4), flipped to the bottom, turned to 0 degrees
- moved C81 79.9 mm to (84.1, 31.4)
- moved C32 69.4 mm to (145.8, 38.1)
- moved C31 69.1 mm to (145.8, 62.5)
- moved C34 68.9 mm to (145.8, 29.8), flipped to the bottom, turned to 0 degrees
- moved C33 67.5 mm to (145.8, 54.4), flipped to the bottom, turned to 0 degrees
- moved R12 59.1 mm to (153.4, 82.9), turned to 90 degrees
- moved C63 58.5 mm to (161.9, 87.6), flipped to the top, turned to 180 degrees
- moved R27 56.8 mm to (137.3, 27.9), flipped to the top
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Connections:
- net BUF13: now also C49.1, U14.2, U15.2; no longer C37.1, U10.2, U11.2
- net BUF14: now also C50.1, U14.4, U15.4; no longer C38.1, U10.4, U11.4
- net BUF15: now also C51.1, U15.9, U18.9; no longer C45.1, U11.9, U12.9
- net BUF16: now also C52.1, U15.7, U18.7; no longer C46.1, U11.7, U12.7
- net BUF17: now also U10.2, U11.2; no longer U13.2, U14.2
- net BUF18: now also U10.4, U11.4; no longer U13.4, U14.4
- net BUF19: now also U11.9, U16.9; no longer U14.9, U15.9
- net BUF20: now also U11.7, U16.7; no longer U14.7, U15.7
- net BUF21: now also U12.2, U13.2; no longer U16.2, U17.2
- net BUF22: now also U12.4, U13.4; no longer U16.4, U17.4
- net BUF23: now also U13.9; no longer U18.9
- net BUF24: now also U13.7; no longer U18.7
- net BUF25: now also C73.1, U21.2, U22.2; no longer C67.1, U19.2, U20.2
- net BUF26: now also C74.1, U21.4, U22.4; no longer C68.1, U19.4, U20.4
- net BUF27: now also U22.9, U24.9; no longer U20.9, U21.9
- net BUF28: now also U22.7, U24.7; no longer U20.7, U21.7
- net BUF29: now also C77.1, U19.2, U20.2; no longer C83.1, U22.2, U23.2
- net BUF30: now also C78.1, U19.4, U20.4; no longer C84.1, U22.4, U23.4
- net BUF31: now also C79.1, U20.9; no longer C85.1, U24.9
- net BUF32: now also C80.1, U20.7; no longer C86.1, U24.7
- net FILT10_OUT: now also R42.2; no longer R10.2
- net FILT11_OUT: now also R43.2; no longer R11.2
- net FILT12_OUT: now also R44.2; no longer R12.2
- net FILT13_BUF: now also U14.7; no longer U10.7
- net FILT13_OUT: now also C49.2, R45.2, U14.6; no longer C37.2, R13.2, U10.6
- net FILT14_BUF: now also U14.9; no longer U10.9
- net FILT14_OUT: now also C50.2, R46.2, U14.10; no longer C38.2, R14.2, U10.10
- net FILT15_BUF: now also U18.2; no longer U12.2
- net FILT15_OUT: now also C51.2, R47.2, U18.1; no longer C45.2, R15.2, U12.1
- net FILT16_BUF: now also U18.4; no longer U12.4
- net FILT16_OUT: now also C52.2, R48.2, U18.5; no longer C46.2, R16.2, U12.5
- net FILT17_BUF: now also U10.7; no longer U13.7
- net FILT17_OUT: now also R49.2, U10.6; no longer R17.2, U13.6
- net FILT18_BUF: now also U10.9; no longer U13.9
- net FILT18_OUT: now also R50.2, U10.10; no longer R18.2, U13.10
- net FILT19_BUF: now also U16.2; no longer U15.2
- net FILT19_OUT: now also R51.2, U16.1; no longer R19.2, U15.1
- net FILT1_OUT: now also R33.2; no longer R1.2
- net FILT20_BUF: now also U16.4; no longer U15.4
- net FILT20_OUT: now also R52.2, U16.5; no longer R20.2, U15.5
- net FILT21_BUF: now also U12.7; no longer U16.7
- net FILT21_OUT: now also R53.2, U12.6; no longer R21.2, U16.6
- net FILT22_BUF: now also U12.9; no longer U16.9
- net FILT22_OUT: now also R54.2, U12.10; no longer R22.2, U16.10
- net FILT23_BUF: now also U17.2; no longer U18.2
- net FILT23_OUT: now also R55.2, U17.1; no longer R23.2, U18.1
- net FILT24_BUF: now also U17.4; no longer U18.4
- net FILT24_OUT: now also R56.2, U17.5; no longer R24.2, U18.5
- net FILT25_BUF: now also U21.7; no longer U19.7
- net FILT25_OUT: now also C73.2, R57.2, U21.6; no longer C67.2, R25.2, U19.6
- net FILT26_BUF: now also U21.9; no longer U19.9
- net FILT26_OUT: now also C74.2, R58.2, U21.10; no longer C68.2, R26.2, U19.10
- net FILT27_BUF: now also U24.2; no longer U21.2
- net FILT27_OUT: now also R59.2, U24.1; no longer R27.2, U21.1
- net FILT28_BUF: now also U24.4; no longer U21.4
- net FILT28_OUT: now also R60.2, U24.5; no longer R28.2, U21.5
- net FILT29_BUF: now also U19.7; no longer U22.7
- net FILT29_OUT: now also C77.2, R61.2, U19.6; no longer C83.2, R29.2, U22.6
- net FILT2_OUT: now also R34.2; no longer R2.2
- net FILT30_BUF: now also U19.9; no longer U22.9
- net FILT30_OUT: now also C78.2, R62.2, U19.10; no longer C84.2, R30.2, U22.10
- net FILT31_BUF: now also U23.2; no longer U24.2
- net FILT31_OUT: now also C79.2, R63.2, U23.1; no longer C85.2, R31.2, U24.1
- net FILT32_BUF: now also U23.4; no longer U24.4
- net FILT32_OUT: now also C80.2, R64.2, U23.5; no longer C86.2, R32.2, U24.5
- net FILT3_OUT: now also R35.2; no longer R3.2
- net FILT4_OUT: now also R36.2; no longer R4.2
- net FILT5_OUT: now also R37.2; no longer R5.2
- net FILT6_OUT: now also R38.2; no longer R6.2
- net FILT7_OUT: now also R39.2; no longer R7.2
- net FILT8_OUT: now also R40.2; no longer R8.2
- net FILT9_OUT: now also R41.2; no longer R9.2
- net GND: now also C37.2, C38.2, C45.2, C46.2, C67.2, C68.2, C83.2, C84.2, C85.2, C86.2, R33.1, R34.1, R35.1, R36.1, R37.1, R38.1, R39.1, R40.1, R41.1, R42.1, R43.1, R44.1, R45.1, R46.1, R47.1, R48.1, R49.1, R50.1, R51.1, R52.1, R53.1, R54.1, R55.1, R56.1, R57.1, R58.1, R59.1, R60.1, R61.1, R62.1, R63.1, R64.1; no longer C49.2, C50.2, C51.2, C52.2, C73.2, C74.2, C77.2, C78.2, C79.2, C80.2
- net PIN1: now also R1.2
- net PIN10: now also R11.2
- net PIN11: now also R19.2
- net PIN12: now also R27.2
- net PIN13: now also R4.2, U14.1, U15.1; no longer U10.1, U11.1
- net PIN14: now also R12.2, U14.5, U15.5; no longer U10.5, U11.5
- net PIN15: now also R20.2, U15.10, U18.10; no longer U11.10, U12.10
- net PIN16: now also R28.2, U15.6, U18.6; no longer U11.6, U12.6
- net PIN17: now also R5.2, U10.1, U11.1; no longer U13.1, U14.1
- net PIN18: now also R13.2, U10.5, U11.5; no longer U13.5, U14.5
- net PIN19: now also R21.2, U11.10, U16.10; no longer U14.10, U15.10
- net PIN2: now also R9.2
- net PIN20: now also R29.2, U11.6, U16.6; no longer U14.6, U15.6
- net PIN21: now also R6.2, U12.1, U13.1; no longer U16.1, U17.1
- net PIN22: now also R14.2, U12.5, U13.5; no longer U16.5, U17.5
- net PIN23: now also R22.2, U13.10; no longer U18.10
- net PIN24: now also R30.2, U13.6; no longer U18.6
- net PIN25: now also R7.2, U21.1, U22.1; no longer U19.1, U20.1
- net PIN26: now also R15.2, U21.5, U22.5; no longer U19.5, U20.5
- net PIN27: now also R23.2, U22.10, U24.10; no longer U20.10, U21.10
- net PIN28: now also R31.2, U22.6, U24.6; no longer U20.6, U21.6
- net PIN29: now also R8.2, U19.1, U20.1; no longer U22.1, U23.1
- net PIN3: now also R17.2
- net PIN30: now also R16.2, U19.5, U20.5; no longer U22.5, U23.5
- net PIN31: now also R24.2, U20.10; no longer U24.10
- net PIN32: now also R32.2, U20.6; no longer U24.6
- net PIN4: now also R25.2
- net PIN5: now also R2.2
- net PIN6: now also R10.2
- net PIN7: now also R18.2
- net PIN8: now also R26.2
- net PIN9: now also R3.2
- net V+: now also C37.1, C38.1, C41.1, C42.1, C46.1, C66.1, C67.1, C68.1, C71.1, C72.1, C83.1, C85.1; no longer C31.1, C33.1, C35.1, C43.1, C51.1, C61.1, C62.1, C69.1, C70.1, C73.1, C77.1, C78.1
- net V-: now also C31.1, C33.1, C35.1, C43.1, C45.1, C61.1, C62.1, C69.1, C70.1, C84.1, C86.1; no longer C41.1, C42.1, C49.1, C50.1, C52.1, C66.1, C71.1, C72.1, C74.1, C79.1, C80.1
Routing:
- net GND: track 658.6 -> 562.8 mm, vias 30 -> 29
- net FILT5_BUF: track 7.96 -> 86.6 mm, vias 0 -> 1
- net FILT6_BUF: track 11.0 -> 87.2 mm, vias 0 -> 1
- net FILT8_BUF: track 6.29 -> 67.0 mm
- net FILT7_BUF: track 9.42 -> 68.8 mm
- net FILT20_BUF: track 6.29 -> 61.7 mm, vias 0 -> 1
- net FILT24_BUF: track 6.55 -> 58.9 mm
- net FILT23_BUF: track 10.3 -> 61.2 mm
- net FILT21_BUF: track 9.00 -> 54.2 mm, vias 0 -> 1
- net FILT22_BUF: track 12.2 -> 54.9 mm, vias 0 -> 1
- net FILT16_BUF: track 9.34 -> 48.0 mm, vias 0 -> 1
- net FILT15_BUF: track 11.9 -> 50.2 mm, vias 0 -> 1
- net FILT29_BUF: track 7.96 -> 40.7 mm
- net FILT4_BUF: track 8.96 -> 41.4 mm
- net FILT3_BUF: track 11.9 -> 44.2 mm
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
Commit message: Finished dsub out and GND routing. Starting V planes
Parts:
- moved X1 14.0 mm to (184.3, 55.2)
- moved R23 1.59 mm to (162.8, 76.6), flipped to the bottom, turned to 270 degrees
- moved C11 0.76 mm to (129.4, 85.7)
- moved C12 0.76 mm to (129.4, 80.0)
- moved C15 0.76 mm to (129.4, 73.3)
- moved C18 0.76 mm to (129.4, 72.0)
- moved C19 0.76 mm to (137.5, 86.2)
- moved C20 0.76 mm to (137.5, 86.2)
- moved C21 0.76 mm to (136.8, 72.8)
- moved C22 0.76 mm to (136.8, 72.8)
- moved C35 0.76 mm to (145.5, 87.0)
- moved C36 0.76 mm to (145.7, 78.6)
- moved C41 0.76 mm to (145.5, 85.7)
- moved C42 0.76 mm to (145.7, 79.9)
- moved C45 0.76 mm to (145.7, 73.3)
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Routing:
- net GND: track 562.8 -> 301.4 mm, vias 29 -> 42
- net V+: track 474.9 -> 239.6 mm
- net V-: track 412.2 -> 254.1 mm
- net FILT2_BUF: track 11.0 -> 113.7 mm, vias 0 -> 2
- net FILT1_BUF: track 7.96 -> 110.3 mm, vias 0 -> 2
- net FILT12_BUF: track 6.55 -> 107.8 mm, vias 0 -> 1
- net FILT11_BUF: track 10.3 -> 106.9 mm, vias 0 -> 1
- net FILT25_BUF: track 7.96 -> 57.6 mm, vias 0 -> 1
- net FILT26_BUF: track 11.0 -> 57.9 mm, vias 0 -> 1
- net FILT19_BUF: track 26.3 -> 72.5 mm
- net FILT9_BUF: track 27.0 -> 64.6 mm
- net FILT3_BUF: track 44.2 -> 81.3 mm, vias 0 -> 1
- net FILT10_BUF: track 29.5 -> 65.7 mm
- net FILT4_BUF: track 41.4 -> 76.9 mm, vias 0 -> 1
- net FILT32_BUF: track 6.29 -> 39.2 mm, vias 0 -> 1
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- added copper zone on layer 2, net V+
- added copper zone on layer 2, net V-
