File: schematics/Connector.Filter.Board/Connector.Board.brd (EAGLE design)
At the start: 188 x 72 mm, 212 parts, among them U1 AD8244, U10 AD8244, U11 AD8244, U12 AD8244, U13 AD8244, U14 AD8244, U15 AD8244, U16 AD8244, U17 AD8244, U18 AD8244, U19 AD8244, U2 AD8244, U20 AD8244, U21 AD8244, U22 AD8244, U23 AD8244, U24 AD8244, U3 AD8244, U4 AD8244, U5 AD8244, U6 AD8244, U7 AD8244, U8 AD8244, U9 AD8244, X1 EEGCON, X2 EITCON

Commit message: Finished PWR GND
Parts:
- added J1, J2: (no value), SparkFun-Connectors:JST-2-SMD
- added JP3, JP4: (no value), pinhead:2X02
- added LED1, LED2: (no value), led:SML0805
- added R65, R66: (no value), resistor:R0402
- C81, C82: value (none) -> 2.2uF
- C83, C84: value (none) -> 0.1uF; device resistor:C0805 -> resistor:C0402
- C85, C86: value (none) -> 10nF; device resistor:C0805 -> resistor:C0402
- JP1, JP2: device pinhead:1X02/90 -> pinhead:1X02
- moved C86 44.6 mm to (121.4, 27.6), flipped to the bottom, turned to 270 degrees
- moved C84 43.3 mm to (120.3, 27.6), flipped to the bottom, turned to 270 degrees
- moved C82 41.7 mm to (118.6, 27.7), flipped to the bottom, turned to 270 degrees
- moved D2 41.4 mm to (118.4, 27.6), flipped to the top, turned to 90 degrees
- moved JP2 34.5 mm to (110.6, 27.6), flipped to the bottom, turned to 90 degrees
- moved C85 7.98 mm to (91.8, 27.3), flipped to the bottom, turned to 90 degrees
- moved JP1 7.97 mm to (81.0, 27.4), flipped to the bottom, turned to 90 degrees
- moved C83 6.61 mm to (90.7, 27.3), flipped to the bottom, turned to 90 degrees
- moved C81 6.41 mm to (89.0, 27.3), flipped to the bottom, turned to 90 degrees
- moved D1 4.87 mm to (88.9, 27.3), flipped to the top, turned to 90 degrees
Connections:
- new net B1+: J1.2, JP1.1, JP3.1
- new net B1-: J1.1, JP1.2, JP3.3
- new net B2+: J2.2, JP2.1, JP4.1
- new net B2-: J2.1, JP2.2, JP4.3
- new net N$11: LED2.C, R66.1
- new net N$9: LED1.C, R65.2
- net GND: now also JP3.4, JP4.2, R65.1, R66.2; no longer JP1.2, JP2.2
- net V+: now also JP3.2, LED1.A; no longer JP1.1
- net V-: now also JP4.4, LED2.A; no longer JP2.1
Routing:
- net GND: track 301.4 -> 243.7 mm
- net V-: track 254.1 -> 237.9 mm
- net V+: track 239.6 -> 224.7 mm, vias 40 -> 39
- net B2-: track 0.00 -> 7.08 mm
- net B2+: track 0.00 -> 7.08 mm
- net B1-: track 0.00 -> 6.95 mm
- net B1+: track 0.00 -> 6.95 mm
- net FILT24_BUF: track 67.7 -> 72.6 mm
- net FILT11_BUF: track 106.9 -> 111.7 mm
- net FILT12_BUF: track 107.8 -> 112.6 mm
- net FILT6_BUF: track 81.4 -> 77.6 mm
- net FILT5_BUF: track 77.9 -> 74.6 mm
- net FILT9_BUF: track 64.6 -> 61.8 mm
- net N$11: track 0.00 -> 1.82 mm
- net N$9: track 0.00 -> 1.82 mm
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
Commit message: Most of pins to AMPs routed
Routing:
- net PIN25: track 40.3 -> 193.9 mm, vias 1 -> 2
- net PIN26: track 56.2 -> 193.0 mm
- net PIN9: track 169.9 -> 47.1 mm
- net PIN10: track 179.9 -> 64.9 mm
- net PIN17: track 50.0 -> 162.9 mm
- net PIN27: track 70.4 -> 181.5 mm, vias 1 -> 2
- net PIN28: track 76.0 -> 185.8 mm
- net PIN11: track 174.2 -> 67.1 mm
- net PIN18: track 64.3 -> 164.4 mm
- net PIN12: track 180.0 -> 83.1 mm
- net PIN29: track 93.5 -> 185.3 mm, vias 1 -> 2
- net PIN19: track 72.7 -> 160.5 mm
- net PIN30: track 114.2 -> 191.9 mm
- net PIN20: track 90.8 -> 166.2 mm, vias 2 -> 3
- net PIN13: track 87.5 -> 160.9 mm, vias 2 -> 3
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