File: schematics/Connector.Filter.Board/Connector.Board.brd (EAGLE design)
At the start: 192 x 73.3 mm, 220 parts, among them J1 V+BATT, J2 V-BATT, U1 AD8244, U10 AD8244, U11 AD8244, U12 AD8244, U13 AD8244, U14 AD8244, U15 AD8244, U16 AD8244, U17 AD8244, U18 AD8244, U19 AD8244, U2 AD8244, U20 AD8244, U21 AD8244, U22 AD8244, U23 AD8244, U24 AD8244, U3 AD8244, U4 AD8244, U5 AD8244, U6 AD8244, U7 AD8244, U8 AD8244, U9 AD8244, X1 EEGCON, X2 EITCON

Commit message: Fiddling with the case design
Parts:
- added C87, C88, C89, C90: 0.1uF, resistor:C0402
- added PAT_GND, PAT_GND2: TOUCHPROOF, connector_board_lib:TOUCHPROOF_PIN
- added U25, U26: AD8244, AD8244:MSOP10
Connections:
- new net PAT_GND: PAT_GND.TP, PAT_GND2.TP, U25.2, U25.4, U25.7, U25.9, U26.2, U26.4, U26.7, U26.9
- net GND: now also C87.2, C88.2, C89.2, C90.2, U25.1, U25.10, U25.5, U25.6, U26.1, U26.10, U26.5, U26.6
- net V+: now also C87.1, C89.1, U25.3, U26.3
- net V-: now also C88.1, C90.1, U25.8, U26.8
Changed lines of the file:
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@@
 <dimension x1="32.893" y1="78.486" x2="30.226" y2="91.948" x3="51.054" y3="85.217" textsize="1.778" layer="47" dtype="vertical"/>
 <dimension x1="32.893" y1="78.486" x2="3.937" y2="91.948" x3="18.415" y3="92.964" textsize="1.778" layer="47" dtype="horizontal"/>
+<dimension x1="88.392" y1="21.971" x2="83.693" y2="40.386" x3="79.375" y3="31.1785" textsize="1.778" layer="47" dtype="vertical"/>
+<dimension x1="121.666" y1="40.386" x2="121.412" y2="22.098" x3="121.539" y3="16.129" textsize="1.778" layer="47" dtype="horizontal"/>
 </plain>
 <attributes>
@@
 <attribute name="VALUE" x="121.285" y="21.082" size="1.27" layer="27" rot="R90"/>
 </element>
+<element name="U25" library="AD8244" package="MSOP10" value="AD8244" x="64.262" y="28.829"/>
+<element name="C87" library="resistor" package="C0402" value="0.1uF" x="-18.034" y="1.905"/>
+<element name="C88" library="resistor" package="C0402" value="0.1uF" x="-18.034" y="-2.921"/>
+<element name="PAT_GND" library="connector_board_lib" package="TOUCHPROOF_PIN" value="TOUCHPROOF" x="38.862" y="29.464">
+<attribute name="TP_SIGNAL_NAME" value="" x="38.862" y="29.464" size="1.778" layer="27" display="off"/>
+</element>
+<element name="PAT_GND2" library="connector_board_lib" package="TOUCHPROOF_PIN" value="TOUCHPROOF" x="52.324" y="29.591">
+<attribute name="TP_SIGNAL_NAME" value="" x="52.324" y="29.591" size="1.778" layer="27" display="off"/>
+</element>
+<element name="U26" library="AD8244" package="MSOP10" value="AD8244" x="-16.764" y="-36.83"/>
+<element name="C89" library="resistor" package="C0402" value="0.1uF" x="-18.034" y="-41.783"/>
+<element name="C90" library="resistor" package="C0402" value="0.1uF" x="-18.034" y="-46.609"/>
 </elements>
 <signals>
@@
 <wire x1="145.019" y1="79.883" x2="145.019" y2="79.98" width="0.2" layer="16"/>
 <wire x1="145.019" y1="79.98" x2="146.558" y2="81.519" width="0.2" layer="16"/>
+<contactref element="C87" pad="2"/>
+<contactref element="C88" pad="2"/>
+<contactref element="U25" pad="1"/>
+<contactref element="U25" pad="5"/>
+<contactref element="U25" pad="10"/>
+<contactref element="U25" pad="6"/>
+<contactref element="C89" pad="2"/>
+<contactref element="C90" pad="2"/>
+<contactref element="U26" pad="1"/>
+<contactref element="U26" pad="5"/>
+<contactref element="U26" pad="10"/>
+<contactref element="U26" pad="6"/>
+<wire x1="63.262" y1="30.879" x2="65.262" y2="30.879" width="0" layer="19" extent="1-1"/>
+<wire x1="65.262" y1="26.779" x2="65.262" y2="30.879" width="0" layer="19" extent="1-1"/>
+<wire x1="63.262" y1="26.779" x2="65.262" y2="26.779" width="0" layer="19" extent="1-1"/>
+<wire x1="69.977" y1="32.385" x2="65.262" y2="30.879" width="0" layer="19" extent="1-1"/>
+<wire x1="-17.384" y1="1.905" x2="63.262" y2="26.779" width="0" layer="19" extent="1-1"/>
+<wire x1="-17.384" y1="-2.921" x2="-17.384" y2="1.905" width="0" layer="19" extent="1-1"/>
+<wire x1="-17.764" y1="-34.78" x2="-17.384" y2="-2.921" width="0" layer="19" extent="1-1"/>
+<wire x1="-15.764" y1="-34.78" x2="-17.764" y2="-34.78" width="0" layer="19" extent="1-1"/>
+<wire x1="-17.764" y1="-38.88" x2="-17.764" y2="-34.78" width="0" layer="19" extent="1-1"/>
+<wire x1="-15.764" y1="-38.88" x2="-17.764" y2="-38.88" width="0" layer="19" extent="1-1"/>
+<wire x1="-17.384" y1="-41.783" x2="-17.764" y2="-38.88" width="0" layer="19" extent="1-1"/>
+<wire x1="-17.384" y1="-46.609" x2="-17.384" y2="-41.783" width="0" layer="19" extent="1-1"/>
 </signal>
 <signal name="V-">
@@
 <wire x1="121.412" y1="23.148" x2="121.412" y2="27.935" width="0.2" layer="1"/>
 <wire x1="121.412" y1="27.935" x2="121.031" y2="28.316" width="0.2" layer="1"/>
+<contactref element="U25" pad="8"/>
+<contactref element="C88" pad="1"/>
+<contactref element="U26" pad="8"/>
+<contactref element="C90" pad="1"/>
+<wire x1="117.729" y1="28.829" x2="64.262" y2="30.879" width="0" layer="19" extent="1-16"/>
+<wire x1="-18.684" y1="-2.921" x2="64.262" y2="30.879" width="0" layer="19" extent="1-1"/>
+<wire x1="-16.764" y1="-34.78" x2="-18.684" y2="-2.921" width="0" layer="19" extent="1-1"/>
+<wire x1="-18.684" y1="-46.609" x2="-16.764" y2="-34.78" width="0" layer="19" extent="1-1"/>
 </signal>
 <signal name="V+">
@@
 <wire x1="91.313" y1="26.655" x2="92.441" y2="26.655" width="0.2" layer="16"/>
 <wire x1="92.441" y1="26.655" x2="92.456" y2="26.67" width="0.2" layer="16"/>
+<contactref element="U25" pad="3"/>
+<contactref element="C87" pad="1"/>
+<contactref element="U26" pad="3"/>
+<contactref element="C89" pad="1"/>
+<wire x1="85.979" y1="26.162" x2="64.262" y2="26.779" width="0" layer="19" extent="1-1"/>
+<wire x1="-18.684" y1="1.905" x2="64.262" y2="26.779" width="0" layer="19" extent="1-1"/>
+<wire x1="-16.764" y1="-38.88" x2="-18.684" y2="1.905" width="0" layer="19" extent="1-1"/>
+<wire x1="-18.684" y1="-41.783" x2="-16.764" y2="-38.88" width="0" layer="19" extent="1-1"/>
 </signal>
 <signal name="FILT1_BUF">
@@
 <wire x1="121.412" y1="21.067" x2="121.412" y2="21.048" width="0.2" layer="1"/>
 </signal>
+<signal name="PAT_GND">
+<contactref element="U25" pad="2"/>
+<contactref element="U25" pad="4"/>
+<contactref element="U25" pad="9"/>
+<contactref element="U25" pad="7"/>
+<contactref element="U26" pad="2"/>
+<contactref element="U26" pad="4"/>
+<contactref element="U26" pad="9"/>
+<contactref element="U26" pad="7"/>
+<contactref element="PAT_GND" pad="TP"/>
+<contactref element="PAT_GND2" pad="TP"/>
+<wire x1="64.762" y1="30.879" x2="63.762" y2="30.879" width="0" layer="19" extent="1-1"/>
+<wire x1="63.762" y1="26.779" x2="63.762" y2="30.879" width="0" layer="19" extent="1-1"/>
+<wire x1="64.762" y1="26.779" x2="63.762" y2="26.779" width="0" layer="19" extent="1-1"/>
+<wire x1="52.324" y1="29.591" x2="63.762" y2="30.879" width="0" layer="19" extent="1-1"/>
+<wire x1="38.862" y1="29.464" x2="52.324" y2="29.591" width="0" layer="19" extent="1-1"/>
+<wire x1="-16.264" y1="-34.78" x2="38.862" y2="29.464" width="0" layer="19" extent="1-1"/>
+<wire x1="-17.264" y1="-34.78" x2="-16.264" y2="-34.78" width="0" layer="19" extent="1-1"/>
+<wire x1="-17.264" y1="-38.88" x2="-17.264" y2="-34.78" width="0" layer="19" extent="1-1"/>
+<wire x1="-16.264" y1="-38.88" x2="-17.264" y2="-38.88" width="0" layer="19" extent="1-1"/>
+</signal>
 </signals>

Commit message: Added buffered ground
Parts:
- added PAT_GND1: TOUCHPROOF, connector_board_lib:TOUCHPROOF_PIN
- moved C90 109.6 mm to (59.8, 30.5), flipped to the bottom
- moved C89 101.2 mm to (59.7, 23.0), flipped to the bottom
- moved U26 99.8 mm to (60.3, 26.5), flipped to the bottom
- moved C88 84.7 mm to (59.8, 30.4), turned to 180 degrees
- moved C87 80.5 mm to (59.7, 23.0), turned to 180 degrees
- moved PAT_GND 12.2 mm to (26.8, 27.4)
- moved PAT_GND2 9.67 mm to (42.9, 27.3)
- moved U25 4.55 mm to (60.3, 26.5)
Connections:
- net PAT_GND: now also PAT_GND1.TP
Routing:
- net V-: track 243.3 -> 314.2 mm, vias 41 -> 42
- net GND: track 246.6 -> 304.7 mm, vias 50 -> 54
- net PAT_GND: track 0.00 -> 52.0 mm, vias 0 -> 1
- net V+: track 273.5 -> 308.2 mm, vias 41 -> 42
Other:
- board text added: "EEG HP FILTER"
- board text added: "UCL EIT"
- board text added: "V1.5"
- board text removed: "UCL EIT EEG HP FILTER"

Commit message: Added battery charger and Voltage inverter
Parts:
- removed J1: V+BATT, SparkFun-Connectors:JST-2-SMD
- removed J2: V-BATT, SparkFun-Connectors:JST-2-SMD
- removed JP1: Batt1_backup, pinhead:1X02
- removed JP2: Batt2_backup, pinhead:1X02
- removed JP3: Batt2_SW, pinhead:2X02
- added C91, C92, C93, C94: 10uF, resistor:C0805
- added JP5: IN, SparkFun:1X02
- added LED3: YELLOW, led:SML0805
- added LED4: GREEN, led:SML0805
- added R67: 2k, rcl:M0805
- added R68: 470, rcl:M0805
- added R69: 1k, rcl:M0805
- added U27: MCP73831, SparkFun-PowerIC:SOT23-5
- added U28: LTC1044ACS8PBF, LTC1044ACS8PBF:SOIC127P600X175-8N
- added X3: (no value), Molex-47346-0001:MOLEX_47346-0001
- added X7: JST-XH-02-PIN-LONG-PAD, Rembrandt Electronics - JST XH Connectors v1-0:JST-XH-02-PACKAGE-LONG-PAD
- moved D2 150.3 mm to (-16.8, -34.9), turned to 0 degrees
- moved D1 119.4 mm to (-16.8, -29.3), turned to 0 degrees
Connections:
- removed net B1+: J1.2, JP1.1, JP4.1
- removed net B1-: J1.1, JP1.2, JP4.3
- removed net B2+: J2.2, JP2.1, JP3.1
- removed net B2-: J2.1, JP2.2, JP3.3
- new net 5VIN: C92.1, D1.C, JP5.1, LED3.A, U27.4, X3.1
- new net BOOST: U28.1
- new net CHRG: LED3.C, R68.2
- new net N$2: C93.1, U28.2
- new net N$3: C93.2, U28.4
- new net N$5: LED4.A, R69.2
- new net PROG: R67.2, U27.5
- new net STAT: R68.1, R69.1, U27.1
- new net VBATT_A: C91.1, D2.C, JP4.1, U27.3, X7.2
- net GND: now also C91.2, C92.2, C94.2, D2.A, JP5.2, LED4.C, R67.1, U27.2, U28.3, X3.5, X7.1; no longer D2.C, JP3.2, JP4.4
- net V+: now also U28.8; no longer D1.C
- net V-: now also C94.1, U28.5; no longer D2.A, JP3.4
Routing:
- net GND: track 304.7 -> 293.6 mm
- net V-: track 314.2 -> 306.7 mm
- net B2-: track 7.33 -> 0.00 mm
- net B2+: track 7.33 -> 0.00 mm
- net B1-: track 7.21 -> 0.00 mm
- net B1+: track 7.21 -> 0.00 mm
- net V+: track 308.2 -> 304.2 mm

Commit message: Inital board layout for Voltage inverter and battery charger
Parts:
- removed C91: 10uF, resistor:C0805
- removed JP4: Batt1_SW, pinhead:2X02
- added S1: PVA1F, switch-misc:PVA1F
- R67, R68, R69: device rcl:M0805 -> rcl:R0402
- moved C94 165.2 mm to (117.0, 26.8), turned to 270 degrees
- moved C93 157.0 mm to (113.8, 20.2)
- moved U28 152.7 mm to (113.2, 25.3), turned to 90 degrees
- moved D2 122.3 mm to (88.3, 27.7), flipped to the bottom, turned to 90 degrees
- moved R68 112.3 mm to (87.5, 21.3), turned to 90 degrees
- moved LED4 111.0 mm to (83.9, 21.0), turned to 90 degrees
- moved X7 110.5 mm to (91.3, 27.9), flipped to the bottom, turned to 270 degrees
- moved D1 108.9 mm to (75.8, 27.9)
- moved R69 106.9 mm to (86.4, 21.3), turned to 90 degrees
- moved U27 106.9 mm to (82.8, 28.8), turned to 90 degrees
- moved JP5 99.2 mm to (74.4, 25.3)
- moved LED3 98.1 mm to (81.7, 21.0), turned to 270 degrees
- moved C92 94.7 mm to (79.6, 28.8), turned to 270 degrees
- moved X3 92.4 mm to (75.7, 22.9)
- moved R67 90.9 mm to (82.5, 25.3), turned to 180 degrees
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Connections:
- net GND: no longer C91.2
- net V+: now also S1.1; no longer JP4.2
- net VBATT_A: now also S1.2; no longer C91.1, JP4.1
Routing:
- net GND: track 293.6 -> 409.4 mm, vias 54 -> 60
- net V+: track 304.2 -> 337.3 mm, vias 42 -> 43
- net 5VIN: track 0.00 -> 30.5 mm, vias 0 -> 2
- net VBATT_A: track 0.00 -> 25.4 mm, vias 0 -> 2
- net V-: track 306.7 -> 325.0 mm, vias 42 -> 43
- net STAT: track 0.00 -> 11.9 mm
- net CHRG: track 0.00 -> 8.02 mm
- net N$3: track 0.00 -> 2.75 mm
- net N$2: track 0.00 -> 2.75 mm
- net PROG: track 0.00 -> 2.66 mm
- net N$5: track 0.00 -> 2.62 mm
- net N$1: track 2.05 -> 1.51 mm

Commit message: removed lib autosaved
Parts:
- moved PAT_GND 0.13 mm to (26.8, 27.3)
Routing:
- net V+: track 337.3 -> 333.5 mm
- net 5VIN: track 30.5 -> 31.0 mm
Other:
- board text added: "5Vin"
- board text added: "CRG"
- board text added: "FULL"
- board text added: "VBatt"
- board text removed: "V+ ON"
- board text removed: "V- ON"
