File: schematics/Connector.Filter.Board/Connector.Board.sch (EAGLE design)
At the start: 12 parts, among them U1 RC4560S08-RC4560

Commit message: Added parts for 2 channels
Parts:
- removed R3: 220k, resistor:R-EU_M0805
- removed R4: 1k, resistor:R-EU_M0805
- removed U1: RC4560S08-RC4560, RC4560:RC4560S08-RC4560
- added C3, C4: (no value), resistor:C-EUC0805
- added JP1, JP2: (no value), pinhead:PINHD-1X2/90
- added TP10, TP11, TP12, TP13, TP14, TP15, TP16, TP17, TP18, TP19, TP20, TP21, TP22, TP23, TP24, TP25, TP26, TP27, TP28, TP29, TP3, TP30, TP31, TP32, TP4, TP5, TP6, TP7, TP8, TP9: TOUCHPROOF, connector_board_lib:TOUCHPROOF
- C2: value 200uF -> (none)
- R2: value 220k -> (none); device resistor:R-EU_M0805 -> resistor:R-EU_R0805
- TP1, TP2: value PTR1PAD1-13 -> TOUCHPROOF; device testpad:PTR1PAD1-13 -> connector_board_lib:TOUCHPROOF
Connections:
- removed net N$2: R2.1, R3.2, U1.POSA
- removed net N$6: R4.2, U1.OUTA
- new net BUF2: C2.1, U$1.OUT_D, U$2.OUT_B
- new net FILT2_BUF: U$1.OUT_C
- new net FILT2_OUT: C2.2, R2.2, U$1.IN_C
- net FILT1_BUF: no longer TP2.TP
- net GND: now also C3.2, C4.2, JP1.2, JP2.2, R2.1; no longer R4.1, U1.NEGA
- net PIN10: now also TP10.TP
- net PIN11: now also TP11.TP
- net PIN12: now also TP12.TP
- net PIN13: now also TP13.TP
- net PIN14: now also TP14.TP
- net PIN15: now also TP15.TP
- net PIN16: now also TP16.TP
- net PIN17: now also TP17.TP
- net PIN18: now also TP18.TP
- net PIN19: now also TP19.TP
- net PIN2: now also TP2.TP, U$1.IN_D, U$2.IN_B
- net PIN20: now also TP20.TP
- net PIN21: now also TP21.TP
- net PIN22: now also TP22.TP
- net PIN23: now also TP23.TP
- net PIN24: now also TP24.TP
- net PIN25: now also TP25.TP
- net PIN26: now also TP26.TP
- net PIN27: now also TP27.TP
- net PIN28: now also TP28.TP
- net PIN29: now also TP29.TP
- net PIN3: now also TP3.TP
- net PIN30: now also TP30.TP
- net PIN31: now also TP31.TP
- net PIN32: now also TP32.TP
- net PIN4: now also TP4.TP
- net PIN5: now also TP5.TP
- net PIN6: now also TP6.TP
- net PIN7: now also TP7.TP
- net PIN8: now also TP8.TP
- net PIN9: now also TP9.TP
- net VDD: now also C4.1, JP2.1; no longer C2.1, R2.2, U1.V+
- net VSS: now also C3.1, JP1.1; no longer C2.2, R3.1, U1.V-

Commit message: example layout for 4 channels
Parts:
- added C10, C11, C12, C5, C6, C7, C8, C9: (no value), resistor:C-EUC0805
- added R3, R4: (no value), resistor:R-EU_R0805
- added U$3: AD8244, AD8244:AD8244
- added X2: (no value), con-subd:M37HP
Connections:
- new net BUF3: C11.1, U$2.OUT_C, U$3.OUT_C
- new net BUF4: C12.1, U$2.OUT_D, U$3.OUT_D
- new net FILT10_BUF: X2.10
- new net FILT11_BUF: X2.11
- new net FILT12_BUF: X2.12
- new net FILT13_BUF: X2.13
- new net FILT14_BUF: X2.14
- new net FILT15_BUF: X2.15
- new net FILT16_BUF: X2.16
- new net FILT17_BUF: X2.17
- new net FILT18_BUF: X2.18
- new net FILT19_BUF: X2.19
- new net FILT20_BUF: X2.20
- new net FILT21_BUF: X2.21
- new net FILT22_BUF: X2.22
- new net FILT23_BUF: X2.23
- new net FILT24_BUF: X2.24
- new net FILT25_BUF: X2.25
- new net FILT26_BUF: X2.26
- new net FILT27_BUF: X2.27
- new net FILT28_BUF: X2.28
- new net FILT29_BUF: X2.29
- new net FILT30_BUF: X2.30
- new net FILT31_BUF: X2.31
- new net FILT32_BUF: X2.32
- new net FILT3_BUF: U$3.OUT_A, X2.3
- new net FILT3_OUT: C11.2, R3.2, U$3.IN_A
- new net FILT4_BUF: U$3.OUT_B, X2.4
- new net FILT4_OUT: C12.2, R4.2, U$3.IN_B
- new net FILT5_BUF: X2.5
- new net FILT6_BUF: X2.6
- new net FILT7_BUF: X2.7
- new net FILT8_BUF: X2.8
- new net FILT9_BUF: X2.9
- net BUF2: now also U$1.OUT_B; no longer U$1.OUT_D
- net FILT1_BUF: now also U$1.OUT_D, X2.1; no longer U$1.OUT_B
- net FILT1_OUT: now also U$1.IN_D; no longer U$1.IN_B
- net FILT2_BUF: now also X2.2
- net GND: now also C10.2, C5.2, C6.2, C7.2, C8.2, C9.2, R3.1, R4.1
- net PIN2: now also U$1.IN_B; no longer U$1.IN_D
- net PIN3: now also U$2.IN_C, U$3.IN_C
- net PIN4: now also U$2.IN_D, U$3.IN_D
- net VDD: now also C10.1, C7.1, C8.1, U$1.V-, U$2.V-, U$3.V-; no longer U$1.V+
- net VSS: now also C5.1, C6.1, C9.1, U$1.V+, U$2.V+, U$3.V+; no longer U$1.V-, U$2.V-
Other:
- moved on the sheet: C1, C2, R1, R2

Commit message: Duplicated layout through renaming parts
Parts:
- added C13, C14, C15, C16, C17, C18, C19, C20, C21, C22: (no value), resistor:C-EUC0805
- added R5, R6, R7, R8: (no value), resistor:R-EU_R0805
- added U$4, U$5, U$6: AD8244, AD8244:AD8244
Connections:
- new net BUF5: C19.1, U$4.OUT_A, U$5.OUT_A
- new net BUF6: C20.1, U$4.OUT_B, U$5.OUT_B
- new net BUF7: C21.1, U$5.OUT_C, U$6.OUT_C
- new net BUF8: C22.1, U$5.OUT_D, U$6.OUT_D
- new net FILT5_OUT: C19.2, R5.2, U$4.IN_D
- new net FILT6_OUT: C20.2, R6.2, U$4.IN_C
- new net FILT7_OUT: C21.2, R7.2, U$6.IN_A
- new net FILT8_OUT: C22.2, R8.2, U$6.IN_B
- net FILT5_BUF: now also U$4.OUT_D
- net FILT6_BUF: now also U$4.OUT_C
- net FILT7_BUF: now also U$6.OUT_A
- net FILT8_BUF: now also U$6.OUT_B
- net GND: now also C13.2, C14.2, C15.2, C16.2, C17.2, C18.2, R5.1, R6.1, R7.1, R8.1
- net PIN5: now also U$4.IN_A, U$5.IN_A
- net PIN6: now also U$4.IN_B, U$5.IN_B
- net PIN7: now also U$5.IN_C, U$6.IN_C
- net PIN8: now also U$5.IN_D, U$6.IN_D
- net VDD: now also C15.1, C16.1, C18.1, U$4.V-, U$5.V-, U$6.V-
- net VSS: now also C13.1, C14.1, C17.1, U$4.V+, U$5.V+, U$6.V+

Commit message: 12 chn board finished
Parts:
- added C23, C24, C25, C26, C27, C28, C29, C30, C31, C32, C33, C34, C35, C36: (no value), resistor:C-EUC0805
- added D1, D3: 1N4148W-7-F, diode:DIODE-SOD123
- added R10, R11, R12, R9: (no value), resistor:R-EU_R0805
- added U$7, U$8, U$9: AD8244, AD8244:AD8244
Connections:
- removed net VDD: C10.1, C15.1, C16.1, C18.1, C4.1, C7.1, C8.1, JP2.1, U$1.V-, U$2.V-, U$3.V-, U$4.V-, U$5.V-, U$6.V-
- removed net VSS: C13.1, C14.1, C17.1, C3.1, C5.1, C6.1, C9.1, JP1.1, U$1.V+, U$2.V+, U$3.V+, U$4.V+, U$5.V+, U$6.V+
- new net BUF10: C28.1, U$7.OUT_B, U$8.OUT_B
- new net BUF11: C29.1, U$8.OUT_C, U$9.OUT_C
- new net BUF12: C30.1, U$8.OUT_D, U$9.OUT_D
- new net BUF9: C27.1, U$7.OUT_A, U$8.OUT_A
- new net FILT10_OUT: C28.2, R10.2, U$7.IN_C
- new net FILT11_OUT: C29.2, R11.2, U$9.IN_A
- new net FILT12_OUT: C30.2, R12.2, U$9.IN_B
- new net FILT9_OUT: C27.2, R9.2, U$7.IN_D
- new net V+: C13.1, C14.1, C17.1, C23.1, C24.1, C3.1, C31.1, C32.1, C35.1, C5.1, C6.1, C9.1, D1.C, JP1.1, U$1.V+, U$2.V+, U$3.V+, U$4.V+, U$5.V+, U$6.V+, U$7.V+, U$8.V+, U$9.V+
- new net V-: C10.1, C15.1, C16.1, C18.1, C25.1, C26.1, C33.1, C34.1, C36.1, C4.1, C7.1, C8.1, D3.A, JP2.1, U$1.V-, U$2.V-, U$3.V-, U$4.V-, U$5.V-, U$6.V-, U$7.V-, U$8.V-, U$9.V-
- net FILT10_BUF: now also U$7.OUT_C
- net FILT11_BUF: now also U$9.OUT_A
- net FILT12_BUF: now also U$9.OUT_B
- net FILT9_BUF: now also U$7.OUT_D
- net GND: now also C23.2, C24.2, C25.2, C26.2, C31.2, C32.2, C33.2, C34.2, C35.2, C36.2, D1.A, D3.C, R10.1, R11.1, R12.1, R9.1
- net PIN10: now also U$7.IN_B, U$8.IN_B
- net PIN11: now also U$8.IN_C, U$9.IN_C
- net PIN12: now also U$8.IN_D, U$9.IN_D
- net PIN9: now also U$7.IN_A, U$8.IN_A
