File: schematics/Connector.Filter.Board/Connector.Board.sch (EAGLE design)
At the start: 95 parts, among them U1 AD8244, U2 AD8244, U3 AD8244, U4 AD8244, U5 AD8244, U6 AD8244, U7 AD8244, U8 AD8244, U9 AD8244, X1 EEGCON, X2 EITCON

Commit message: Renaming Sch and Brd but not matching yet
Parts:
- added C37, C38, C46, C53, C54, C55, C56, C57, C58, C59, C60, C67, C68, C76, C83, C84, C85, C86: (no value), resistor:C-EUC0805
- added C39, C40, C41, C42, C43, C44, C45, C47, C48, C49, C50, C51, C52, C61, C62, C63, C64, C65, C66, C69, C70, C71, C72, C73, C74, C75, C77, C78, C79, C80, C81, C82: 0.1uF, resistor:C-EUC0805
- added R13, R14, R15, R16, R17, R18, R19, R20, R21, R22, R23, R24, R25, R26, R27, R28, R29, R30, R31, R32: (no value), resistor:R-EU_R0805
- added U10, U11, U12, U13, U14, U15, U16, U17, U18, U19, U20, U21, U22, U23, U24: AD8244, AD8244:AD8244
Connections:
- new net BUF13: C37.1, U10.OUT_A, U11.OUT_A
- new net BUF14: C38.1, U10.OUT_B, U11.OUT_B
- new net BUF15: C45.1, U11.OUT_C, U12.OUT_C
- new net BUF16: C46.1, U11.OUT_D, U12.OUT_D
- new net BUF17: C53.1, U13.OUT_A, U14.OUT_A
- new net BUF18: C54.1, U13.OUT_B, U14.OUT_B
- new net BUF19: C55.1, U14.OUT_C, U15.OUT_C
- new net BUF20: C56.1, U14.OUT_D, U15.OUT_D
- new net BUF21: C57.1, U16.OUT_A, U17.OUT_A
- new net BUF22: C58.1, U16.OUT_B, U17.OUT_B
- new net BUF23: C59.1, U17.OUT_C, U18.OUT_C
- new net BUF24: C60.1, U17.OUT_D, U18.OUT_D
- new net BUF25: C67.1, U19.OUT_A, U20.OUT_A
- new net BUF26: C68.1, U19.OUT_B, U20.OUT_B
- new net BUF27: C75.1, U20.OUT_C, U21.OUT_C
- new net BUF28: C76.1, U20.OUT_D, U21.OUT_D
- new net BUF29: C83.1, U22.OUT_A, U23.OUT_A
- new net BUF30: C84.1, U22.OUT_B, U23.OUT_B
- new net BUF31: C85.1, U23.OUT_C, U24.OUT_C
- new net BUF32: C86.1, U23.OUT_D, U24.OUT_D
- new net FILT13_OUT: C37.2, R13.2, U10.IN_D
- new net FILT14_OUT: C38.2, R14.2, U10.IN_C
- new net FILT15_OUT: C45.2, R15.2, U12.IN_A
- new net FILT16_OUT: C46.2, R16.2, U12.IN_B
- new net FILT17_OUT: C53.2, R17.2, U13.IN_D
- new net FILT18_OUT: C54.2, R18.2, U13.IN_C
- new net FILT19_OUT: C55.2, R19.2, U15.IN_A
- new net FILT20_OUT: C56.2, R20.2, U15.IN_B
- new net FILT21_OUT: C57.2, R21.2, U16.IN_D
- new net FILT22_OUT: C58.2, R22.2, U16.IN_C
- new net FILT23_OUT: C59.2, R23.2, U18.IN_A
- new net FILT24_OUT: C60.2, R24.2, U18.IN_B
- new net FILT25_OUT: C67.2, R25.2, U19.IN_D
- new net FILT26_OUT: C68.2, R26.2, U19.IN_C
- new net FILT27_OUT: C75.2, R27.2, U21.IN_A
- new net FILT28_OUT: C76.2, R28.2, U21.IN_B
- new net FILT29_OUT: C83.2, R29.2, U22.IN_D
- new net FILT30_OUT: C84.2, R30.2, U22.IN_C
- new net FILT31_OUT: C85.2, R31.2, U24.IN_A
- new net FILT32_OUT: C86.2, R32.2, U24.IN_B
- net FILT13_BUF: now also U10.OUT_D
- net FILT14_BUF: now also U10.OUT_C
- net FILT15_BUF: now also U12.OUT_A
- net FILT16_BUF: now also U12.OUT_B
- net FILT17_BUF: now also U13.OUT_D
- net FILT18_BUF: now also U13.OUT_C
- net FILT19_BUF: now also U15.OUT_A
- net FILT20_BUF: now also U15.OUT_B
- net FILT21_BUF: now also U16.OUT_D
- net FILT22_BUF: now also U16.OUT_C
- net FILT23_BUF: now also U18.OUT_A
- net FILT24_BUF: now also U18.OUT_B
- net FILT25_BUF: now also U19.OUT_D
- net FILT26_BUF: now also U19.OUT_C
- net FILT27_BUF: now also U21.OUT_A
- net FILT28_BUF: now also U21.OUT_B
- net FILT29_BUF: now also U22.OUT_D
- net FILT30_BUF: now also U22.OUT_C
- net FILT31_BUF: now also U24.OUT_A
- net FILT32_BUF: now also U24.OUT_B
- net GND: now also C39.2, C40.2, C41.2, C42.2, C43.2, C44.2, C47.2, C48.2, C49.2, C50.2, C51.2, C52.2, C61.2, C62.2, C63.2, C64.2, C65.2, C66.2, C69.2, C70.2, C71.2, C72.2, C73.2, C74.2, C77.2, C78.2, C79.2, C80.2, C81.2, C82.2, R13.1, R14.1, R15.1, R16.1, R17.1, R18.1, R19.1, R20.1, R21.1, R22.1, R23.1, R24.1, R25.1, R26.1, R27.1, R28.1, R29.1, R30.1, R31.1, R32.1
- net PIN13: now also U10.IN_A, U11.IN_A
- net PIN14: now also U10.IN_B, U11.IN_B
- net PIN15: now also U11.IN_C, U12.IN_C
- net PIN16: now also U11.IN_D, U12.IN_D
- net PIN17: now also U13.IN_A, U14.IN_A
- net PIN18: now also U13.IN_B, U14.IN_B
- net PIN19: now also U14.IN_C, U15.IN_C
- net PIN20: now also U14.IN_D, U15.IN_D
- net PIN21: now also U16.IN_A, U17.IN_A
- net PIN22: now also U16.IN_B, U17.IN_B
- net PIN23: now also U17.IN_C, U18.IN_C
- net PIN24: now also U17.IN_D, U18.IN_D
- net PIN25: now also U19.IN_A, U20.IN_A
- net PIN26: now also U19.IN_B, U20.IN_B
- net PIN27: now also U20.IN_C, U21.IN_C
- net PIN28: now also U20.IN_D, U21.IN_D
- net PIN29: now also U22.IN_A, U23.IN_A
- net PIN30: now also U22.IN_B, U23.IN_B
- net PIN31: now also U23.IN_C, U24.IN_C
- net PIN32: now also U23.IN_D, U24.IN_D
- net V+: now also C39.1, C40.1, C43.1, C47.1, C48.1, C51.1, C61.1, C62.1, C65.1, C69.1, C70.1, C73.1, C77.1, C78.1, C81.1, U10.V+, U11.V+, U12.V+, U13.V+, U14.V+, U15.V+, U16.V+, U17.V+, U18.V+, U19.V+, U20.V+, U21.V+, U22.V+, U23.V+, U24.V+
- net V-: now also C41.1, C42.1, C44.1, C49.1, C50.1, C52.1, C63.1, C64.1, C66.1, C71.1, C72.1, C74.1, C79.1, C80.1, C82.1, U10.V-, U11.V-, U12.V-, U13.V-, U14.V-, U15.V-, U16.V-, U17.V-, U18.V-, U19.V-, U20.V-, U21.V-, U22.V-, U23.V-, U24.V-
Other:
- moved on the sheet: C19, C20, C21, C22, C23, C24, C25, C26, C27, C28, C29, C30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

Commit message: switched bypass caps to 0402
Parts:
- C1, C10, C11, C12, C13, C14, C15, C16, C17, C18, C2, C3, C39, C4, C40, C41, C42, C43, C44, C47, C48, C49, C5, C50, C51, C52, C6, C61, C62, C63, C64, C65, C66, C69, C7, C70, C71, C72, C73, C74, C77, C78, C79, C8, C80, C81, C82, C9: device resistor:C-EUC0805 -> resistor:C-EUC0402

Commit message: Added Input resistor to ground. Started routing Dsub out
Parts:
- added R33, R34, R35, R36, R37, R38, R39, R40, R41, R42, R43, R44, R45, R46, R47, R48, R49, R50, R51, R52, R53, R54, R55, R56, R57, R58, R59, R60, R61, R62, R63, R64: (no value), resistor:R-EU_R0805
- C31, C32, C33, C34, C35, C36, C37, C38, C46, C67, C68: value (none) -> 0.1uF; device resistor:C-EUC0805 -> resistor:C-EUC0402
- C45: device resistor:C-EUC0805 -> resistor:C-EUC0402
- C49, C50, C52, C73, C74, C77, C78, C79, C80, C81, C82: value 0.1uF -> (none); device resistor:C-EUC0402 -> resistor:C-EUC0805
- C51: device resistor:C-EUC0402 -> resistor:C-EUC0805
- R1, R10, R11, R12, R13, R14, R15, R16, R17, R18, R19, R2, R20, R21, R22, R23, R24, R25, R26, R27, R28, R29, R3, R30, R31, R32, R4, R5, R6, R7, R8, R9: device resistor:R-EU_R0805 -> resistor:R-EU_R0402
Connections:
- net BUF13: now also C49.1, U14.OUT_A, U15.OUT_A; no longer C37.1, U10.OUT_A, U11.OUT_A
- net BUF14: now also C50.1, U14.OUT_B, U15.OUT_B; no longer C38.1, U10.OUT_B, U11.OUT_B
- net BUF15: now also C51.1, U15.OUT_C, U18.OUT_C; no longer C45.1, U11.OUT_C, U12.OUT_C
- net BUF16: now also C52.1, U15.OUT_D, U18.OUT_D; no longer C46.1, U11.OUT_D, U12.OUT_D
- net BUF17: now also U10.OUT_A, U11.OUT_A; no longer U13.OUT_A, U14.OUT_A
- net BUF18: now also U10.OUT_B, U11.OUT_B; no longer U13.OUT_B, U14.OUT_B
- net BUF19: now also U11.OUT_C, U16.OUT_C; no longer U14.OUT_C, U15.OUT_C
- net BUF20: now also U11.OUT_D, U16.OUT_D; no longer U14.OUT_D, U15.OUT_D
- net BUF21: now also U12.OUT_A, U13.OUT_A; no longer U16.OUT_A, U17.OUT_A
- net BUF22: now also U12.OUT_B, U13.OUT_B; no longer U16.OUT_B, U17.OUT_B
- net BUF23: now also U13.OUT_C; no longer U18.OUT_C
- net BUF24: now also U13.OUT_D; no longer U18.OUT_D
- net BUF25: now also C73.1, U21.OUT_A, U22.OUT_A; no longer C67.1, U19.OUT_A, U20.OUT_A
- net BUF26: now also C74.1, U21.OUT_B, U22.OUT_B; no longer C68.1, U19.OUT_B, U20.OUT_B
- net BUF27: now also U22.OUT_C, U24.OUT_C; no longer U20.OUT_C, U21.OUT_C
- net BUF28: now also U22.OUT_D, U24.OUT_D; no longer U20.OUT_D, U21.OUT_D
- net BUF29: now also C77.1, U19.OUT_A, U20.OUT_A; no longer C83.1, U22.OUT_A, U23.OUT_A
- net BUF30: now also C78.1, U19.OUT_B, U20.OUT_B; no longer C84.1, U22.OUT_B, U23.OUT_B
- net BUF31: now also C79.1, U20.OUT_C; no longer C85.1, U24.OUT_C
- net BUF32: now also C80.1, U20.OUT_D; no longer C86.1, U24.OUT_D
- net FILT10_OUT: now also R42.2; no longer R10.2
- net FILT11_OUT: now also R43.2; no longer R11.2
- net FILT12_OUT: now also R44.2; no longer R12.2
- net FILT13_BUF: now also U14.OUT_D; no longer U10.OUT_D
- net FILT13_OUT: now also C49.2, R45.2, U14.IN_D; no longer C37.2, R13.2, U10.IN_D
- net FILT14_BUF: now also U14.OUT_C; no longer U10.OUT_C
- net FILT14_OUT: now also C50.2, R46.2, U14.IN_C; no longer C38.2, R14.2, U10.IN_C
- net FILT15_BUF: now also U18.OUT_A; no longer U12.OUT_A
- net FILT15_OUT: now also C51.2, R47.2, U18.IN_A; no longer C45.2, R15.2, U12.IN_A
- net FILT16_BUF: now also U18.OUT_B; no longer U12.OUT_B
- net FILT16_OUT: now also C52.2, R48.2, U18.IN_B; no longer C46.2, R16.2, U12.IN_B
- net FILT17_BUF: now also U10.OUT_D; no longer U13.OUT_D
- net FILT17_OUT: now also R49.2, U10.IN_D; no longer R17.2, U13.IN_D
- net FILT18_BUF: now also U10.OUT_C; no longer U13.OUT_C
- net FILT18_OUT: now also R50.2, U10.IN_C; no longer R18.2, U13.IN_C
- net FILT19_BUF: now also U16.OUT_A; no longer U15.OUT_A
- net FILT19_OUT: now also R51.2, U16.IN_A; no longer R19.2, U15.IN_A
- net FILT1_OUT: now also R33.2; no longer R1.2
- net FILT20_BUF: now also U16.OUT_B; no longer U15.OUT_B
- net FILT20_OUT: now also R52.2, U16.IN_B; no longer R20.2, U15.IN_B
- net FILT21_BUF: now also U12.OUT_D; no longer U16.OUT_D
- net FILT21_OUT: now also R53.2, U12.IN_D; no longer R21.2, U16.IN_D
- net FILT22_BUF: now also U12.OUT_C; no longer U16.OUT_C
- net FILT22_OUT: now also R54.2, U12.IN_C; no longer R22.2, U16.IN_C
- net FILT23_BUF: now also U17.OUT_A; no longer U18.OUT_A
- net FILT23_OUT: now also R55.2, U17.IN_A; no longer R23.2, U18.IN_A
- net FILT24_BUF: now also U17.OUT_B; no longer U18.OUT_B
- net FILT24_OUT: now also R56.2, U17.IN_B; no longer R24.2, U18.IN_B
- net FILT25_BUF: now also U21.OUT_D; no longer U19.OUT_D
- net FILT25_OUT: now also C73.2, R57.2, U21.IN_D; no longer C67.2, R25.2, U19.IN_D
- net FILT26_BUF: now also U21.OUT_C; no longer U19.OUT_C
- net FILT26_OUT: now also C74.2, R58.2, U21.IN_C; no longer C68.2, R26.2, U19.IN_C
- net FILT27_BUF: now also U24.OUT_A; no longer U21.OUT_A
- net FILT27_OUT: now also R59.2, U24.IN_A; no longer R27.2, U21.IN_A
- net FILT28_BUF: now also U24.OUT_B; no longer U21.OUT_B
- net FILT28_OUT: now also R60.2, U24.IN_B; no longer R28.2, U21.IN_B
- net FILT29_BUF: now also U19.OUT_D; no longer U22.OUT_D
- net FILT29_OUT: now also C77.2, R61.2, U19.IN_D; no longer C83.2, R29.2, U22.IN_D
- net FILT2_OUT: now also R34.2; no longer R2.2
- net FILT30_BUF: now also U19.OUT_C; no longer U22.OUT_C
- net FILT30_OUT: now also C78.2, R62.2, U19.IN_C; no longer C84.2, R30.2, U22.IN_C
- net FILT31_BUF: now also U23.OUT_A; no longer U24.OUT_A
- net FILT31_OUT: now also C79.2, R63.2, U23.IN_A; no longer C85.2, R31.2, U24.IN_A
- net FILT32_BUF: now also U23.OUT_B; no longer U24.OUT_B
- net FILT32_OUT: now also C80.2, R64.2, U23.IN_B; no longer C86.2, R32.2, U24.IN_B
- net FILT3_OUT: now also R35.2; no longer R3.2
- net FILT4_OUT: now also R36.2; no longer R4.2
- net FILT5_OUT: now also R37.2; no longer R5.2
- net FILT6_OUT: now also R38.2; no longer R6.2
- net FILT7_OUT: now also R39.2; no longer R7.2
- net FILT8_OUT: now also R40.2; no longer R8.2
- net FILT9_OUT: now also R41.2; no longer R9.2
- net GND: now also C37.2, C38.2, C45.2, C46.2, C67.2, C68.2, C83.2, C84.2, C85.2, C86.2, R33.1, R34.1, R35.1, R36.1, R37.1, R38.1, R39.1, R40.1, R41.1, R42.1, R43.1, R44.1, R45.1, R46.1, R47.1, R48.1, R49.1, R50.1, R51.1, R52.1, R53.1, R54.1, R55.1, R56.1, R57.1, R58.1, R59.1, R60.1, R61.1, R62.1, R63.1, R64.1; no longer C49.2, C50.2, C51.2, C52.2, C73.2, C74.2, C77.2, C78.2, C79.2, C80.2
- net PIN1: now also R1.2
- net PIN10: now also R11.2
- net PIN11: now also R19.2
- net PIN12: now also R27.2
- net PIN13: now also R4.2, U14.IN_A, U15.IN_A; no longer U10.IN_A, U11.IN_A
- net PIN14: now also R12.2, U14.IN_B, U15.IN_B; no longer U10.IN_B, U11.IN_B
- net PIN15: now also R20.2, U15.IN_C, U18.IN_C; no longer U11.IN_C, U12.IN_C
- net PIN16: now also R28.2, U15.IN_D, U18.IN_D; no longer U11.IN_D, U12.IN_D
- net PIN17: now also R5.2, U10.IN_A, U11.IN_A; no longer U13.IN_A, U14.IN_A
- net PIN18: now also R13.2, U10.IN_B, U11.IN_B; no longer U13.IN_B, U14.IN_B
- net PIN19: now also R21.2, U11.IN_C, U16.IN_C; no longer U14.IN_C, U15.IN_C
- net PIN2: now also R9.2
- net PIN20: now also R29.2, U11.IN_D, U16.IN_D; no longer U14.IN_D, U15.IN_D
- net PIN21: now also R6.2, U12.IN_A, U13.IN_A; no longer U16.IN_A, U17.IN_A
- net PIN22: now also R14.2, U12.IN_B, U13.IN_B; no longer U16.IN_B, U17.IN_B
- net PIN23: now also R22.2, U13.IN_C; no longer U18.IN_C
- net PIN24: now also R30.2, U13.IN_D; no longer U18.IN_D
- net PIN25: now also R7.2, U21.IN_A, U22.IN_A; no longer U19.IN_A, U20.IN_A
- net PIN26: now also R15.2, U21.IN_B, U22.IN_B; no longer U19.IN_B, U20.IN_B
- net PIN27: now also R23.2, U22.IN_C, U24.IN_C; no longer U20.IN_C, U21.IN_C
- net PIN28: now also R31.2, U22.IN_D, U24.IN_D; no longer U20.IN_D, U21.IN_D
- net PIN29: now also R8.2, U19.IN_A, U20.IN_A; no longer U22.IN_A, U23.IN_A
- net PIN3: now also R17.2
- net PIN30: now also R16.2, U19.IN_B, U20.IN_B; no longer U22.IN_B, U23.IN_B
- net PIN31: now also R24.2, U20.IN_C; no longer U24.IN_C
- net PIN32: now also R32.2, U20.IN_D; no longer U24.IN_D
- net PIN4: now also R25.2
- net PIN5: now also R2.2
- net PIN6: now also R10.2
- net PIN7: now also R18.2
- net PIN8: now also R26.2
- net PIN9: now also R3.2
- net V+: now also C37.1, C38.1, C41.1, C42.1, C46.1, C66.1, C67.1, C68.1, C71.1, C72.1, C83.1, C85.1; no longer C31.1, C33.1, C35.1, C43.1, C51.1, C61.1, C62.1, C69.1, C70.1, C73.1, C77.1, C78.1
- net V-: now also C31.1, C33.1, C35.1, C43.1, C45.1, C61.1, C62.1, C69.1, C70.1, C84.1, C86.1; no longer C41.1, C42.1, C49.1, C50.1, C52.1, C66.1, C71.1, C72.1, C74.1, C79.1, C80.1
