File: schematics/Connector.Filter.Board/Connector.Board.sch (EAGLE design)
At the start: 228 parts, among them J1 V+BATT, J2 V-BATT, U1 AD8244, U10 AD8244, U11 AD8244, U12 AD8244, U13 AD8244, U14 AD8244, U15 AD8244, U16 AD8244, U17 AD8244, U18 AD8244, U19 AD8244, U2 AD8244, U20 AD8244, U21 AD8244, U22 AD8244, U23 AD8244, U24 AD8244, U25 AD8244, U26 AD8244, U3 AD8244, U4 AD8244, U5 AD8244, U6 AD8244, U7 AD8244, U8 AD8244, U9 AD8244, X1 EEGCON, X2 EITCON

Commit message: Added buffered ground
Parts:
- added PAT_GND1: TOUCHPROOF, connector_board_lib:TOUCHPROOF
Connections:
- net PAT_GND: now also PAT_GND1.TP
Changed lines of the file:
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@@
 <part name="GND116" library="supply1" deviceset="GND" device=""/>
 <part name="GND118" library="supply1" deviceset="GND" device=""/>
+<part name="PAT_GND1" library="connector_board_lib" deviceset="TOUCHPROOF" device=""/>
 </parts>
 <sheets>
@@
 <instance part="GND116" gate="1" x="25.4" y="-50.8"/>
 <instance part="GND118" gate="1" x="0" y="-20.32"/>
+<instance part="PAT_GND1" gate="G$1" x="154.94" y="48.26" rot="R270"/>
 </instances>
 <busses>
@@
 <junction x="172.72" y="58.42"/>
 <label x="180.34" y="58.42" size="1.778" layer="95"/>
+<pinref part="PAT_GND1" gate="G$1" pin="TP"/>
+<wire x1="160.02" y1="48.26" x2="172.72" y2="48.26" width="0.1524" layer="91"/>
+<wire x1="172.72" y1="48.26" x2="172.72" y2="55.88" width="0.1524" layer="91"/>
+<junction x="172.72" y="55.88"/>
 </segment>
 </net>

Commit message: Added battery charger and Voltage inverter
Parts:
- removed J1: V+BATT, SparkFun-Connectors:JST_2MM_MALE
- removed J2: V-BATT, SparkFun-Connectors:JST_2MM_MALE
- removed JP1: Batt1_backup, pinhead:PINHD-1X2
- removed JP2: Batt2_backup, pinhead:PINHD-1X2
- removed JP3: Batt2_SW, pinhead:PINHD-2X2
- added C91, C92, C93, C94: 10uF, resistor:C-EUC0805
- added JP5: IN, SparkFun:M02PTH
- added LED3: YELLOW, led:LEDSML0805
- added LED4: GREEN, led:LEDSML0805
- added R67: 2k, rcl:R-EU_M0805
- added R68: 470, rcl:R-EU_M0805
- added R69: 1k, rcl:R-EU_M0805
- added U27: MCP73831, SparkFun-PowerIC:MCP73831
- added U28: LTC1044ACS8PBF, LTC1044ACS8PBF:LTC1044ACS8PBF
- added X3: (no value), Molex-47346-0001:47346-0001
- added X7: JST-XH-02-PIN-LONG-PAD, Rembrandt Electronics - JST XH Connectors v1-0:JST-XH-02-PIN-LONG-PAD
Connections:
- removed net B1+: J1.+, JP1.1, JP4.1
- removed net B1-: J1.-, JP1.2, JP4.3
- removed net B2+: J2.+, JP2.1, JP3.1
- removed net B2-: J2.-, JP2.2, JP3.3
- new net 5VIN: C92.1, D1.C, JP5.1, LED3.A, U27.VIN, X3.1
- new net CHRG: LED3.C, R68.2
- new net N$2: C93.1, U28.CAP+
- new net N$3: C93.2, U28.CAP-
- new net N$5: LED4.A, R69.2
- new net PROG: R67.2, U27.PROG
- new net STAT: R68.1, R69.1, U27.STAT
- new net VBATT_A: C91.1, D2.C, JP4.1, U27.VBAT, X7-2.S
- net GND: now also C91.2, C92.2, C94.2, D2.A, JP5.2, LED4.C, R67.1, U27.VSS, U28.GROUND, X3.5, X7-1.S; no longer D2.C, JP3.2, JP4.4
- net V+: now also U28.V+; no longer D1.C
- net V-: now also C94.1, U28.VOUT; no longer D2.A, JP3.4
Other:
- note added: "2K R programs for 500mA output (i think this is most efficient)"
- note added: "BATTERY CHARGER"
- moved on the sheet: C81, C82, C83, C84, C85, C86, D1, D2, JP4, LED1, LED2, R65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

Commit message: Inital board layout for Voltage inverter and battery charger
Parts:
- removed C91: 10uF, resistor:C-EUC0805
- removed JP4: Batt1_SW, pinhead:PINHD-2X2
- added S1: PVA1F, switch-misc:PVA1F
- R67, R68, R69: device rcl:R-EU_M0805 -> rcl:R-EU_R0402
Connections:
- net GND: no longer C91.2
- net V+: now also S11.S; no longer JP4.2
- net VBATT_A: now also S11.P; no longer C91.1, JP4.1
Other:
- moved on the sheet: D2
