File: schematics/Current.Source.AD9954/Low.Noise.Current.Source.brd (EAGLE design)
At the start: 160 x 100 mm, 77 parts, among them IC1 REG1117, IC2 REG1117, U1 AD9954YSVZ, U2 LTC69000, U4 LTC1044CS8PBF

Commit message: Final layout tweaks done and Gerbers generated
Parts:
- renumbered TP6 to IOUT+, TP7 to IOUT-
Other:
- board text added: "Ard"
- board text added: "Bat"
- board text added: "Flip switch up for Arduino power and down for external battery"
- board text added: "Set jumper for output current: 2k: 500uA 5k: 200uA 10k: 100uA"
- board text added: "UCL AD9954 Current Source T. Dowrick 17.7.17"
- board text added: "Use .1% resistors in this area"
- board text removed: "Checklist DAC Decoupling done Todo Power/ground planes for DDS"

Commit message: Schematic and PCB desig for AD9954 low noise current source
Parts:
- R_SET1_0.1%: value 7.838k -> 7.87k
Changed lines of the file:
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@@
 <attribute name="VALUE" x="128.822" y="65.006" size="1.27" layer="27" rot="R180"/>
 </element>
-<element name="R_SET1_0.1%" library="adafruit" package="R0805" value="7.838k" x="87.28" y="75.34" smashed="yes">
+<element name="R_SET1_0.1%" library="adafruit" package="R0805" value="7.87k" x="87.28" y="75.34" smashed="yes">
 <attribute name="VALUE" x="85.718" y="77.054" size="1.27" layer="27"/>
 </element>
