File: schematics/Current.Source.AD9954/Low.Noise.Current.Source.sch (EAGLE design)
At the start: 77 parts, among them IC1 REG1117, IC2 REG1117, U1 AD9954YSVZ, U2 LTC69000, U4 LTC1044CS8PBF

Commit message: Final layout tweaks done and Gerbers generated
Parts:
- renumbered TP6 to IOUT+, TP7 to IOUT-
Other:
- note removed: "TODO: EPAD is the ICB bottom paddle. Needs to be connected to AGND"
- note removed: "TODO: Is a 3.3V regulator needed for DVDD_I/O?"
Changed lines of the file:
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@@
 <part name="GND21" library="supply1" deviceset="GND" device=""/>
 <part name="TP5" library="testpad" deviceset="PTR1" device="PAD1-13"/>
-<part name="TP6" library="testpad" deviceset="PTR1" device="PAD1-13"/>
-<part name="TP7" library="testpad" deviceset="PTR1" device="PAD1-13"/>
+<part name="IOUT+" library="testpad" deviceset="PTR1" device="PAD1-13"/>
+<part name="IOUT-" library="testpad" deviceset="PTR1" device="PAD1-13"/>
 <part name="VIN_POS" library="testpad" deviceset="PTR1" device="PAD1-13"/>
 <part name="VIN_NEG" library="testpad" deviceset="PTR1" device="PAD1-13"/>
@@
 Switch selects between the two.</text>
 <text x="121.92" y="246.38" size="1.778" layer="91">Battery Connectors</text>
-<text x="15.24" y="76.2" size="1.778" layer="91">TODO: Is a 3.3V regulator needed for DVDD_I/O?</text>
 <text x="160.02" y="182.88" size="1.778" layer="91">All other voltages supplied by Arduino/regulators</text>
 </plain>
@@
 <text x="-134.62" y="96.52" size="1.778" layer="91">Set CLKMODESELECT low to enable
 external clock input on REFCLK</text>
-<text x="-134.62" y="22.86" size="1.778" layer="91">TODO: EPAD is the ICB bottom paddle.
-Needs to be connected to AGND</text>
 <text x="-134.62" y="60.96" size="1.778" layer="91">DAC output current set by:
 R_SET = 39.19/I_OUT
@@
 <instance part="GND21" gate="1" x="157.48" y="81.28"/>
 <instance part="TP5" gate="G$1" x="99.06" y="134.62" rot="R180"/>
-<instance part="TP6" gate="G$1" x="165.1" y="119.38" rot="R180"/>
-<instance part="TP7" gate="G$1" x="165.1" y="99.06" rot="R180"/>
+<instance part="IOUT+" gate="G$1" x="165.1" y="119.38" rot="R180"/>
+<instance part="IOUT-" gate="G$1" x="165.1" y="99.06" rot="R180"/>
 <instance part="C34" gate="G$1" x="208.28" y="-20.32" rot="R180"/>
 <instance part="C38" gate="G$1" x="208.28" y="-43.18" rot="R180"/>
@@
 <wire x1="157.48" y1="96.52" x2="157.48" y2="83.82" width="0.1524" layer="91"/>
 <pinref part="GND21" gate="1" pin="GND"/>
-<pinref part="TP7" gate="G$1" pin="TP"/>
+<pinref part="IOUT-" gate="G$1" pin="TP"/>
 <junction x="157.48" y="96.52"/>
 </segment>
@@
 <wire x1="157.48" y1="116.84" x2="165.1" y2="116.84" width="0.1524" layer="91"/>
 <wire x1="157.48" y1="116.84" x2="157.48" y2="111.76" width="0.1524" layer="91"/>
-<pinref part="TP6" gate="G$1" pin="TP"/>
+<pinref part="IOUT+" gate="G$1" pin="TP"/>
 <junction x="157.48" y="116.84"/>
 <junction x="139.7" y="116.84"/>

Commit message: Schematic and PCB desig for AD9954 low noise current source
Parts:
- R_SET1_0.1%: value 7.838k -> 7.87k
Other:
- note added: "DAC output current set by: R_SET = 39.19/I_OUT 7.838k = 5mA (Using 7.87k, closest standard value) Iout affects the resistor values needed for the DAC output stage Using 5mA means that the resistor values needed are close to 'standard' values."
- note removed: "DAC output current set by: R_SET = 39.19/I_OUT 7.838k = 5mA Iout affects the resistor values needed for the DAC output stage Using 5mA means that the resistor values needed are close to 'standard' values."
Changed lines of the file:
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@@
 <part name="C27" library="resistor" deviceset="C-EU" device="C0603" value="0.1uF"/>
 <part name="C28" library="resistor" deviceset="C-EU" device="C0603" value="10uF"/>
-<part name="R_SET1_0.1%" library="adafruit" deviceset="R-US_" device="R0805" value="7.838k"/>
+<part name="R_SET1_0.1%" library="adafruit" deviceset="R-US_" device="R0805" value="7.87k"/>
 <part name="RX_DAC_1%" library="adafruit" deviceset="R-US_" device="R0805" value="287"/>
 <part name="R4_DAC_1%" library="adafruit" deviceset="R-US_" device="R0805" value="1150"/>
@@
 <text x="-134.62" y="60.96" size="1.778" layer="91">DAC output current set by:
 R_SET = 39.19/I_OUT
-7.838k = 5mA
+7.838k = 5mA (Using 7.87k,
+closest standard value)
 Iout affects the resistor values
 needed for the DAC output stage
